File: nu.ai_motor_controller/microcontroller.sch (KiCad schematic (older format))
At the start: 11 parts

Commit message: automated commit
Parts:
- removed R?: RC0603JR-071KL, 0603, symbol custom:RC0603JR-071KL
- added D?: CM1293A-04SO, SOT-457, symbol custom:CM1293A-04SO
- added F?: MF-MSMF050-2, 1812, symbol custom:MF-MSMF050-2
- added R?: RMCF0603FT22R0, 0603, symbol custom:RMCF0603FT22R0
- added R?: RC0603JR-070RL, Resistor_SMD:R_0603_1608Metric, symbol custom:RC0603JR-070RL
- added R?: RC0603JR-071KL, 0603, symbol custom:RC0603JR-071KL
Connections:
- wire segments 47 -> 59
Other:
- note added: "PLACE CLOSE TO\nMICRO USB\nCONNECTOR"
- note removed: "put .5A resettable fuse on vbus\n"
- note removed: "use CM1293A-04SO on data lines"
- moved on the sheet: C?, J?, R?

Commit message: automated commit
Parts:
- added C? (x2): C0603C180K5RACAUTO, Capacitor_SMD:C_0603_1608Metric, symbol custom:C0603C180K5RACAUTO
- added C?: CL10B104KO8NNNC, Capacitor_SMD:C_0603_1608Metric, symbol custom:CL10B104KO8NNNC
- added C?: ‎CL21A475KLCLQNC‎, Capacitor_SMD:C_0805_2012Metric, symbol custom:‎CL21A475KLCLQNC‎
- added C?: NP_C_0603, Capacitor_SMD:C_0603_1608Metric, symbol custom:NP_C_0603
- added C?: NP_C_0402, Capacitor_SMD:C_0402_1005Metric, symbol custom:NP_C_0402
- added Y?: 7M-16.000MAAE-T, symbol custom:7M-16.000MAAE-T
Connections:
- net +5V: now also C?.1, C?.1, C?.1, C?.1
- net GND: now also C?.2, C?.2, C?.2, C?.2, C?.2, C?.2, Y?.2, Y?.4
- net at U?.16 (XTAL2): now also C?.1, Y?.3
- net at U?.17 (XTAL1): now also C?.1, Y?.1
- no-connect marks 1 -> 2
Other:
- note added: "PLACE CLOSE\nTO IC PINS"
- moved on the sheet: C?, D?, F?, J?, L?, R?, U?
