File: nu.ai_motor_controller/microcontroller.sch (KiCad schematic (older format))
At the start: 35 parts, among them J10 Conn_02x05_Odd_Even, J11 DX4R105JJCR1800, J9 Conn_02x12_Odd_Even, SW1 TACTILE_SWITCH, U9 ATmega32U4-AU, Y1 7M-16.000MAAE-T

Commit message: automated commit
Changed lines of the file:
@@
 	1725 1800 1600 1800
 Connection ~ 1725 950
-Text Notes 1500 2575 2    50   ~ 0
+Text Notes 850  2575 0    50   ~ 0
 PLACE CLOSE TO\nTACTILE SWITCH
 $Comp

Commit message: automated commit
Parts:
- removed D?: CM1293A-04SO, SOT-457, symbol custom:CM1293A-04SO
- added D1: CM1293A-04SO, SOT-457, symbol custom:CM1293A-04SO
- gave numbers to parts that had none: 5
Connections:
- net +5V: now also D1.5 (V+)
- net GND: now also SW1.1, SW1.2, D1.2 (V-)
- net RESET: no longer R13.2, U9.13 (~RESET)
- net uC_RSTn: now reaches SW1.3
- net uC_RSTn: now also R13.2, SW1.4, U9.13 (~RESET), D1.1 (CH1)
- net BAT_TEST renamed RESETn
- new net RST_TVS: D1.3 (CH2)
- no-connect marks 6 -> 5
Other:
- note added: "PLACE CLOSE TO\nTACTILE SWITCH PINS"
- note removed: "PLACE CLOSE TO\nTACTILE SWITCH"
- moved on the sheet: C21, D6, F1, J11, R15, R16, R17, R18, R19, SW1

Commit message: automated commit
Connections:
- net RESET is gone; now on net uC_RSTn: J10.10 (Pin_10)
Changed lines of the file:
@@
 	1    0    0    -1
 $EndComp
-Text GLabel 9525 3175 2    50   Input ~ 0
-RESET
-Wire Wire Line
-	9525 3175 9450 3175
+Wire Wire Line
+	10275 3175 9450 3175
 Wire Wire Line
 	4450 2150 4450 2450
@@
 Wire Wire Line
 	1150 1325 1550 1325
+Text Label 10275 3175 2    50   ~ 0
+uC_RSTn
 $EndSCHEMATC

Commit message: automated commit
Parts:
- added BZ?: Buzzer, symbol Device:Buzzer
- added R?: RC0603JR-071KL, 0603, symbol custom:RC0603JR-071KL
Connections:
- new net: BZ?.2 (+), R?.2
- new net VDD_BAT: BZ?.1 (-), R?.1
Changed lines of the file:
@@
 	1    0    0    -1
 $EndComp
-Text GLabel 9525 1475 2    50   Input ~ 0
-PWM_0A
 Text GLabel 9525 1575 2    50   Input ~ 0
 PWM_3A
@@
 Wire Wire Line
 	9525 1575 9450 1575
-Wire Wire Line
-	9450 1475 9525 1475
 Wire Wire Line
 	10000 1375 9450 1375
@@
 Text Label 10275 3175 2    50   ~ 0
 uC_RSTn
+$Comp
+L Device:Buzzer BZ?
+U 1 1 5C57289E
+P 7500 2950
+AR Path="/5C100B31/5C57289E" Ref="BZ?"  Part="1"
+AR Path="/5C3EC885/5C57289E" Ref="BZ?"  Part="1"
+F 0 "BZ?" H 7650 3000 50  0000 L CNN
+F 1 "Buzzer" H 7650 2900 50  0000 L CNN
+F 2 "" V 7475 3050 50  0001 C CNN
+F 3 "~" V 7475 3050 50  0001 C CNN
+	1    7500 2950
+	1    0    0    -1
+$EndComp
+$Comp
+L custom:RC0603JR-071KL R?
+U 1 1 5C58FAC1
+P 7125 2950
+AR Path="/5C58FAC1" Ref="R?"  Part="1"
+AR Path="/5C3EC885/5C58FAC1" Ref="R?"  Part="1"
+F 0 "R?" H 7175 2975 50  0000 L BNN
+F 1 "RC0603JR-071KL" H 7200 2875 50  0001 L BNN
+F 2 "0603" H 7200 2950 50  0001 L BNN
+F 3 "~/datasheets/PYu-RC_Group_51_RoHS_L_10.pdf" H 7065 2960 50  0001 C CNN
+F 4 "1k0" V 7125 2950 50  0000 C CNN "Resistance"
+	1    7125 2950
+	1    0    0    -1
+$EndComp
+Wire Wire Line
+	7400 2850 7350 2850
+Wire Wire Line
+	7350 2850 7350 2750
+Wire Wire Line
+	7350 2750 7125 2750
+Wire Wire Line
+	7125 2750 7125 2800
+Wire Wire Line
+	7125 3100 7125 3150
+Wire Wire Line
+	7125 3150 7350 3150
+Wire Wire Line
+	7350 3150 7350 3050
+Wire Wire Line
+	7350 3050 7400 3050
+$Comp
+L custom:VDD_BAT #PWR?
+U 1 1 5C5F90BF
+P 7125 2625
+F 0 "#PWR?" H 7325 2675 50  0001 C CNN
+F 1 "VDD_BAT" H 6975 2775 50  0000 L BNN
+F 2 "" H 7125 2625 50  0001 C CNN
+F 3 "" H 7125 2625 50  0001 C CNN
+	1    7125 2625
+	1    0    0    -1
+$EndComp
+Wire Wire Line
+	7125 2625 7125 2750
+Connection ~ 7125 2750
+Wire Wire Line
+	9450 1475 9525 1475
+Text GLabel 9525 1475 2    50   Input ~ 0
+PWM_0A
 $EndSCHEMATC

Commit message: automated commit
Parts:
- added JP?: Jumper_3_Bridged12, symbol Jumper:Jumper_3_Bridged12
- added Q?: SSM3K35AMFV, Package_TO_SOT_SMD:SOT-723, symbol custom:SSM3K35AMFV
- added R?: RC0603JR-071KL, 0603, symbol custom:RC0603JR-071KL
- added R?: NP_R_0603, 0603, symbol custom:NP_R_0603
Connections:
- net +1V8: now also J9.7 (Pin_7), J9.8 (Pin_8); no longer J9.5 (Pin_5), J9.6 (Pin_6)
- net +3V3: now also JP?.3 (B)
- net +5V: now also JP?.1 (A), R?.2; no longer C10.1, C11.1, C12.1, C13.1, C14.1, C15.1, C9.1, D1.5 (V+), D2.5 (V+), D3.5 (V+), D4.5 (V+), D5.5 (V+), D6.5 (V+), J10.1 (Pin_1), L1.1, R13.1, U9.14 (VCC), U9.2 (UVCC), U9.34 (VCC)
- net GND: now also J9.5 (Pin_5), J9.6 (Pin_6), J9.9 (Pin_9), Q?.2 (S), R?.2; no longer J9.7 (Pin_7), J9.8 (Pin_8)
- net PWM_0A: no longer J9.12 (Pin_12), U9.12 (PB7)
- net PWM_3A: now also J9.11 (Pin_11); no longer J9.14 (Pin_14)
- net PWM_4A: now also J9.12 (Pin_12); no longer J9.9 (Pin_9)
- net PWM_4D: now also J9.14 (Pin_14); no longer J9.11 (Pin_11)
- net at BZ?.2 (+), R?.2: now also Q?.3 (D)
- new net: Q?.1 (G), R?.1, U9.12 (PB7)
- new net: D6.5 (V+), R?.1
- new net VDD_uC: C10.1, C11.1, C12.1, C13.1, C14.1, C15.1, C9.1, D1.5 (V+), D2.5 (V+), D3.5 (V+), D4.5 (V+), D5.5 (V+), J10.1 (Pin_1), JP?.2 (C), L1.1, R13.1, U9.14 (VCC), U9.2 (UVCC), U9.34 (VCC)
Other:
- note added: "PWM_0A"
- moved on the sheet: BZ?, C10, C11, C12, C13, C14, C15, C16, C17, C18, C19, C20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

Commit message: automated commit
Parts:
- added TP34, TP35, TP36, TP37, TP38, TP39, TP40, TP41, TP42, TP43, TP44, TP45, TP46, TP47, TP48, TP49, TP50, TP51: PTH_0.5_mm, symbol custom:PTH_0.5_mm
- gave numbers to parts that had none: 6
Connections:
- net I2C_SCL: now also TP45.1
- net I2C_SDA: now also TP47.1
- net JTAG_TCK: now also TP43.1
- net JTAG_TDI: now also TP37.1
- net JTAG_TDO: now also TP39.1
- net JTAG_TMS: now also TP41.1
- net PWM_3A: now also TP44.1
- net PWM_4A: now also TP46.1
- net PWM_4D: now also TP48.1
- net RESETn: now also TP50.1
- net SPI_MISO: now also TP42.1
- net SPI_MOSI: now also TP40.1
- net SPI_SCK: now also TP38.1
- net SPI_SSn: now also TP36.1
- net USART_RX: now also TP49.1
- net USART_TX: now also TP51.1
- net VBUS: now also TP35.1
- net VDD_uC: now also TP34.1
- net MOTOR_L renamed R_MOTOR
- net MOTOR_R renamed L_MOTOR
Other:
- moved on the sheet: J10, J9, JP2

Commit message: automated commit
Parts:
- removed C9: ‎CL21A475KLCLQNC‎, Capacitor_SMD:C_0805_2012Metric, symbol custom:‎CL21A475KLCLQNC‎
- added C31: CL10B105KA8NNNC, Capacitor_SMD:C_0603_1608Metric, symbol custom:CL10B105KA8NNNC
- added C9: CL10B103KB8SFNC, Capacitor_SMD:C_0603_1608Metric, symbol custom:CL10B103KB8SFNC
- BZ1: footprint (none) -> custom:0.5_IN_BUZZER
- D1, D2, D3, D4, D5, D6: footprint SOT-457 -> custom:SOT-457
- J10: footprint (none) -> Connector_PinHeader_2.54mm:PinHeader_2x05_P2.54mm_Vertical
- J9: footprint (none) -> Connector_PinHeader_2.54mm:PinHeader_2x12_P2.54mm_Vertical
- JP2: footprint (none) -> Connector_PinHeader_2.54mm:PinHeader_1x03_P2.54mm_Vertical
- L1, L2: footprint 0603 -> Inductor_SMD:L_0603_1608Metric
- R13, R14, R15, R16, R17, R34, R35: footprint 0603 -> Resistor_SMD:R_0603_1608Metric
- R36: footprint 0603 -> custom:NP_0603
- TP34, TP35, TP36, TP37, TP38, TP39, TP40, TP41, TP42, TP43, TP44, TP45, TP46, TP47, TP48, TP49, TP50, TP51: footprint (none) -> TestPoint:TestPoint_THTPad_D1.0mm_Drill0.5mm
- Y1: footprint (none) -> Crystal:Crystal_SMD_3225-4Pin_3.2x2.5mm
Connections:
- net GND: now also C31.2, C9.2
- net VDD_uC: now also C9.1; no longer C14.1, C15.1
- net uC_AVCC: now reaches L1.2, U9.24 (AVCC), U9.44 (AVCC)
- net uC_AVCC: now also C14.1, C15.1, C31.1
Other:
- moved on the sheet: C10, C11, C12, C13, C14, C15, D2, D3, D4, D5, JP2, TP34

Commit message: automated commit
Parts:
- F1: footprint 1812 -> custom:MF-MSMF050-2
- J11: footprint (none) -> custom:DX4R105JJCR1800‎_MICRO_USB_B_CONNECTOR
Changed lines of the file:
@@
 F 0 "J11" H 1125 5525 50  0000 L BNN
 F 1 "DX4R105JJCR1800" H 1025 4275 50  0001 L BNN
-F 2 "" H 1475 5025 50  0001 C CNN
+F 2 "custom:DX4R105JJCR1800‎_MICRO_USB_B_CONNECTOR" H 1475 5025 50  0001 C CNN
 F 3 "SJ113218.pdf" H 1475 5025 50  0001 L BNN
 F 4 "Micro_USB_B" H 1125 5425 50  0000 L BNN "Description"
@@
 Text Label 2975 5175 2    50   ~ 0
 M_USB_IC-
-$Comp
-L custom:MF-MSMF050-2 F1
-U 1 1 5C440655
-P 1875 4725
-F 0 "F1" V 1825 4600 50  0000 L BNN
-F 1 "MF-MSMF050-2" H 1775 4200 50  0001 L BNN
-F 2 "1812" H 1775 4275 50  0001 L BNN
-F 3 "~/datasheets/mfmsmf.pdf" H 1775 4100 50  0001 L BNN
-F 4 "0.5 A" V 1975 4700 50  0000 L BNN "Rating"
-	1    1875 4725
-	0    1    1    0
-$EndComp
 Wire Wire Line
 	2025 4725 2275 4725
@@
 uC_AVCC
 Connection ~ 5150 1200
+$Comp
+L custom:MF-MSMF050-2 F1
+U 1 1 5C5A71F2
+P 1875 4725
+F 0 "F1" V 1825 4625 50  0000 L BNN
+F 1 "MF-MSMF050-2" H 1775 4200 50  0001 L BNN
+F 2 "custom:MF-MSMF050-2" H 1775 4275 50  0001 L BNN
+F 3 "/home/dj/datasheets/mfmsmf.pdf" H 1775 4100 50  0001 L BNN
+F 4 "0.5 A" V 2025 4625 50  0000 L BNN "Rating"
+	1    1875 4725
+	0    1    1    0
+$EndComp
 $EndSCHEMATC
