File: nu.ai_motor_controller/nu.ai_motor_controller.sch (KiCad schematic (older format))
At the start: 11 parts

Commit message: cleaned up and renamed project files. Changed custom library management scheme. It now resides in my homedir as a seperate git project, and is pointed to in kicad's symbol library manager
Parts:
- J? (x8): symbol nu-rescue:PTH_1_mm-custom -> custom:PTH_1_mm
- J? (x2): symbol nu-rescue:PTH_3_mm-custom -> custom:PTH_3_mm
Changed lines of the file:
@@
 EESchema Schematic File Version 4
-LIBS:nu-cache
+LIBS:nu.ai_motor_controller-cache
 EELAYER 26 0
 EELAYER END
@@
 $EndComp
 $Comp
-L nu-rescue:PTH_3_mm-custom J?
+L custom:PTH_3_mm J?
 U 1 1 5C162A1D
 P 1250 4200
@@
 $EndComp
 $Comp
-L nu-rescue:PTH_3_mm-custom J?
+L custom:PTH_3_mm J?
 U 1 1 5C162B98
 P 1250 3950
@@
 	-1   0    0    -1
 $EndComp
-Wire Wire Line
-	1400 3950 1850 3950
 Wire Wire Line
 	1400 4200 1750 4200
@@
 	9950 2700 10100 2700
 $Comp
-L nu-rescue:PTH_1_mm-custom J?
+L custom:PTH_1_mm J?
 U 1 1 5C14202A
 P 10550 2200
@@
 $EndComp
 $Comp
-L nu-rescue:PTH_1_mm-custom J?
+L custom:PTH_1_mm J?
 U 1 1 5C1420FB
 P 10550 2400
@@
 $EndComp
 $Comp
-L nu-rescue:PTH_1_mm-custom J?
+L custom:PTH_1_mm J?
 U 1 1 5C142269
 P 10550 2700
@@
 $EndComp
 $Comp
-L nu-rescue:PTH_1_mm-custom J?
+L custom:PTH_1_mm J?
 U 1 1 5C14226F
 P 10550 2900
@@
 $EndComp
 $Comp
-L nu-rescue:PTH_1_mm-custom J?
+L custom:PTH_1_mm J?
 U 1 1 5C1426F8
 P 10550 3200
@@
 $EndComp
 $Comp
-L nu-rescue:PTH_1_mm-custom J?
+L custom:PTH_1_mm J?
 U 1 1 5C1426FE
 P 10550 3400
@@
 $EndComp
 $Comp
-L nu-rescue:PTH_1_mm-custom J?
+L custom:PTH_1_mm J?
 U 1 1 5C142704
 P 10550 3700
@@
 $EndComp
 $Comp
-L nu-rescue:PTH_1_mm-custom J?
+L custom:PTH_1_mm J?
 U 1 1 5C14270A
 P 10550 3900
@@
 F1 "microcontroller.sch" 50
 $EndSheet
+Wire Wire Line
+	1400 3950 1850 3950
 $EndSCHEMATC

Commit message: automated commit
Changed lines of the file:
@@
 $EndDescr
 $Sheet
-S 4350 2200 1300 1000
+S 5500 2250 1300 1000
 U 5C100B31
 F0 "power" 50
@@
 ADD 2 mm STRAIN RELIEF HOLES
 $Sheet
-S 2050 2025 1300 1175
+S 3200 2075 1300 1175
 U 5C3EC885
 F0 "microcontroller" 50

Commit message: automated commit
Changed lines of the file:
@@
 $EndDescr
 $Sheet
-S 5500 2250 1300 1000
+S 1275 1125 1300 1000
 U 5C100B31
 F0 "power" 50
@@
 F0 "driver" 50
 F1 "driver.sch" 50
-F2 "IN_1_A" I L 9050 2700 50
-F3 "IN_2_A" I L 9050 2800 50
-F4 "IN_2_B" I L 9050 3000 50
-F5 "IN_1_C" I L 9050 3100 50
-F6 "IN_2_C" I L 9050 3200 50
-F7 "IN_1_D" I L 9050 3300 50
-F8 "IN_2_D" I L 9050 3400 50
-F9 "OUT_1_A" O R 9950 2700 50
-F10 "OUT_2_A" O R 9950 2800 50
-F11 "OUT_1_B" O R 9950 2900 50
-F12 "OUT_2_B" O R 9950 3000 50
-F13 "OUT_1_C" O R 9950 3100 50
-F14 "OUT_2_C" O R 9950 3200 50
-F15 "OUT_1_D" O R 9950 3300 50
-F16 "OUT_2_D" O R 9950 3400 50
-F17 "IN_1_B" I L 9050 2900 50
+F2 "OUT_1_A" O R 9950 2700 50
+F3 "OUT_2_A" O R 9950 2800 50
+F4 "OUT_1_B" O R 9950 2900 50
+F5 "OUT_2_B" O R 9950 3000 50
+F6 "OUT_1_C" O R 9950 3100 50
+F7 "OUT_2_C" O R 9950 3200 50
+F8 "OUT_1_D" O R 9950 3300 50
+F9 "OUT_2_D" O R 9950 3400 50
+F10 "IN_1_L" I L 9050 2700 50
+F11 "IN_2_L" I L 9050 2800 50
+F12 "IN_1_R" I L 9050 3000 50
+F13 "IN_2_R" I L 9050 3100 50
 $EndSheet
 Wire Wire Line
@@
 ADD 2 mm STRAIN RELIEF HOLES
 $Sheet
-S 3200 2075 1300 1175
+S 5975 2250 900  1375
 U 5C3EC885
 F0 "microcontroller" 50

Commit message: automated commit
Parts:
- added R? (x4): RC0603JR-071KL, 0603, symbol custom:RC0603JR-071KL
Connections:
- net labels added: GND
- wire segments 28 -> 49
Changed lines of the file:
@@
 ADD 2 mm STRAIN RELIEF HOLES
 $Sheet
-S 5975 2250 900  1375
+S 5075 2250 900  1375
 U 5C3EC885
 F0 "microcontroller" 50
 F1 "microcontroller.sch" 50
+F2 "MOTOR_L" O R 5975 2375 50
+F3 "MOTOR_R" O R 5975 2925 50
+F4 "L_DIR" O R 5975 2500 50
+F5 "R_DIR" O R 5975 3050 50
 $EndSheet
 Wire Wire Line
 	1400 3950 1850 3950
+$Comp
+L custom:RC0603JR-071KL R?
+U 1 1 5C4509EC
+P 8175 3350
+F 0 "R?" V 8125 3300 50  0000 L BNN
+F 1 "RC0603JR-071KL" H 8250 3275 50  0001 L BNN
+F 2 "0603" H 8250 3350 50  0001 L BNN
+F 3 "~/datasheets/PYu-RC_Group_51_RoHS_L_10.pdf" H 8115 3360 50  0001 C CNN
+F 4 "1k" V 8200 3300 50  0000 L BNN "Resistance"
+	1    8175 3350
+	1    0    0    -1
+$EndComp
+$Comp
+L custom:RC0603JR-071KL R?
+U 1 1 5C450BAD
+P 8375 3350
+F 0 "R?" V 8325 3300 50  0000 L BNN
+F 1 "RC0603JR-071KL" H 8450 3275 50  0001 L BNN
+F 2 "0603" H 8450 3350 50  0001 L BNN
+F 3 "~/datasheets/PYu-RC_Group_51_RoHS_L_10.pdf" H 8315 3360 50  0001 C CNN
+F 4 "1k" V 8400 3300 50  0000 L BNN "Resistance"
+	1    8375 3350
+	1    0    0    -1
+$EndComp
+$Comp
+L custom:RC0603JR-071KL R?
+U 1 1 5C450C05
+P 8575 3350
+F 0 "R?" V 8525 3300 50  0000 L BNN
+F 1 "RC0603JR-071KL" H 8650 3275 50  0001 L BNN
+F 2 "0603" H 8650 3350 50  0001 L BNN
+F 3 "~/datasheets/PYu-RC_Group_51_RoHS_L_10.pdf" H 8515 3360 50  0001 C CNN
+F 4 "1k" V 8600 3300 50  0000 L BNN "Resistance"
+	1    8575 3350
+	1    0    0    -1
+$EndComp
+$Comp
+L custom:RC0603JR-071KL R?
+U 1 1 5C450C5F
+P 8775 3350
+F 0 "R?" V 8725 3300 50  0000 L BNN
+F 1 "RC0603JR-071KL" H 8850 3275 50  0001 L BNN
+F 2 "0603" H 8850 3350 50  0001 L BNN
+F 3 "~/datasheets/PYu-RC_Group_51_RoHS_L_10.pdf" H 8715 3360 50  0001 C CNN
+F 4 "1k" V 8800 3300 50  0000 L BNN "Resistance"
+	1    8775 3350
+	1    0    0    -1
+$EndComp
+$Comp
+L power:GND #PWR?
+U 1 1 5C4512F4
+P 8475 3600
+F 0 "#PWR?" H 8475 3350 50  0001 C CNN
+F 1 "GND" H 8475 3450 50  0000 C CNN
+F 2 "" H 8475 3600 50  0001 C CNN
+F 3 "" H 8475 3600 50  0001 C CNN
+	1    8475 3600
+	1    0    0    -1
+$EndComp
+Wire Wire Line
+	8775 3500 8775 3550
+Wire Wire Line
+	8775 3550 8575 3550
+Wire Wire Line
+	8175 3550 8175 3500
+Wire Wire Line
+	8475 3550 8475 3600
+Wire Wire Line
+	8375 3500 8375 3550
+Connection ~ 8375 3550
+Wire Wire Line
+	8375 3550 8175 3550
+Wire Wire Line
+	8575 3500 8575 3550
+Connection ~ 8575 3550
+Wire Wire Line
+	8575 3550 8475 3550
+Wire Wire Line
+	8775 3200 8775 3100
+Wire Wire Line
+	8775 3100 9050 3100
+Wire Wire Line
+	9050 3000 8575 3000
+Wire Wire Line
+	8575 3000 8575 3200
+Wire Wire Line
+	8375 3200 8375 2800
+Wire Wire Line
+	8375 2800 9050 2800
+Wire Wire Line
+	9050 2700 8175 2700
+Wire Wire Line
+	8175 2700 8175 3200
+Wire Wire Line
+	8175 2700 7450 2700
+Connection ~ 8175 2700
+Wire Wire Line
+	8375 2800 7450 2800
+Connection ~ 8375 2800
+Wire Wire Line
+	8575 3000 7450 3000
+Connection ~ 8575 3000
+Wire Wire Line
+	8775 3100 7450 3100
+Connection ~ 8775 3100
+Connection ~ 8475 3550
+Wire Wire Line
+	8475 3550 8375 3550
 $EndSCHEMATC

Commit message: automated commit
Parts:
- added U? (x2): SGM3157YC6, Package_TO_SOT_SMD:SOT-23-6, symbol custom:SGM3157YC6
Connections:
- net labels added: +5V
- wire segments 49 -> 65
Other:
- moved on the sheet: J?

Commit message: automated commit
Parts:
- added R? (x4): RC0603JR-071KL, 0603, symbol custom:RC0603JR-071KL
Connections:
- wire segments 65 -> 78
Other:
- moved on the sheet: R?, U?

Commit message: automated commit
Parts:
- removed J?: Screw_Terminal_01x02, symbol Connector:Screw_Terminal_01x02
- removed J? (x2): PTH_3_mm, symbol custom:PTH_3_mm
Connections:
- wire segments 78 -> 74
Other:
- note removed: "INDICATE POS AND NEG\nON SILKSCREEN"
- note removed: "XT60 MALE CABLE ASSEMBLY\nADD 4 mm STRAIN RELIEF HOLES"
Changed lines of the file:
@@
 F1 "power.sch" 50
 $EndSheet
-$Comp
-L Connector:Screw_Terminal_01x02 J?
-U 1 1 5C0FEC80
-P 9150 1250
-F 0 "J?" H 9150 1350 50  0000 C CNN
-F 1 "Screw_Terminal_01x02" H 9150 1050 50  0000 C CNN
-F 2 "" H 9150 1250 50  0001 C CNN
-F 3 "~" H 9150 1250 50  0001 C CNN
-	1    9150 1250
-	1    0    0    -1
-$EndComp
-$Comp
-L custom:PTH_3_mm J?
-U 1 1 5C162A1D
-P 1250 4200
-F 0 "J?" H 1400 4200 50  0000 C CNN
-F 1 "PTH_3_mm" H 1250 4100 50  0000 C CNN
-F 2 "" H 1250 4200 50  0001 C CNN
-F 3 "" H 1250 4200 50  0001 C CNN
-	1    1250 4200
-	-1   0    0    -1
-$EndComp
-$Comp
-L custom:PTH_3_mm J?
-U 1 1 5C162B98
-P 1250 3950
-F 0 "J?" H 1400 3950 50  0000 C CNN
-F 1 "PTH_3_mm" H 1250 3850 50  0000 C CNN
-F 2 "" H 1250 3950 50  0001 C CNN
-F 3 "" H 1250 3950 50  0001 C CNN
-	1    1250 3950
-	-1   0    0    -1
-$EndComp
-Wire Wire Line
-	1400 4200 1750 4200
-Text Notes 9500 1000 2    67   ~ 0
-INDICATE POS AND NEG\nON SILKSCREEN
-Text Notes 800  4600 0    67   ~ 0
-XT60 MALE CABLE ASSEMBLY\nADD 4 mm STRAIN RELIEF HOLES
-Wire Wire Line
-	8950 1250 8200 1250
-Wire Wire Line
-	8950 1350 8200 1350
 $Sheet
 S 9050 2600 900  900
@@
 F5 "R_DIR" O R 5575 3400 50
 $EndSheet
-Wire Wire Line
-	1400 3950 1850 3950
 $Comp
 L custom:RC0603JR-071KL R?

Commit message: automated commit
Changed lines of the file:
@@
 $Descr A4 11693 8268
 encoding utf-8
-Sheet 1 4
+Sheet 1 5
 Title ""
 Date ""
@@
 Wire Wire Line
 	6000 2800 5575 2800
+$Sheet
+S 1525 3325 1250 1025
+U 5C5AE643
+F0 "battery" 50
+F1 "battery.sch" 50
+$EndSheet
 $EndSCHEMATC
