File: nu.ai_motor_controller/nu.ai_motor_controller.sch (KiCad schematic (older format))
At the start: 18 parts

Commit message: automated commit
Parts:
- removed R? (x8): RC0603JR-071KL, 0603, symbol custom:RC0603JR-071KL
- added R? (x8): RC0603JR-071KL, 0603, symbol custom:RC0603JR-071KL
Connections:
- net GND: now also R?.2, R?.2, R?.2, R?.2, R?.2, R?.2, R?.2, R?.2
- net driver/IN_1_L: now also R?.1
- net driver/IN_1_R: now also R?.1
- net driver/IN_2_L: now also R?.1
- net driver/IN_2_R: now also R?.1
- net microcontroller/L_DIR: now also R?.1
- net microcontroller/MOTOR_L: now also R?.1
- net microcontroller/MOTOR_R: now also R?.1
- net microcontroller/R_DIR: now also R?.1
Changed lines of the file:
@@
 $EndSheet
-$Comp
-L custom:RC0603JR-071KL R?
-U 1 1 5C4509EC
-P 8175 3625
-F 0 "R?" V 8125 3575 50  0000 L BNN
-F 1 "RC0603JR-071KL" H 8250 3550 50  0001 L BNN
-F 2 "0603" H 8250 3625 50  0001 L BNN
-F 3 "~/datasheets/PYu-RC_Group_51_RoHS_L_10.pdf" H 8115 3635 50  0001 C CNN
-F 4 "1k" V 8200 3575 50  0000 L BNN "Resistance"
-	1    8175 3625
-	1    0    0    -1
-$EndComp
-$Comp
-L custom:RC0603JR-071KL R?
-U 1 1 5C450BAD
-P 8375 3625
-F 0 "R?" V 8325 3575 50  0000 L BNN
-F 1 "RC0603JR-071KL" H 8450 3550 50  0001 L BNN
-F 2 "0603" H 8450 3625 50  0001 L BNN
-F 3 "~/datasheets/PYu-RC_Group_51_RoHS_L_10.pdf" H 8315 3635 50  0001 C CNN
-F 4 "1k" V 8400 3575 50  0000 L BNN "Resistance"
-	1    8375 3625
-	1    0    0    -1
-$EndComp
-$Comp
-L custom:RC0603JR-071KL R?
-U 1 1 5C450C05
-P 8575 3625
-F 0 "R?" V 8525 3575 50  0000 L BNN
-F 1 "RC0603JR-071KL" H 8650 3550 50  0001 L BNN
-F 2 "0603" H 8650 3625 50  0001 L BNN
-F 3 "~/datasheets/PYu-RC_Group_51_RoHS_L_10.pdf" H 8515 3635 50  0001 C CNN
-F 4 "1k" V 8600 3575 50  0000 L BNN "Resistance"
-	1    8575 3625
-	1    0    0    -1
-$EndComp
-$Comp
-L custom:RC0603JR-071KL R?
-U 1 1 5C450C5F
-P 8775 3625
-F 0 "R?" V 8725 3575 50  0000 L BNN
-F 1 "RC0603JR-071KL" H 8850 3550 50  0001 L BNN
-F 2 "0603" H 8850 3625 50  0001 L BNN
-F 3 "~/datasheets/PYu-RC_Group_51_RoHS_L_10.pdf" H 8715 3635 50  0001 C CNN
-F 4 "1k" V 8800 3575 50  0000 L BNN "Resistance"
-	1    8775 3625
-	1    0    0    -1
-$EndComp
 $Comp
 L power:GND #PWR?
@@
 	5575 3400 6600 3400
 $Comp
-L custom:RC0603JR-071KL R?
-U 1 1 5C59C0EF
-P 6000 3725
-F 0 "R?" V 5950 3675 50  0000 L BNN
-F 1 "RC0603JR-071KL" H 6075 3650 50  0001 L BNN
-F 2 "0603" H 6075 3725 50  0001 L BNN
-F 3 "~/datasheets/PYu-RC_Group_51_RoHS_L_10.pdf" H 5940 3735 50  0001 C CNN
-F 4 "1k" V 6025 3675 50  0000 L BNN "Resistance"
-	1    6000 3725
-	1    0    0    -1
-$EndComp
-$Comp
-L custom:RC0603JR-071KL R?
-U 1 1 5C59C0F7
-P 6200 3725
-F 0 "R?" V 6150 3675 50  0000 L BNN
-F 1 "RC0603JR-071KL" H 6275 3650 50  0001 L BNN
-F 2 "0603" H 6275 3725 50  0001 L BNN
-F 3 "~/datasheets/PYu-RC_Group_51_RoHS_L_10.pdf" H 6140 3735 50  0001 C CNN
-F 4 "1k" V 6225 3675 50  0000 L BNN "Resistance"
-	1    6200 3725
-	1    0    0    -1
-$EndComp
-$Comp
-L custom:RC0603JR-071KL R?
-U 1 1 5C59C0FF
-P 6400 3725
-F 0 "R?" V 6350 3675 50  0000 L BNN
-F 1 "RC0603JR-071KL" H 6475 3650 50  0001 L BNN
-F 2 "0603" H 6475 3725 50  0001 L BNN
-F 3 "~/datasheets/PYu-RC_Group_51_RoHS_L_10.pdf" H 6340 3735 50  0001 C CNN
-F 4 "1k" V 6425 3675 50  0000 L BNN "Resistance"
-	1    6400 3725
-	1    0    0    -1
-$EndComp
-$Comp
-L custom:RC0603JR-071KL R?
-U 1 1 5C59C107
-P 6600 3725
-F 0 "R?" V 6550 3675 50  0000 L BNN
-F 1 "RC0603JR-071KL" H 6675 3650 50  0001 L BNN
-F 2 "0603" H 6675 3725 50  0001 L BNN
-F 3 "~/datasheets/PYu-RC_Group_51_RoHS_L_10.pdf" H 6540 3735 50  0001 C CNN
-F 4 "1k" V 6625 3675 50  0000 L BNN "Resistance"
-	1    6600 3725
-	1    0    0    -1
-$EndComp
-$Comp
 L power:GND #PWR?
 U 1 1 5C59C10E
@@
 F1 "battery.sch" 50
 $EndSheet
+$Comp
+L custom:RC0603JR-071KL R?
+U 1 1 5C519E2B
+P 6000 3725
+F 0 "R?" V 5950 3675 50  0000 L BNN
+F 1 "RC0603JR-071KL" H 6075 3650 50  0001 L BNN
+F 2 "0603" H 6075 3725 50  0001 L BNN
+F 3 "~/datasheets/PYu-RC_Group_51_RoHS_L_10.pdf" H 5940 3735 50  0001 C CNN
+F 4 "1k0" V 6000 3725 50  0000 C CNN "Resistance"
+	1    6000 3725
+	1    0    0    -1
+$EndComp
+$Comp
+L custom:RC0603JR-071KL R?
+U 1 1 5C51DF38
+P 6200 3725
+F 0 "R?" V 6150 3675 50  0000 L BNN
+F 1 "RC0603JR-071KL" H 6275 3650 50  0001 L BNN
+F 2 "0603" H 6275 3725 50  0001 L BNN
+F 3 "~/datasheets/PYu-RC_Group_51_RoHS_L_10.pdf" H 6140 3735 50  0001 C CNN
+F 4 "1k0" V 6200 3725 50  0000 C CNN "Resistance"
+	1    6200 3725
+	1    0    0    -1
+$EndComp
+$Comp
+L custom:RC0603JR-071KL R?
+U 1 1 5C51DF72
+P 6400 3725
+F 0 "R?" V 6350 3675 50  0000 L BNN
+F 1 "RC0603JR-071KL" H 6475 3650 50  0001 L BNN
+F 2 "0603" H 6475 3725 50  0001 L BNN
+F 3 "~/datasheets/PYu-RC_Group_51_RoHS_L_10.pdf" H 6340 3735 50  0001 C CNN
+F 4 "1k0" V 6400 3725 50  0000 C CNN "Resistance"
+	1    6400 3725
+	1    0    0    -1
+$EndComp
+$Comp
+L custom:RC0603JR-071KL R?
+U 1 1 5C51DFB2
+P 6600 3725
+F 0 "R?" V 6550 3675 50  0000 L BNN
+F 1 "RC0603JR-071KL" H 6675 3650 50  0001 L BNN
+F 2 "0603" H 6675 3725 50  0001 L BNN
+F 3 "~/datasheets/PYu-RC_Group_51_RoHS_L_10.pdf" H 6540 3735 50  0001 C CNN
+F 4 "1k0" V 6600 3725 50  0000 C CNN "Resistance"
+	1    6600 3725
+	1    0    0    -1
+$EndComp
+$Comp
+L custom:RC0603JR-071KL R?
+U 1 1 5C51E1B2
+P 8175 3625
+F 0 "R?" V 8125 3575 50  0000 L BNN
+F 1 "RC0603JR-071KL" H 8250 3550 50  0001 L BNN
+F 2 "0603" H 8250 3625 50  0001 L BNN
+F 3 "~/datasheets/PYu-RC_Group_51_RoHS_L_10.pdf" H 8115 3635 50  0001 C CNN
+F 4 "1k0" V 8175 3625 50  0000 C CNN "Resistance"
+	1    8175 3625
+	1    0    0    -1
+$EndComp
+$Comp
+L custom:RC0603JR-071KL R?
+U 1 1 5C51E1BA
+P 8375 3625
+F 0 "R?" V 8325 3575 50  0000 L BNN
+F 1 "RC0603JR-071KL" H 8450 3550 50  0001 L BNN
+F 2 "0603" H 8450 3625 50  0001 L BNN
+F 3 "~/datasheets/PYu-RC_Group_51_RoHS_L_10.pdf" H 8315 3635 50  0001 C CNN
+F 4 "1k0" V 8375 3625 50  0000 C CNN "Resistance"
+	1    8375 3625
+	1    0    0    -1
+$EndComp
+$Comp
+L custom:RC0603JR-071KL R?
+U 1 1 5C51E1C2
+P 8575 3625
+F 0 "R?" V 8525 3575 50  0000 L BNN
+F 1 "RC0603JR-071KL" H 8650 3550 50  0001 L BNN
+F 2 "0603" H 8650 3625 50  0001 L BNN
+F 3 "~/datasheets/PYu-RC_Group_51_RoHS_L_10.pdf" H 8515 3635 50  0001 C CNN
+F 4 "1k0" V 8575 3625 50  0000 C CNN "Resistance"
+	1    8575 3625
+	1    0    0    -1
+$EndComp
+$Comp
+L custom:RC0603JR-071KL R?
+U 1 1 5C51E1CA
+P 8775 3625
+F 0 "R?" V 8725 3575 50  0000 L BNN
+F 1 "RC0603JR-071KL" H 8850 3550 50  0001 L BNN
+F 2 "0603" H 8850 3625 50  0001 L BNN
+F 3 "~/datasheets/PYu-RC_Group_51_RoHS_L_10.pdf" H 8715 3635 50  0001 C CNN
+F 4 "1k0" V 8775 3625 50  0000 C CNN "Resistance"
+	1    8775 3625
+	1    0    0    -1
+$EndComp
 $EndSCHEMATC

Commit message: automated commit
Parts:
- gave numbers to parts that had none: 18
Other:
- note added: "add mounting holes"
- moved on the sheet: J1, J2, J3, J4, J5, J6, J7, J8, R1, R2, R3, R4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

Commit message: automated commit
Other:
- note added: "add buzzer"
- note added: "consider power cutoff (LED high side switch?)"
Changed lines of the file:
@@
 Text Notes 2900 1050 0    50   ~ 0
 add mounting holes
+Text Notes 3050 1350 0    50   ~ 0
+add buzzer
+Text Notes 2500 1600 0    50   ~ 0
+consider power cutoff (LED high side switch?)
 $EndSCHEMATC

Commit message: automated commit
Other:
- note added: "allow uC power to be switched between 5V and 3.3V"
- note removed: "consider power cutoff (LED high side switch?)"
Changed lines of the file:
@@
 Wire Wire Line
 	7625 4000 7525 4000
-$Comp
-L custom:SGM3157YC6 U1
-U 1 1 5C556725
-P 6400 2925
-F 0 "U1" H 6150 3150 50  0000 L BNN
-F 1 "SGM3157YC6" H 6000 2575 50  0001 L BNN
-F 2 "Package_TO_SOT_SMD:SOT-23-6" H 6000 2475 50  0001 L BNN
-F 3 "~/datahseets/SGM3157YC6.pdf" H 6000 2375 50  0001 L BNN
-	1    6400 2925
-	1    0    0    -1
-$EndComp
-$Comp
-L custom:SGM3157YC6 U2
-U 1 1 5C55A5EE
-P 6400 3425
-F 0 "U2" H 6150 3650 50  0000 L BNN
-F 1 "SGM3157YC6" H 6000 3075 50  0001 L BNN
-F 2 "Package_TO_SOT_SMD:SOT-23-6" H 6000 2975 50  0001 L BNN
-F 3 "~/datahseets/SGM3157YC6.pdf" H 6000 2875 50  0001 L BNN
-	1    6400 3425
-	1    0    0    -1
-$EndComp
 Connection ~ 7725 3275
 Connection ~ 7925 3375
@@
 Text Notes 3050 1350 0    50   ~ 0
 add buzzer
-Text Notes 2500 1600 0    50   ~ 0
-consider power cutoff (LED high side switch?)
+Text Notes 2375 1575 0    50   ~ 0
+allow uC power to be switched between 5V and 3.3V
+$Comp
+L custom:SGM3157YC6 U1
+U 1 1 5CA760BE
+P 6400 2925
+F 0 "U1" H 6150 3150 50  0000 L BNN
+F 1 "SGM3157YC6" H 6150 2750 50  0000 L BNN
+F 2 "Package_TO_SOT_SMD:SOT-23-6" H 6150 2625 50  0001 L BNN
+F 3 "/home/dj/datasheets/SGM3157YC6.pdf" H 6150 2525 50  0001 L BNN
+	1    6400 2925
+	1    0    0    -1
+$EndComp
+$Comp
+L custom:SGM3157YC6 U2
+U 1 1 5CA7613D
+P 6400 3425
+F 0 "U2" H 6150 3650 50  0000 L BNN
+F 1 "SGM3157YC6" H 6150 3250 50  0000 L BNN
+F 2 "Package_TO_SOT_SMD:SOT-23-6" H 6150 3125 50  0001 L BNN
+F 3 "/home/dj/datasheets/SGM3157YC6.pdf" H 6150 3025 50  0001 L BNN
+	1    6400 3425
+	1    0    0    -1
+$EndComp
 $EndSCHEMATC

Commit message: automated commit
Parts:
- removed R1, R2, R3, R4, R5, R6, R7, R8: RC0603JR-071KL, 0603, symbol custom:RC0603JR-071KL
- removed U1, U2: SGM3157YC6, Package_TO_SOT_SMD:SOT-23-6, symbol custom:SGM3157YC6
Other:
- note removed: "add buzzer"
- note removed: "allow uC power to be switched between 5V and 3.3V"

Commit message: automated commit
Parts:
- removed J1, J2, J3, J4, J5, J6, J7, J8: PTH_1_mm, symbol custom:PTH_1_mm
Other:
- note added: "NOTES:"
- note added: "TABLE OF CONTENTS:\n1. BATTERY\n2. POWER\n3. MICROCONTROLLER\n4. MOTOR DRIVER"
- note added: "TODO:\nADD MOUNTING HOLES"
- note removed: "ADD 2 mm STRAIN RELIEF HOLES"
- note removed: "add mounting holes"
Changed lines of the file:
@@
 $EndDescr
 $Sheet
-S 2675 2950 675  350
+S 9825 1400 675  350
 U 5C100B31
 F0 "power" 50
@@
 $EndSheet
 $Sheet
-S 8200 2675 900  900
+S 9825 2750 675  350
 U 5C10107F
 F0 "driver" 50
 F1 "driver.sch" 50
-F2 "OUT_1_A" O R 9100 2775 50
-F3 "OUT_2_A" O R 9100 2875 50
-F4 "OUT_1_B" O R 9100 2975 50
-F5 "OUT_2_B" O R 9100 3075 50
-F6 "OUT_1_C" O R 9100 3175 50
-F7 "OUT_2_C" O R 9100 3275 50
-F8 "OUT_1_D" O R 9100 3375 50
-F9 "OUT_2_D" O R 9100 3475 50
-F10 "IN_1_L" I L 8200 2775 50
-F11 "IN_2_L" I L 8200 2875 50
-F12 "IN_1_R" I L 8200 3275 50
-F13 "IN_2_R" I L 8200 3375 50
 $EndSheet
-Wire Wire Line
-	9100 3475 9250 3475
-Wire Wire Line
-	9100 2775 9250 2775
-$Comp
-L custom:PTH_1_mm J1
-U 1 1 5C14202A
-P 9700 2175
-F 0 "J1" H 9800 2175 50  0000 C CNN
-F 1 "PTH_1_mm" H 9700 2075 50  0000 C CNN
-F 2 "" H 9700 2175 50  0001 C CNN
-F 3 "" H 9700 2175 50  0001 C CNN
-	1    9700 2175
-	1    0    0    -1
-$EndComp
-$Comp
-L custom:PTH_1_mm J2
-U 1 1 5C1420FB
-P 9700 2375
-F 0 "J2" H 9800 2375 50  0000 C CNN
-F 1 "PTH_1_mm" H 9700 2275 50  0000 C CNN
-F 2 "" H 9700 2375 50  0001 C CNN
-F 3 "" H 9700 2375 50  0001 C CNN
-	1    9700 2375
-	1    0    0    -1
-$EndComp
-$Comp
-L custom:PTH_1_mm J3
-U 1 1 5C142269
-P 9700 2725
-F 0 "J3" H 9800 2725 50  0000 C CNN
-F 1 "PTH_1_mm" H 9700 2625 50  0000 C CNN
-F 2 "" H 9700 2725 50  0001 C CNN
-F 3 "" H 9700 2725 50  0001 C CNN
-	1    9700 2725
-	1    0    0    -1
-$EndComp
-$Comp
-L custom:PTH_1_mm J4
-U 1 1 5C14226F
-P 9700 2925
-F 0 "J4" H 9800 2925 50  0000 C CNN
-F 1 "PTH_1_mm" H 9700 2825 50  0000 C CNN
-F 2 "" H 9700 2925 50  0001 C CNN
-F 3 "" H 9700 2925 50  0001 C CNN
-	1    9700 2925
-	1    0    0    -1
-$EndComp
-$Comp
-L custom:PTH_1_mm J5
-U 1 1 5C1426F8
-P 9700 3325
-F 0 "J5" H 9800 3325 50  0000 C CNN
-F 1 "PTH_1_mm" H 9700 3225 50  0000 C CNN
-F 2 "" H 9700 3325 50  0001 C CNN
-F 3 "" H 9700 3325 50  0001 C CNN
-	1    9700 3325
-	1    0    0    -1
-$EndComp
-$Comp
-L custom:PTH_1_mm J6
-U 1 1 5C1426FE
-P 9700 3525
-F 0 "J6" H 9800 3525 50  0000 C CNN
-F 1 "PTH_1_mm" H 9700 3425 50  0000 C CNN
-F 2 "" H 9700 3525 50  0001 C CNN
-F 3 "" H 9700 3525 50  0001 C CNN
-	1    9700 3525
-	1    0    0    -1
-$EndComp
-$Comp
-L custom:PTH_1_mm J7
-U 1 1 5C142704
-P 9700 3875
-F 0 "J7" H 9800 3875 50  0000 C CNN
-F 1 "PTH_1_mm" H 9700 3775 50  0000 C CNN
-F 2 "" H 9700 3875 50  0001 C CNN
-F 3 "" H 9700 3875 50  0001 C CNN
-	1    9700 3875
-	1    0    0    -1
-$EndComp
-$Comp
-L custom:PTH_1_mm J8
-U 1 1 5C14270A
-P 9700 4075
-F 0 "J8" H 9800 4075 50  0000 C CNN
-F 1 "PTH_1_mm" H 9700 3975 50  0000 C CNN
-F 2 "" H 9700 4075 50  0001 C CNN
-F 3 "" H 9700 4075 50  0001 C CNN
-	1    9700 4075
-	1    0    0    -1
-$EndComp
-Wire Wire Line
-	9550 2175 9250 2175
-Wire Wire Line
-	9250 2175 9250 2775
-Wire Wire Line
-	9300 2875 9300 2375
-Wire Wire Line
-	9300 2375 9550 2375
-Wire Wire Line
-	9100 2875 9300 2875
-Wire Wire Line
-	9350 2975 9350 2725
-Wire Wire Line
-	9350 2725 9550 2725
-Wire Wire Line
-	9100 2975 9350 2975
-Wire Wire Line
-	9400 3075 9400 2925
-Wire Wire Line
-	9400 2925 9550 2925
-Wire Wire Line
-	9100 3075 9400 3075
-Wire Wire Line
-	9250 3475 9250 4075
-Wire Wire Line
-	9250 4075 9550 4075
-Wire Wire Line
-	9300 3375 9300 3875
-Wire Wire Line
-	9300 3875 9550 3875
-Wire Wire Line
-	9100 3375 9300 3375
-Wire Wire Line
-	9550 3525 9350 3525
-Wire Wire Line
-	9350 3525 9350 3275
-Wire Wire Line
-	9100 3275 9350 3275
-Wire Wire Line
-	9400 3175 9400 3325
-Wire Wire Line
-	9400 3325 9550 3325
-Wire Wire Line
-	9100 3175 9400 3175
-Text Notes 8200 4425 0    67   ~ 0
-ADD 2 mm STRAIN RELIEF HOLES
 $Sheet
-S 3825 2800 900  725
+S 9825 2075 675  350
 U 5C3EC885
 F0 "microcontroller" 50
@@
 $EndSheet
 $Sheet
-S 1625 2950 675  350
+S 9825 750  675  350
 U 5C5AE643
 F0 "battery" 50
 F1 "battery.sch" 50
 $EndSheet
-Text Notes 2900 1050 0    50   ~ 0
-add mounting holes
+Text Notes 6450 1000 0    118  ~ 0
+TODO:\nADD MOUNTING HOLES
+Text Notes 625  1550 0    118  ~ 0
+TABLE OF CONTENTS:\n1. BATTERY\n2. POWER\n3. MICROCONTROLLER\n4. MOTOR DRIVER
+Text Notes 3775 825  0    118  ~ 0
+NOTES:
 $EndSCHEMATC

Commit message: automated commit
Other:
- note added: "TABLE OF CONTENTS:\n1. CONTENTS\n2. BATTERY\n3. POWER\n4. MICROCONTROLLER\n5. MOTOR DRIVER"
- note removed: "TABLE OF CONTENTS:\n1. BATTERY\n2. POWER\n3. MICROCONTROLLER\n4. MOTOR DRIVER"
Changed lines of the file:
@@
 Text Notes 6450 1000 0    118  ~ 0
 TODO:\nADD MOUNTING HOLES
-Text Notes 625  1550 0    118  ~ 0
-TABLE OF CONTENTS:\n1. BATTERY\n2. POWER\n3. MICROCONTROLLER\n4. MOTOR DRIVER
+Text Notes 650  1725 0    118  ~ 0
+TABLE OF CONTENTS:\n1. CONTENTS\n2. BATTERY\n3. POWER\n4. MICROCONTROLLER\n5. MOTOR DRIVER
 Text Notes 3775 825  0    118  ~ 0
 NOTES:

Commit message: automated commit
Parts:
- added MH1, MH2, MH3, MH4: M4_MOUNTING_HOLE, MountingHole:MountingHole_4.3mm_M4_Pad, symbol custom:M4_MOUNTING_HOLE
- added R37, R38, R39, R40: NP_R_0603, custom:NP_0603, symbol custom:NP_R_0603
Connections:
- new net: MH4.1, R40.1
- new net: MH3.1, R39.1
- new net: MH2.1, R38.1
- new net: MH1.1, R37.1
- new net GND: R37.2, R38.2, R39.2, R40.2
Other:
- note removed: "NOTES:"
- note removed: "TODO:\nADD MOUNTING HOLES"
Changed lines of the file:
@@
 F1 "battery.sch" 50
 $EndSheet
-Text Notes 6450 1000 0    118  ~ 0
-TODO:\nADD MOUNTING HOLES
 Text Notes 650  1725 0    118  ~ 0
 TABLE OF CONTENTS:\n1. CONTENTS\n2. BATTERY\n3. POWER\n4. MICROCONTROLLER\n5. MOTOR DRIVER
-Text Notes 3775 825  0    118  ~ 0
-NOTES:
+$Comp
+L custom:M4_MOUNTING_HOLE MH4
+U 1 1 5C5777F1
+P 10725 4225
+F 0 "MH4" H 10675 4375 50  0000 L BNN
+F 1 "M4_MOUNTING_HOLE" H 10725 3825 50  0001 L BNN
+F 2 "MountingHole:MountingHole_4.3mm_M4_Pad" H 10725 3725 50  0001 L BNN
+F 3 "" H 10725 4475 50  0001 L BNN
+F 4 "M4" H 10775 4175 50  0000 L BNN "SIZE"
+	1    10725 4225
+	1    0    0    -1
+$EndComp
+$Comp
+L custom:M4_MOUNTING_HOLE MH3
+U 1 1 5C577895
+P 10425 4225
+F 0 "MH3" H 10375 4375 50  0000 L BNN
+F 1 "M4_MOUNTING_HOLE" H 10425 3825 50  0001 L BNN
+F 2 "MountingHole:MountingHole_4.3mm_M4_Pad" H 10425 3725 50  0001 L BNN
+F 3 "" H 10425 4475 50  0001 L BNN
+F 4 "M4" H 10475 4175 50  0000 L BNN "SIZE"
+	1    10425 4225
+	1    0    0    -1
+$EndComp
+$Comp
+L custom:M4_MOUNTING_HOLE MH2
+U 1 1 5C577978
+P 10125 4225
+F 0 "MH2" H 10075 4375 50  0000 L BNN
+F 1 "M4_MOUNTING_HOLE" H 10125 3825 50  0001 L BNN
+F 2 "MountingHole:MountingHole_4.3mm_M4_Pad" H 10125 3725 50  0001 L BNN
+F 3 "" H 10125 4475 50  0001 L BNN
+F 4 "M4" H 10175 4175 50  0000 L BNN "SIZE"
+	1    10125 4225
+	1    0    0    -1
+$EndComp
+$Comp
+L custom:M4_MOUNTING_HOLE MH1
+U 1 1 5C577980
+P 9825 4225
+F 0 "MH1" H 9775 4375 50  0000 L BNN
+F 1 "M4_MOUNTING_HOLE" H 9825 3825 50  0001 L BNN
+F 2 "MountingHole:MountingHole_4.3mm_M4_Pad" H 9825 3725 50  0001 L BNN
+F 3 "" H 9825 4475 50  0001 L BNN
+F 4 "M4" H 9875 4175 50  0000 L BNN "SIZE"
+	1    9825 4225
+	1    0    0    -1
+$EndComp
+$Comp
+L power:GND #PWR085
+U 1 1 5C577B88
+P 10725 4725
+F 0 "#PWR085" H 10725 4475 50  0001 C CNN
+F 1 "GND" H 10725 4575 50  0000 C CNN
+F 2 "" H 10725 4725 50  0001 C CNN
+F 3 "" H 10725 4725 50  0001 C CNN
+	1    10725 4725
+	1    0    0    -1
+$EndComp
+$Comp
+L custom:NP_R_0603 R40
+U 1 1 5C577F21
+P 10725 4525
+F 0 "R40" V 10665 4475 50  0000 L BNN
+F 1 "NP_R_0603" V 10850 4200 50  0001 L BNN
+F 2 "custom:NP_0603" V 10925 4425 50  0001 L BNN
+F 3 "" V 10665 4485 50  0001 C CNN
+F 4 "NP" V 10755 4465 50  0000 L BNN "NOPOP"
+	1    10725 4525
+	1    0    0    -1
+$EndComp
+Wire Wire Line
+	10725 4725 10725 4675
+Wire Wire Line
+	10725 4375 10725 4325
+$Comp
+L power:GND #PWR084
+U 1 1 5C578042
+P 10425 4725
+F 0 "#PWR084" H 10425 4475 50  0001 C CNN
+F 1 "GND" H 10425 4575 50  0000 C CNN
+F 2 "" H 10425 4725 50  0001 C CNN
+F 3 "" H 10425 4725 50  0001 C CNN
+	1    10425 4725
+	1    0    0    -1
+$EndComp
+$Comp
+L custom:NP_R_0603 R39
+U 1 1 5C578049
+P 10425 4525
+F 0 "R39" V 10365 4475 50  0000 L BNN
+F 1 "NP_R_0603" V 10550 4200 50  0001 L BNN
+F 2 "custom:NP_0603" V 10625 4425 50  0001 L BNN
+F 3 "" V 10365 4485 50  0001 C CNN
+F 4 "NP" V 10455 4465 50  0000 L BNN "NOPOP"
+	1    10425 4525
+	1    0    0    -1
+$EndComp
+Wire Wire Line
+	10425 4725 10425 4675
+Wire Wire Line
+	10425 4375 10425 4325
+$Comp
+L power:GND #PWR083
+U 1 1 5C57808A
+P 10125 4725
+F 0 "#PWR083" H 10125 4475 50  0001 C CNN
+F 1 "GND" H 10125 4575 50  0000 C CNN
+F 2 "" H 10125 4725 50  0001 C CNN
+F 3 "" H 10125 4725 50  0001 C CNN
+	1    10125 4725
+	1    0    0    -1
+$EndComp
+$Comp
+L custom:NP_R_0603 R38
+U 1 1 5C578091
+P 10125 4525
+F 0 "R38" V 10065 4475 50  0000 L BNN
+F 1 "NP_R_0603" V 10250 4200 50  0001 L BNN
+F 2 "custom:NP_0603" V 10325 4425 50  0001 L BNN
+F 3 "" V 10065 4485 50  0001 C CNN
+F 4 "NP" V 10155 4465 50  0000 L BNN "NOPOP"
+	1    10125 4525
+	1    0    0    -1
+$EndComp
+Wire Wire Line
+	10125 4725 10125 4675
+Wire Wire Line
+	10125 4375 10125 4325
+$Comp
+L power:GND #PWR082
+U 1 1 5C57810A
+P 9825 4725
+F 0 "#PWR082" H 9825 4475 50  0001 C CNN
+F 1 "GND" H 9825 4575 50  0000 C CNN
+F 2 "" H 9825 4725 50  0001 C CNN
+F 3 "" H 9825 4725 50  0001 C CNN
+	1    9825 4725
+	1    0    0    -1
+$EndComp
+$Comp
+L custom:NP_R_0603 R37
+U 1 1 5C578111
+P 9825 4525
+F 0 "R37" V 9765 4475 50  0000 L BNN
+F 1 "NP_R_0603" V 9950 4200 50  0001 L BNN
+F 2 "custom:NP_0603" V 10025 4425 50  0001 L BNN
+F 3 "" V 9765 4485 50  0001 C CNN
+F 4 "NP" V 9855 4465 50  0000 L BNN "NOPOP"
+	1    9825 4525
+	1    0    0    -1
+$EndComp
+Wire Wire Line
+	9825 4725 9825 4675
+Wire Wire Line
+	9825 4375 9825 4325
 $EndSCHEMATC
