File: nu.ai_motor_controller/nu.ai_motor_controller.sch (KiCad schematic (older format))
At the start: 8 parts

Commit message: automated commit
Parts:
- added MH5: M4_MOUNTING_HOLE, MountingHole:MountingHole_4.3mm_M4_Pad, symbol custom:M4_MOUNTING_HOLE
- added R42: NP_R_0603, custom:NP_0603, symbol custom:NP_R_0603
Connections:
- net GND: now also R42.2
- new net: MH5.1, R42.1
Other:
- moved on the sheet: MH1, MH2, MH3, MH4, R37, R38, R39, R40
Changed lines of the file:
@@
 L custom:M4_MOUNTING_HOLE MH4
 U 1 1 5C5777F1
-P 10725 4225
-F 0 "MH4" H 10675 4375 50  0000 L BNN
-F 1 "M4_MOUNTING_HOLE" H 10725 3825 50  0001 L BNN
-F 2 "MountingHole:MountingHole_4.3mm_M4_Pad" H 10725 3725 50  0001 L BNN
-F 3 "" H 10725 4475 50  0001 L BNN
-F 4 "M4" H 10775 4175 50  0000 L BNN "SIZE"
-	1    10725 4225
+P 10525 4225
+F 0 "MH4" H 10475 4375 50  0000 L BNN
+F 1 "M4_MOUNTING_HOLE" H 10525 3825 50  0001 L BNN
+F 2 "MountingHole:MountingHole_4.3mm_M4_Pad" H 10525 3725 50  0001 L BNN
+F 3 "" H 10525 4475 50  0001 L BNN
+F 4 "M4" H 10575 4175 50  0000 L BNN "SIZE"
+	1    10525 4225
 	1    0    0    -1
 $EndComp
@@
 L custom:M4_MOUNTING_HOLE MH3
 U 1 1 5C577895
-P 10425 4225
-F 0 "MH3" H 10375 4375 50  0000 L BNN
-F 1 "M4_MOUNTING_HOLE" H 10425 3825 50  0001 L BNN
-F 2 "MountingHole:MountingHole_4.3mm_M4_Pad" H 10425 3725 50  0001 L BNN
-F 3 "" H 10425 4475 50  0001 L BNN
-F 4 "M4" H 10475 4175 50  0000 L BNN "SIZE"
-	1    10425 4225
+P 10225 4225
+F 0 "MH3" H 10175 4375 50  0000 L BNN
+F 1 "M4_MOUNTING_HOLE" H 10225 3825 50  0001 L BNN
+F 2 "MountingHole:MountingHole_4.3mm_M4_Pad" H 10225 3725 50  0001 L BNN
+F 3 "" H 10225 4475 50  0001 L BNN
+F 4 "M4" H 10275 4175 50  0000 L BNN "SIZE"
+	1    10225 4225
 	1    0    0    -1
 $EndComp
@@
 L custom:M4_MOUNTING_HOLE MH2
 U 1 1 5C577978
-P 10125 4225
-F 0 "MH2" H 10075 4375 50  0000 L BNN
-F 1 "M4_MOUNTING_HOLE" H 10125 3825 50  0001 L BNN
-F 2 "MountingHole:MountingHole_4.3mm_M4_Pad" H 10125 3725 50  0001 L BNN
-F 3 "" H 10125 4475 50  0001 L BNN
-F 4 "M4" H 10175 4175 50  0000 L BNN "SIZE"
-	1    10125 4225
+P 9925 4225
+F 0 "MH2" H 9875 4375 50  0000 L BNN
+F 1 "M4_MOUNTING_HOLE" H 9925 3825 50  0001 L BNN
+F 2 "MountingHole:MountingHole_4.3mm_M4_Pad" H 9925 3725 50  0001 L BNN
+F 3 "" H 9925 4475 50  0001 L BNN
+F 4 "M4" H 9975 4175 50  0000 L BNN "SIZE"
+	1    9925 4225
 	1    0    0    -1
 $EndComp
@@
 L custom:M4_MOUNTING_HOLE MH1
 U 1 1 5C577980
-P 9825 4225
-F 0 "MH1" H 9775 4375 50  0000 L BNN
-F 1 "M4_MOUNTING_HOLE" H 9825 3825 50  0001 L BNN
-F 2 "MountingHole:MountingHole_4.3mm_M4_Pad" H 9825 3725 50  0001 L BNN
-F 3 "" H 9825 4475 50  0001 L BNN
-F 4 "M4" H 9875 4175 50  0000 L BNN "SIZE"
-	1    9825 4225
+P 9625 4225
+F 0 "MH1" H 9575 4375 50  0000 L BNN
+F 1 "M4_MOUNTING_HOLE" H 9625 3825 50  0001 L BNN
+F 2 "MountingHole:MountingHole_4.3mm_M4_Pad" H 9625 3725 50  0001 L BNN
+F 3 "" H 9625 4475 50  0001 L BNN
+F 4 "M4" H 9675 4175 50  0000 L BNN "SIZE"
+	1    9625 4225
 	1    0    0    -1
 $EndComp
@@
 L power:GND #PWR085
 U 1 1 5C577B88
-P 10725 4725
-F 0 "#PWR085" H 10725 4475 50  0001 C CNN
-F 1 "GND" H 10725 4575 50  0000 C CNN
-F 2 "" H 10725 4725 50  0001 C CNN
-F 3 "" H 10725 4725 50  0001 C CNN
-	1    10725 4725
+P 10525 4725
+F 0 "#PWR085" H 10525 4475 50  0001 C CNN
+F 1 "GND" H 10525 4575 50  0000 C CNN
+F 2 "" H 10525 4725 50  0001 C CNN
+F 3 "" H 10525 4725 50  0001 C CNN
+	1    10525 4725
 	1    0    0    -1
 $EndComp
@@
 L custom:NP_R_0603 R40
 U 1 1 5C577F21
-P 10725 4525
-F 0 "R40" V 10665 4475 50  0000 L BNN
-F 1 "NP_R_0603" V 10850 4200 50  0001 L BNN
-F 2 "custom:NP_0603" V 10925 4425 50  0001 L BNN
-F 3 "" V 10665 4485 50  0001 C CNN
-F 4 "NP" V 10755 4465 50  0000 L BNN "NOPOP"
-	1    10725 4525
+P 10525 4525
+F 0 "R40" V 10465 4475 50  0000 L BNN
+F 1 "NP_R_0603" V 10650 4200 50  0001 L BNN
+F 2 "custom:NP_0603" V 10725 4425 50  0001 L BNN
+F 3 "" V 10465 4485 50  0001 C CNN
+F 4 "NP" V 10555 4465 50  0000 L BNN "NOPOP"
+	1    10525 4525
 	1    0    0    -1
 $EndComp
 Wire Wire Line
-	10725 4725 10725 4675
+	10525 4725 10525 4675
 Wire Wire Line
-	10725 4375 10725 4325
+	10525 4375 10525 4325
 $Comp
 L power:GND #PWR084
 U 1 1 5C578042
-P 10425 4725
-F 0 "#PWR084" H 10425 4475 50  0001 C CNN
-F 1 "GND" H 10425 4575 50  0000 C CNN
-F 2 "" H 10425 4725 50  0001 C CNN
-F 3 "" H 10425 4725 50  0001 C CNN
-	1    10425 4725
+P 10225 4725
+F 0 "#PWR084" H 10225 4475 50  0001 C CNN
+F 1 "GND" H 10225 4575 50  0000 C CNN
+F 2 "" H 10225 4725 50  0001 C CNN
+F 3 "" H 10225 4725 50  0001 C CNN
+	1    10225 4725
 	1    0    0    -1
 $EndComp
@@
 L custom:NP_R_0603 R39
 U 1 1 5C578049
-P 10425 4525
-F 0 "R39" V 10365 4475 50  0000 L BNN
-F 1 "NP_R_0603" V 10550 4200 50  0001 L BNN
-F 2 "custom:NP_0603" V 10625 4425 50  0001 L BNN
-F 3 "" V 10365 4485 50  0001 C CNN
-F 4 "NP" V 10455 4465 50  0000 L BNN "NOPOP"
-	1    10425 4525
+P 10225 4525
+F 0 "R39" V 10165 4475 50  0000 L BNN
+F 1 "NP_R_0603" V 10350 4200 50  0001 L BNN
+F 2 "custom:NP_0603" V 10425 4425 50  0001 L BNN
+F 3 "" V 10165 4485 50  0001 C CNN
+F 4 "NP" V 10255 4465 50  0000 L BNN "NOPOP"
+	1    10225 4525
 	1    0    0    -1
 $EndComp
 Wire Wire Line
-	10425 4725 10425 4675
+	10225 4725 10225 4675
 Wire Wire Line
-	10425 4375 10425 4325
+	10225 4375 10225 4325
 $Comp
 L power:GND #PWR083
 U 1 1 5C57808A
-P 10125 4725
-F 0 "#PWR083" H 10125 4475 50  0001 C CNN
-F 1 "GND" H 10125 4575 50  0000 C CNN
-F 2 "" H 10125 4725 50  0001 C CNN
-F 3 "" H 10125 4725 50  0001 C CNN
-	1    10125 4725
+P 9925 4725
+F 0 "#PWR083" H 9925 4475 50  0001 C CNN
+F 1 "GND" H 9925 4575 50  0000 C CNN
+F 2 "" H 9925 4725 50  0001 C CNN
+F 3 "" H 9925 4725 50  0001 C CNN
+	1    9925 4725
 	1    0    0    -1
 $EndComp
@@
 L custom:NP_R_0603 R38
 U 1 1 5C578091
-P 10125 4525
-F 0 "R38" V 10065 4475 50  0000 L BNN
-F 1 "NP_R_0603" V 10250 4200 50  0001 L BNN
-F 2 "custom:NP_0603" V 10325 4425 50  0001 L BNN
-F 3 "" V 10065 4485 50  0001 C CNN
-F 4 "NP" V 10155 4465 50  0000 L BNN "NOPOP"
-	1    10125 4525
+P 9925 4525
+F 0 "R38" V 9865 4475 50  0000 L BNN
+F 1 "NP_R_0603" V 10050 4200 50  0001 L BNN
+F 2 "custom:NP_0603" V 10125 4425 50  0001 L BNN
+F 3 "" V 9865 4485 50  0001 C CNN
+F 4 "NP" V 9955 4465 50  0000 L BNN "NOPOP"
+	1    9925 4525
 	1    0    0    -1
 $EndComp
 Wire Wire Line
-	10125 4725 10125 4675
+	9925 4725 9925 4675
 Wire Wire Line
-	10125 4375 10125 4325
+	9925 4375 9925 4325
 $Comp
 L power:GND #PWR082
 U 1 1 5C57810A
-P 9825 4725
-F 0 "#PWR082" H 9825 4475 50  0001 C CNN
-F 1 "GND" H 9825 4575 50  0000 C CNN
-F 2 "" H 9825 4725 50  0001 C CNN
-F 3 "" H 9825 4725 50  0001 C CNN
-	1    9825 4725
+P 9625 4725
+F 0 "#PWR082" H 9625 4475 50  0001 C CNN
+F 1 "GND" H 9625 4575 50  0000 C CNN
+F 2 "" H 9625 4725 50  0001 C CNN
+F 3 "" H 9625 4725 50  0001 C CNN
+	1    9625 4725
 	1    0    0    -1
 $EndComp
@@
 L custom:NP_R_0603 R37
 U 1 1 5C578111
-P 9825 4525
-F 0 "R37" V 9765 4475 50  0000 L BNN
-F 1 "NP_R_0603" V 9950 4200 50  0001 L BNN
-F 2 "custom:NP_0603" V 10025 4425 50  0001 L BNN
-F 3 "" V 9765 4485 50  0001 C CNN
-F 4 "NP" V 9855 4465 50  0000 L BNN "NOPOP"
-	1    9825 4525
+P 9625 4525
+F 0 "R37" V 9565 4475 50  0000 L BNN
+F 1 "NP_R_0603" V 9750 4200 50  0001 L BNN
+F 2 "custom:NP_0603" V 9825 4425 50  0001 L BNN
+F 3 "" V 9565 4485 50  0001 C CNN
+F 4 "NP" V 9655 4465 50  0000 L BNN "NOPOP"
+	1    9625 4525
 	1    0    0    -1
 $EndComp
 Wire Wire Line
-	9825 4725 9825 4675
+	9625 4725 9625 4675
 Wire Wire Line
-	9825 4375 9825 4325
+	9625 4375 9625 4325
+$Comp
+L custom:M4_MOUNTING_HOLE MH5
+U 1 1 5C9BA1C6
+P 10825 4225
+F 0 "MH5" H 10775 4375 50  0000 L BNN
+F 1 "M4_MOUNTING_HOLE" H 10825 3825 50  0001 L BNN
+F 2 "MountingHole:MountingHole_4.3mm_M4_Pad" H 10825 3725 50  0001 L BNN
+F 3 "" H 10825 4475 50  0001 L BNN
+F 4 "M4" H 10875 4175 50  0000 L BNN "SIZE"
+	1    10825 4225
+	1    0    0    -1
+$EndComp
+$Comp
+L power:GND #PWR089
+U 1 1 5C9BA1CD
+P 10825 4725
+F 0 "#PWR089" H 10825 4475 50  0001 C CNN
+F 1 "GND" H 10825 4575 50  0000 C CNN
+F 2 "" H 10825 4725 50  0001 C CNN
+F 3 "" H 10825 4725 50  0001 C CNN
+	1    10825 4725
+	1    0    0    -1
+$EndComp
+$Comp
+L custom:NP_R_0603 R42
+U 1 1 5C9BA1D4
+P 10825 4525
+F 0 "R42" V 10765 4475 50  0000 L BNN
+F 1 "NP_R_0603" V 10950 4200 50  0001 L BNN
+F 2 "custom:NP_0603" V 11025 4425 50  0001 L BNN
+F 3 "" V 10765 4485 50  0001 C CNN
+F 4 "NP" V 10855 4465 50  0000 L BNN "NOPOP"
+	1    10825 4525
+	1    0    0    -1
+$EndComp
+Wire Wire Line
+	10825 4325 10825 4375
+Wire Wire Line
+	10825 4675 10825 4725
 $EndSCHEMATC

Commit message: automated commit
Parts:
- MH1, MH2, MH3, MH4, MH5: footprint MountingHole:MountingHole_4.3mm_M4_Pad -> custom:MountingHole_4.3mm_M4_Pad
Changed lines of the file:
@@
 F 0 "MH4" H 10475 4375 50  0000 L BNN
 F 1 "M4_MOUNTING_HOLE" H 10525 3825 50  0001 L BNN
-F 2 "MountingHole:MountingHole_4.3mm_M4_Pad" H 10525 3725 50  0001 L BNN
+F 2 "custom:MountingHole_4.3mm_M4_Pad" H 10525 3725 50  0001 L BNN
 F 3 "" H 10525 4475 50  0001 L BNN
 F 4 "M4" H 10575 4175 50  0000 L BNN "SIZE"
@@
 F 0 "MH3" H 10175 4375 50  0000 L BNN
 F 1 "M4_MOUNTING_HOLE" H 10225 3825 50  0001 L BNN
-F 2 "MountingHole:MountingHole_4.3mm_M4_Pad" H 10225 3725 50  0001 L BNN
+F 2 "custom:MountingHole_4.3mm_M4_Pad" H 10225 3725 50  0001 L BNN
 F 3 "" H 10225 4475 50  0001 L BNN
 F 4 "M4" H 10275 4175 50  0000 L BNN "SIZE"
@@
 F 0 "MH2" H 9875 4375 50  0000 L BNN
 F 1 "M4_MOUNTING_HOLE" H 9925 3825 50  0001 L BNN
-F 2 "MountingHole:MountingHole_4.3mm_M4_Pad" H 9925 3725 50  0001 L BNN
+F 2 "custom:MountingHole_4.3mm_M4_Pad" H 9925 3725 50  0001 L BNN
 F 3 "" H 9925 4475 50  0001 L BNN
 F 4 "M4" H 9975 4175 50  0000 L BNN "SIZE"
@@
 F 0 "MH1" H 9575 4375 50  0000 L BNN
 F 1 "M4_MOUNTING_HOLE" H 9625 3825 50  0001 L BNN
-F 2 "MountingHole:MountingHole_4.3mm_M4_Pad" H 9625 3725 50  0001 L BNN
+F 2 "custom:MountingHole_4.3mm_M4_Pad" H 9625 3725 50  0001 L BNN
 F 3 "" H 9625 4475 50  0001 L BNN
 F 4 "M4" H 9675 4175 50  0000 L BNN "SIZE"
@@
 F 0 "MH5" H 10775 4375 50  0000 L BNN
 F 1 "M4_MOUNTING_HOLE" H 10825 3825 50  0001 L BNN
-F 2 "MountingHole:MountingHole_4.3mm_M4_Pad" H 10825 3725 50  0001 L BNN
+F 2 "custom:MountingHole_4.3mm_M4_Pad" H 10825 3725 50  0001 L BNN
 F 3 "" H 10825 4475 50  0001 L BNN
 F 4 "M4" H 10875 4175 50  0000 L BNN "SIZE"
