File: nu.ai_motor_controller/power.sch (KiCad schematic (older format))
At the start: 6 parts

Commit message: cleaned up and renamed project files. Changed custom library management scheme. It now resides in my homedir as a seperate git project, and is pointed to in kicad's symbol library manager
Parts:
- J? (x3): symbol nu-rescue:S4B-XH-A-custom -> custom:S4B-XH-A
Changed lines of the file:
@@
 EESchema Schematic File Version 4
-LIBS:nu-cache
+LIBS:nu.ai_motor_controller-cache
 EELAYER 26 0
 EELAYER END
@@
 $EndDescr
 $Comp
-L nu-rescue:S4B-XH-A-custom J?
+L custom:S4B-XH-A J?
 U 1 1 5C34712D
 P 6025 3000
@@
 BATTERY\nTAPS
 $Comp
-L nu-rescue:S4B-XH-A-custom J?
+L custom:S4B-XH-A J?
 U 1 1 5C36BCF1
 P 6025 3700
@@
 $EndComp
 $Comp
-L nu-rescue:S4B-XH-A-custom J?
+L custom:S4B-XH-A J?
 U 1 1 5C36BD2D
 P 6025 2300

Commit message: automated commit
Other:
- note added: "TO ADCs"
Changed lines of the file:
@@
 Connection ~ 5350 3000
 Connection ~ 5250 2900
+Text Notes 3450 2325 0    50   ~ 0
+TO ADCs
 $EndSCHEMATC

Commit message: automated commit
Parts:
- removed R? (x3): RC0603JR-071KL, 0603, symbol custom:RC0603JR-071KL
- added J?: Screw_Terminal_01x02, symbol Connector:Screw_Terminal_01x02
- added J? (x2): PTH_3_mm, symbol custom:PTH_3_mm
- added Q? (x6): DMG6602, TSOT-23-6, symbol custom:DMG6602
- added R? (x9): CR0603-JW-103ELF, 0603, symbol custom:CR0603-JW-103ELF
- added R? (x3): RC0603JR-071KL, 0603, symbol custom:RC0603JR-071KL
- added TP? (x7): PTH_0.5_mm, symbol custom:PTH_0.5_mm
Connections:
- net labels added: BAT_0, BAT_1, BAT_2, BAT_TEST, TAP_0, TAP_1, TAP_2
- wire segments 27 -> 89
Other:
- note added: "INDICATE POS AND NEG\nON SILKSCREEN"
- note added: "INDICATE VOLTAGES\nON SILKSCREEN"
- note added: "XT60 MALE CABLE ASSEMBLY\nADD 4 mm STRAIN RELIEF HOLES"
- note removed: "TO ADCs"

Commit message: automated commit
Parts:
- removed Q? (x2): DMG6602, TSOT-23-6, symbol custom:DMG6602
- added Q? (x2): DMG6602, TSOT-23-6, symbol custom:DMG6602
- added SW? (x2): RA_SLIDE_SWITCH_DPDT, Connector_PinHeader_2.54mm:PinHeader_2x03_P2.54mm_Vertical, symbol custom:RA_SLIDE_SWITCH_DPDT
- J?: value Screw_Terminal_01x02 -> NP_Screw_Terminal_01x02
Connections:
- net labels added: VDD_BAT
- wire segments 89 -> 99
Other:
- note added: "XT60 MALE CABLE ASSEMBLY.\nADD 4 mm STRAIN RELIEF HOLES.\nINDICATE POS AND NEG\nON SILKSCREEN"
- note removed: "XT60 MALE CABLE ASSEMBLY\nADD 4 mm STRAIN RELIEF HOLES"
- moved on the sheet: J?, TP?

Commit message: automated commit
Parts:
- removed J? (x3): S4B-XH-A, Connector_PinHeader_2.54mm:PinHeader_1x04_P2.54mm_Horizontal, symbol custom:S4B-XH-A
- removed J?: NP_Screw_Terminal_01x02, symbol Connector:Screw_Terminal_01x02
- removed J? (x2): PTH_3_mm, symbol custom:PTH_3_mm
- removed Q? (x6): DMG6602, TSOT-23-6, symbol custom:DMG6602
- removed R? (x9): CR0603-JW-103ELF, 0603, symbol custom:CR0603-JW-103ELF
- removed R? (x3): RC0603JR-071KL, 0603, symbol custom:RC0603JR-071KL
- removed SW? (x2): RA_SLIDE_SWITCH_DPDT, Connector_PinHeader_2.54mm:PinHeader_2x03_P2.54mm_Vertical, symbol custom:RA_SLIDE_SWITCH_DPDT
- removed TP? (x7): PTH_0.5_mm, symbol custom:PTH_0.5_mm
Other:
- note removed: "BATTERY\nTAPS"
- note removed: "INDICATE POS AND NEG\nON SILKSCREEN"
- note removed: "INDICATE VOLTAGES\nON SILKSCREEN"
- note removed: "XT60 MALE CABLE ASSEMBLY.\nADD 4 mm STRAIN RELIEF HOLES.\nINDICATE POS AND NEG\nON SILKSCREEN"

Commit message: automated commit
Parts:
- added U?: AZ2117, Package_TO_SOT_SMD:SOT-223, symbol custom:AZ2117
Other:
- note added: "add 10uf caps"
Changed lines of the file:
@@
 Comment4 ""
 $EndDescr
+$Comp
+L custom:AZ2117 U?
+U 1 1 5C50287B
+P 6900 1900
+F 0 "U?" H 6650 2100 60  0000 L BNN
+F 1 "AZ2117" H 7000 1300 60  0001 L BNN
+F 2 "Package_TO_SOT_SMD:SOT-223" H 6950 1500 60  0001 L BNN
+F 3 "/home/dj/datasheets/AZ2117.pdf" H 6950 1400 60  0001 L BNN
+	1    6900 1900
+	1    0    0    -1
+$EndComp
+Text Notes 5825 1975 0    50   ~ 0
+add 10uf caps
 $EndSCHEMATC

Commit message: automated commit
Other:
- note added: "For 3V3, R2=7.5k, R1=4.7k\nFor 1V8, R2=2k, R1=4.7k"
Changed lines of the file:
@@
 Text Notes 5825 1975 0    50   ~ 0
 add 10uf caps
+Text Notes 7575 2250 0    50   ~ 0
+For 3V3, R2=7.5k, R1=4.7k\nFor 1V8, R2=2k, R1=4.7k
 $EndSCHEMATC

Commit message: automated commit
Parts:
- removed U?: AZ2117, Package_TO_SOT_SMD:SOT-223, symbol custom:AZ2117
- added C? (x4): CL10B103KB8SFNC, Capacitor_SMD:C_0603_1608Metric, symbol custom:CL10B103KB8SFNC
- added R? (x2): RMCF0603FT4K70, Resistor_SMD:R_0603_1608Metric, symbol custom:RMCF0603FT4K70
- added R?: RMCF0603FT7K50, Resistor_SMD:R_0603_1608Metric, symbol custom:RMCF0603FT7K50
- added R?: RMCF0603FT2K00, Resistor_SMD:R_0603_1608Metric, symbol custom:RMCF0603FT2K00
- added U? (x2): AZ2117, Package_TO_SOT_SMD:SOT-223, symbol custom:AZ2117
Connections:
- new net: R?.1, R?.2, U?.1 (ADJ) (x2)
- new net +1V8: C?.1, R?.1, U?.2 (VOUT), U?.4 (VOUT)
- new net +3V3: C?.1, R?.1, U?.2 (VOUT), U?.4 (VOUT)
- new net +5V: C?.1, C?.1, U?.3 (VIN), U?.3 (VIN)
- new net GND: C?.2, C?.2, C?.2, C?.2, R?.2, R?.2
Other:
- note added: "1V8 LDO"
- note added: "3V3 LDO"
- note added: "PAGE 1 IN AZ2117-ADJ DATASHEET:\nV_OUT = V_REF * (1 + R2 / R1) + I_ADJ * R2\nFOR 3V3, R2=7k5, R1=4k7\nFOR 1V8, R2=2k0, R1=4k7"
- note removed: "For 3V3, R2=7.5k, R1=4.7k\nFor 1V8, R2=2k, R1=4.7k"
- note removed: "add 10uf caps"
