File: nu.ai_motor_controller/power.sch (KiCad schematic (older format))
At the start: 10 parts

Commit message: automated commit
Parts:
- gave numbers to parts that had none: 10
Changed lines of the file:
@@
 PAGE 1 IN AZ2117-ADJ DATASHEET:\nV_OUT = V_REF * (1 + R2 / R1) + I_ADJ * R2\nFOR 3V3, R2=7k5, R1=4k7\nFOR 1V8, R2=2k0, R1=4k7
 $Comp
-L custom:CL10B103KB8SFNC C?
+L custom:CL10B103KB8SFNC C1
 U 1 1 5C5133B1
 P 5625 1850
-F 0 "C?" H 5775 1950 50  0000 L BNN
+F 0 "C1" H 5775 1950 50  0000 L BNN
 F 1 "CL10B103KB8SFNC" H 4875 1400 50  0001 L BNN
 F 2 "Capacitor_SMD:C_0603_1608Metric" H 4875 1300 50  0001 L BNN
@@
 $EndComp
 $Comp
-L custom:CL10B103KB8SFNC C?
+L custom:CL10B103KB8SFNC C2
 U 1 1 5C513508
 P 7300 1850
-F 0 "C?" H 7450 1950 50  0000 L BNN
+F 0 "C2" H 7450 1950 50  0000 L BNN
 F 1 "CL10B103KB8SFNC" H 6550 1400 50  0001 L BNN
 F 2 "Capacitor_SMD:C_0603_1608Metric" H 6550 1300 50  0001 L BNN
@@
 $EndComp
 $Comp
-L power:GND #PWR?
+L power:GND #PWR09
 U 1 1 5C513781
 P 5625 2075
-F 0 "#PWR?" H 5625 1825 50  0001 C CNN
+F 0 "#PWR09" H 5625 1825 50  0001 C CNN
 F 1 "GND" H 5625 1925 50  0000 C CNN
 F 2 "" H 5625 2075 50  0001 C CNN
@@
 $EndComp
 $Comp
-L power:GND #PWR?
+L power:GND #PWR010
 U 1 1 5C5138BD
 P 7300 2075
-F 0 "#PWR?" H 7300 1825 50  0001 C CNN
+F 0 "#PWR010" H 7300 1825 50  0001 C CNN
 F 1 "GND" H 7300 1925 50  0000 C CNN
 F 2 "" H 7300 2075 50  0001 C CNN
@@
 	6875 1600 7300 1600
 $Comp
-L custom:RMCF0603FT4K70 R?
+L custom:RMCF0603FT4K70 R9
 U 1 1 5C57045F
 P 6875 2075
-F 0 "R?" H 6950 2050 50  0000 L BNN
+F 0 "R9" H 6950 2050 50  0000 L BNN
 F 1 "RMCF0603FT4K70" H 6175 1675 50  0001 L BNN
 F 2 "Resistor_SMD:R_0603_1608Metric" H 6175 1575 50  0001 L BNN
@@
 $EndComp
 $Comp
-L custom:RMCF0603FT7K50 R?
+L custom:RMCF0603FT7K50 R11
 U 1 1 5C570675
 P 6875 2475
-F 0 "R?" H 6950 2450 50  0000 L BNN
+F 0 "R11" H 6950 2450 50  0000 L BNN
 F 1 "RMCF0603FT7K50" H 6175 2075 50  0001 L BNN
 F 2 "Resistor_SMD:R_0603_1608Metric" H 6175 1975 50  0001 L BNN
@@
 Connection ~ 6875 1700
 $Comp
-L power:GND #PWR?
+L power:GND #PWR013
 U 1 1 5C5709A4
 P 6875 2700
-F 0 "#PWR?" H 6875 2450 50  0001 C CNN
+F 0 "#PWR013" H 6875 2450 50  0001 C CNN
 F 1 "GND" H 6875 2550 50  0000 C CNN
 F 2 "" H 6875 2700 50  0001 C CNN
@@
 3V3 LDO
 $Comp
-L custom:RMCF0603FT2K00 R?
+L custom:RMCF0603FT2K00 R12
 U 1 1 5C570BE1
 P 9525 2475
-F 0 "R?" H 9600 2450 50  0000 L BNN
+F 0 "R12" H 9600 2450 50  0000 L BNN
 F 1 "RMCF0603FT2K00" H 8825 2075 50  0001 L BNN
 F 2 "Resistor_SMD:R_0603_1608Metric" H 8825 1975 50  0001 L BNN
@@
 $EndComp
 $Comp
-L custom:CL10B103KB8SFNC C?
+L custom:CL10B103KB8SFNC C3
 U 1 1 5C57128D
 P 8275 1850
-F 0 "C?" H 8425 1950 50  0000 L BNN
+F 0 "C3" H 8425 1950 50  0000 L BNN
 F 1 "CL10B103KB8SFNC" H 7525 1400 50  0001 L BNN
 F 2 "Capacitor_SMD:C_0603_1608Metric" H 7525 1300 50  0001 L BNN
@@
 $EndComp
 $Comp
-L custom:CL10B103KB8SFNC C?
+L custom:CL10B103KB8SFNC C4
 U 1 1 5C571296
 P 9950 1850
-F 0 "C?" H 10100 1950 50  0000 L BNN
+F 0 "C4" H 10100 1950 50  0000 L BNN
 F 1 "CL10B103KB8SFNC" H 9200 1400 50  0001 L BNN
 F 2 "Capacitor_SMD:C_0603_1608Metric" H 9200 1300 50  0001 L BNN
@@
 $EndComp
 $Comp
-L power:GND #PWR?
+L power:GND #PWR011
 U 1 1 5C57129D
 P 8275 2075
-F 0 "#PWR?" H 8275 1825 50  0001 C CNN
+F 0 "#PWR011" H 8275 1825 50  0001 C CNN
 F 1 "GND" H 8275 1925 50  0000 C CNN
 F 2 "" H 8275 2075 50  0001 C CNN
@@
 $EndComp
 $Comp
-L power:GND #PWR?
+L power:GND #PWR012
 U 1 1 5C5712A3
 P 9950 2075
-F 0 "#PWR?" H 9950 1825 50  0001 C CNN
+F 0 "#PWR012" H 9950 1825 50  0001 C CNN
 F 1 "GND" H 9950 1925 50  0000 C CNN
 F 2 "" H 9950 2075 50  0001 C CNN
@@
 	9525 1600 9950 1600
 $Comp
-L custom:RMCF0603FT4K70 R?
+L custom:RMCF0603FT4K70 R10
 U 1 1 5C5712B4
 P 9525 2075
-F 0 "R?" H 9600 2050 50  0000 L BNN
+F 0 "R10" H 9600 2050 50  0000 L BNN
 F 1 "RMCF0603FT4K70" H 8825 1675 50  0001 L BNN
 F 2 "Resistor_SMD:R_0603_1608Metric" H 8825 1575 50  0001 L BNN
@@
 Connection ~ 9525 1700
 $Comp
-L power:GND #PWR?
+L power:GND #PWR014
 U 1 1 5C5712CA
 P 9525 2700
-F 0 "#PWR?" H 9525 2450 50  0001 C CNN
+F 0 "#PWR014" H 9525 2450 50  0001 C CNN
 F 1 "GND" H 9525 2550 50  0000 C CNN
 F 2 "" H 9525 2700 50  0001 C CNN
@@
 1V8 LDO
 $Comp
-L power:+5V #PWR?
+L power:+5V #PWR05
 U 1 1 5C572245
 P 5625 1500
-F 0 "#PWR?" H 5625 1350 50  0001 C CNN
+F 0 "#PWR05" H 5625 1350 50  0001 C CNN
 F 1 "+5V" H 5625 1640 50  0000 C CNN
 F 2 "" H 5625 1500 50  0001 C CNN
@@
 Connection ~ 5625 1600
 $Comp
-L power:+5V #PWR?
+L power:+5V #PWR07
 U 1 1 5C572632
 P 8275 1500
-F 0 "#PWR?" H 8275 1350 50  0001 C CNN
+F 0 "#PWR07" H 8275 1350 50  0001 C CNN
 F 1 "+5V" H 8275 1640 50  0000 C CNN
 F 2 "" H 8275 1500 50  0001 C CNN
@@
 Connection ~ 7300 1600
 $Comp
-L power:+1V8 #PWR?
+L power:+1V8 #PWR08
 U 1 1 5C57377B
 P 9950 1500
-F 0 "#PWR?" H 9950 1350 50  0001 C CNN
+F 0 "#PWR08" H 9950 1350 50  0001 C CNN
 F 1 "+1V8" H 9950 1640 50  0000 C CNN
 F 2 "" H 9950 1500 50  0001 C CNN
@@
 Connection ~ 9950 1600
 $Comp
-L power:+3V3 #PWR?
+L power:+3V3 #PWR06
 U 1 1 5C573CCE
 P 7300 1500
-F 0 "#PWR?" H 7300 1350 50  0001 C CNN
+F 0 "#PWR06" H 7300 1350 50  0001 C CNN
 F 1 "+3V3" H 7300 1640 50  0000 C CNN
 F 2 "" H 7300 1500 50  0001 C CNN
@@
 $EndComp
 $Comp
-L custom:AZ2117 U?
+L custom:AZ2117 U3
 U 1 1 5C57714B
 P 6350 1650
-F 0 "U?" H 6100 1950 60  0000 L BNN
+F 0 "U3" H 6100 1950 60  0000 L BNN
 F 1 "AZ2117" H 6100 1850 60  0000 L BNN
 F 2 "Package_TO_SOT_SMD:SOT-223" H 6100 800 60  0001 L BNN
@@
 $EndComp
 $Comp
-L custom:AZ2117 U?
+L custom:AZ2117 U4
 U 1 1 5C577182
 P 9000 1650
-F 0 "U?" H 8750 1950 60  0000 L BNN
+F 0 "U4" H 8750 1950 60  0000 L BNN
 F 1 "AZ2117" H 8750 1850 60  0000 L BNN
 F 2 "Package_TO_SOT_SMD:SOT-223" H 8750 800 60  0001 L BNN

Commit message: automated commit
Parts:
- added U?: LMR23625CFDDAR, custom:8-PowerSOIC, symbol custom:LMR23625CFDDAR
Connections:
- net GND: now also U?.6 (AGND), U?.8 (PGND), U?.9 (PAD)
Changed lines of the file:
@@
 	1    0    0    -1
 $EndComp
+$Comp
+L custom:LMR23625CFDDAR U?
+U 1 1 5C55BD05
+P 2600 2325
+F 0 "U?" H 2300 2925 50  0000 L BNN
+F 1 "LMR23625CFDDAR" H 2300 2825 50  0000 L BNN
+F 2 "custom:8-PowerSOIC" H 2550 2375 50  0001 L BNN
+F 3 "/home/dj/datasheets/lmr23625.pdf" H 2100 1175 50  0001 L BNN
+	1    2600 2325
+	1    0    0    -1
+$EndComp
+$Comp
+L power:GND #PWR?
+U 1 1 5C55C2F7
+P 2650 2975
+F 0 "#PWR?" H 2650 2725 50  0001 C CNN
+F 1 "GND" H 2650 2825 50  0000 C CNN
+F 2 "" H 2650 2975 50  0001 C CNN
+F 3 "" H 2650 2975 50  0001 C CNN
+	1    2650 2975
+	1    0    0    -1
+$EndComp
+Wire Wire Line
+	2650 2975 2650 2925
+Wire Wire Line
+	2650 2925 2550 2925
+Wire Wire Line
+	2450 2925 2450 2875
+Connection ~ 2650 2925
+Wire Wire Line
+	2650 2925 2650 2875
+Wire Wire Line
+	2550 2875 2550 2925
+Connection ~ 2550 2925
+Wire Wire Line
+	2550 2925 2450 2925
 $EndSCHEMATC

Commit message: automated commit
Parts:
- added C?: CL10B104KO8NNNC, Capacitor_SMD:C_0603_1608Metric, symbol custom:CL10B104KO8NNNC
- added C?: NP_C_0603, Capacitor_SMD:C_0603_1608Metric, symbol custom:NP_C_0603
Connections:
- net labels added: VDD_BAT
- wire segments 40 -> 55
Changed lines of the file:
@@
 Wire Wire Line
 	2550 2925 2450 2925
+$Comp
+L custom:CL10B104KO8NNNC C?
+U 1 1 5C5383E5
+P 3200 2125
+F 0 "C?" H 3350 2225 50  0000 L BNN
+F 1 "CL10B104KO8NNNC" H 2250 1675 50  0001 L BNN
+F 2 "Capacitor_SMD:C_0603_1608Metric" H 2250 1575 50  0001 L BNN
+F 3 "datasheets/CL10B104KO8NNNC.pdf" H 2250 1475 50  0001 L BNN
+F 4 "0.1uF" H 3350 2125 50  0000 L BNN "Capacitance"
+F 5 "16V" H 3350 2025 50  0000 L BNN "Rating"
+	1    3200 2125
+	1    0    0    -1
+$EndComp
+Wire Wire Line
+	875  1975 875  1925
+Wire Wire Line
+	875  1925 1375 1925
+Wire Wire Line
+	1375 1975 1375 1925
+Connection ~ 1375 1925
+Wire Wire Line
+	1375 1925 2200 1925
+$Comp
+L power:GND #PWR?
+U 1 1 5C53B227
+P 875 2325
+F 0 "#PWR?" H 875 2075 50  0001 C CNN
+F 1 "GND" H 875 2175 50  0000 C CNN
+F 2 "" H 875 2325 50  0001 C CNN
+F 3 "" H 875 2325 50  0001 C CNN
+	1    875  2325
+	1    0    0    -1
+$EndComp
+Wire Wire Line
+	875  2325 875  2275
+$Comp
+L power:GND #PWR?
+U 1 1 5C53BD04
+P 1375 2325
+F 0 "#PWR?" H 1375 2075 50  0001 C CNN
+F 1 "GND" H 1375 2175 50  0000 C CNN
+F 2 "" H 1375 2325 50  0001 C CNN
+F 3 "" H 1375 2325 50  0001 C CNN
+	1    1375 2325
+	1    0    0    -1
+$EndComp
+Wire Wire Line
+	1375 2325 1375 2275
+$Comp
+L custom:VDD_BAT #PWR?
+U 1 1 5C54089D
+P 875 1725
+AR Path="/5C5AE643/5C54089D" Ref="#PWR?"  Part="1"
+AR Path="/5C100B31/5C54089D" Ref="#PWR?"  Part="1"
+F 0 "#PWR?" H 1075 1775 50  0001 C CNN
+F 1 "VDD_BAT" H 725 1875 50  0000 L BNN
+F 2 "" H 875 1725 50  0001 C CNN
+F 3 "" H 875 1725 50  0001 C CNN
+	1    875  1725
+	1    0    0    -1
+$EndComp
+Wire Wire Line
+	875  1725 875  1925
+Connection ~ 875  1925
+Wire Wire Line
+	3050 2325 3200 2325
+Wire Wire Line
+	3700 2325 3700 2275
+Wire Wire Line
+	3200 2275 3200 2325
+Connection ~ 3200 2325
+Wire Wire Line
+	3200 2325 3700 2325
+Wire Wire Line
+	3050 1925 3200 1925
+Wire Wire Line
+	3700 1925 3700 1975
+Wire Wire Line
+	3200 1975 3200 1925
+Connection ~ 3200 1925
+Wire Wire Line
+	3200 1925 3700 1925
+$Comp
+L custom:NP_C_0603 C?
+U 1 1 5C54A84C
+P 3700 2125
+F 0 "C?" H 3750 2225 50  0000 L BNN
+F 1 "NP_C_0603" H 2750 1675 50  0001 L BNN
+F 2 "Capacitor_SMD:C_0603_1608Metric" H 2750 1575 50  0001 L BNN
+F 3 "" H 2750 1475 50  0001 L BNN
+F 4 "NP" H 3750 1975 50  0000 L BNN "NP"
+	1    3700 2125
+	1    0    0    -1
+$EndComp
 $EndSCHEMATC

Commit message: automated commit
Parts:
- gave numbers to parts that had none: 3
Changed lines of the file:
@@
 $EndComp
 $Comp
-L custom:LMR23625CFDDAR U?
+L custom:LMR23625CFDDAR U5
 U 1 1 5C55BD05
 P 2600 2325
-F 0 "U?" H 2300 2925 50  0000 L BNN
+F 0 "U5" H 2300 2925 50  0000 L BNN
 F 1 "LMR23625CFDDAR" H 2300 2825 50  0000 L BNN
 F 2 "custom:8-PowerSOIC" H 2550 2375 50  0001 L BNN
@@
 $EndComp
 $Comp
-L power:GND #PWR?
+L power:GND #PWR055
 U 1 1 5C55C2F7
 P 2650 2975
-F 0 "#PWR?" H 2650 2725 50  0001 C CNN
+F 0 "#PWR055" H 2650 2725 50  0001 C CNN
 F 1 "GND" H 2650 2825 50  0000 C CNN
 F 2 "" H 2650 2975 50  0001 C CNN
@@
 	2550 2925 2450 2925
 $Comp
-L custom:CL10B104KO8NNNC C?
+L custom:CL10B104KO8NNNC C22
 U 1 1 5C5383E5
 P 3200 2125
-F 0 "C?" H 3350 2225 50  0000 L BNN
+F 0 "C22" H 3350 2225 50  0000 L BNN
 F 1 "CL10B104KO8NNNC" H 2250 1675 50  0001 L BNN
 F 2 "Capacitor_SMD:C_0603_1608Metric" H 2250 1575 50  0001 L BNN
@@
 	1375 1925 2200 1925
 $Comp
-L power:GND #PWR?
+L power:GND #PWR031
 U 1 1 5C53B227
 P 875 2325
-F 0 "#PWR?" H 875 2075 50  0001 C CNN
+F 0 "#PWR031" H 875 2075 50  0001 C CNN
 F 1 "GND" H 875 2175 50  0000 C CNN
 F 2 "" H 875 2325 50  0001 C CNN
@@
 	875  2325 875  2275
 $Comp
-L power:GND #PWR?
+L power:GND #PWR054
 U 1 1 5C53BD04
 P 1375 2325
-F 0 "#PWR?" H 1375 2075 50  0001 C CNN
+F 0 "#PWR054" H 1375 2075 50  0001 C CNN
 F 1 "GND" H 1375 2175 50  0000 C CNN
 F 2 "" H 1375 2325 50  0001 C CNN
@@
 P 875 1725
 AR Path="/5C5AE643/5C54089D" Ref="#PWR?"  Part="1"
-AR Path="/5C100B31/5C54089D" Ref="#PWR?"  Part="1"
-F 0 "#PWR?" H 1075 1775 50  0001 C CNN
+AR Path="/5C100B31/5C54089D" Ref="#PWR028"  Part="1"
+F 0 "#PWR028" H 1075 1775 50  0001 C CNN
 F 1 "VDD_BAT" H 725 1875 50  0000 L BNN
 F 2 "" H 875 1725 50  0001 C CNN
@@
 	3200 1925 3700 1925
 $Comp
-L custom:NP_C_0603 C?
+L custom:NP_C_0603 C23
 U 1 1 5C54A84C
 P 3700 2125
-F 0 "C?" H 3750 2225 50  0000 L BNN
+F 0 "C23" H 3750 2225 50  0000 L BNN
 F 1 "NP_C_0603" H 2750 1675 50  0001 L BNN
 F 2 "Capacitor_SMD:C_0603_1608Metric" H 2750 1575 50  0001 L BNN

Commit message: automated commit
Parts:
- removed C1, C2, C3, C4: CL10B103KB8SFNC, Capacitor_SMD:C_0603_1608Metric, symbol custom:CL10B103KB8SFNC
- removed C22: CL10B104KO8NNNC, Capacitor_SMD:C_0603_1608Metric, symbol custom:CL10B104KO8NNNC
- removed C23: NP_C_0603, Capacitor_SMD:C_0603_1608Metric, symbol custom:NP_C_0603
- removed R10, R9: RMCF0603FT4K70, Resistor_SMD:R_0603_1608Metric, symbol custom:RMCF0603FT4K70
- removed R11: RMCF0603FT7K50, Resistor_SMD:R_0603_1608Metric, symbol custom:RMCF0603FT7K50
- removed R12: RMCF0603FT2K00, Resistor_SMD:R_0603_1608Metric, symbol custom:RMCF0603FT2K00
- removed U3, U4: AZ2117, Package_TO_SOT_SMD:SOT-223, symbol custom:AZ2117
- added C?: GRM188R61E225KA12D, Capacitor_SMD:C_0603_1608Metric, symbol custom:GRM188R61E225KA12D
- added C? (x2): CL10B105KA8NNNC, Capacitor_SMD:C_0603_1608Metric, symbol custom:CL10B105KA8NNNC
- added C? (x5): CL10B103KB8SFNC, Capacitor_SMD:C_0603_1608Metric, symbol custom:CL10B103KB8SFNC
- added C?: C0603C180K5RACAUTO, Capacitor_SMD:C_0603_1608Metric, symbol custom:C0603C180K5RACAUTO
- added C?: CL10B474KO8NNNC, Capacitor_SMD:C_0603_1608Metric, symbol custom:CL10B474KO8NNNC
- added C?: ESH336M035AC3AA, Capacitor_THT:CP_Radial_D5.0mm_P2.00mm, symbol custom:ESH336M035AC3AA
- added JP?: Jumper_3_Bridged12, symbol Jumper:Jumper_3_Bridged12
- added L?: NR6028T2R2N, symbol custom:NR6028T2R2N
- added R?: CR0603-JW-103ELF, 0603, symbol custom:CR0603-JW-103ELF
- added R?: RMCF0603FT40K2, 0603, symbol custom:RMCF0603FT40K2
- added R? (x2): RMCF0603FT4K70, Resistor_SMD:R_0603_1608Metric, symbol custom:RMCF0603FT4K70
- added R?: RMCF0603FT7K50, Resistor_SMD:R_0603_1608Metric, symbol custom:RMCF0603FT7K50
- added R?: RMCF0603FT2K00, Resistor_SMD:R_0603_1608Metric, symbol custom:RMCF0603FT2K00
- added U? (x2): AZ2117, Package_TO_SOT_SMD:SOT-223, symbol custom:AZ2117
Connections:
- wire segments 55 -> 80
Other:
- note added: "1.8 V @ 0.3 A\n(SUPPLIED FROM +5V)"
- note added: "3.3 V @ 0.5 A"
- note added: "5 V @ 2.5 A"
- note added: "USED RECOMMENDED VALUES\nIN DATASHEET APPNOTE"
- note added: "V_FB = 1 V\nV_OUT = 5.02 V"
- note removed: "1V8 LDO"
- note removed: "3V3 LDO"
- moved on the sheet: U5

Commit message: automated commit
Parts:
- added TP10, TP11, TP12, TP13, TP14, TP15, TP16, TP17, TP8, TP9: PTH_0.5_mm, symbol custom:PTH_0.5_mm
- gave numbers to parts that had none: 21
Connections:
- net +1V8: now also TP13.1
- net +3V3: now also TP12.1
- net +5V: now also TP14.1, TP9.1
- net VDD_BAT: now also TP8.1
- net at C3.2, L3.1, U5.1 (SW): now also TP10.1
- net at C4.2, R1.2, R2.1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: now also TP11.1
- net at R3.2, R5.1, U1.1 (ADJ): now also TP16.1
- net at R4.2, R6.1, U2.1 (ADJ): now also TP17.1
- net at C27.1, JP1.2 (C), U2.3 (VIN): now also TP15.1
Other:
- moved on the sheet: C22, C23, C25, C26, C27, C28, C4, JP1, L3, R1, R2
