File: nu.ai_motor_controller/power.sch (KiCad schematic (older format))
At the start: 32 parts, among them U1 AZ2117, U2 AZ2117, U5 LMR23625CFDDAR

Commit message: automated commit
Parts:
- JP1: footprint (none) -> Connector_PinHeader_2.54mm:PinHeader_1x03_P2.54mm_Vertical
- L3: footprint (none) -> Inductor_SMD:L_Taiyo-Yuden_NR-60xx
- R1, R2: footprint 0603 -> Resistor_SMD:R_0603_1608Metric
- TP10, TP11, TP12, TP13, TP14, TP15, TP16, TP17, TP8, TP9: footprint (none) -> TestPoint:TestPoint_THTPad_D1.0mm_Drill0.5mm
Changed lines of the file:
@@
 F 0 "R2" H 6650 2350 50  0000 L BNN
 F 1 "CR0603-JW-103ELF" V 6725 2125 50  0001 L BNN
-F 2 "0603" V 6800 2350 50  0001 L BNN
+F 2 "Resistor_SMD:R_0603_1608Metric" V 6800 2350 50  0001 L BNN
 F 3 "~/datasheets/chpreztr.pdf" V 6900 2000 50  0001 L BNN
 F 4 "10k0" V 6600 2450 50  0000 C CNN "Resistance"
@@
 F 0 "R1" H 6800 1950 50  0000 L BNN
 F 1 "RMCF0603FT40K2" H 6825 2025 50  0001 L BNN
-F 2 "0603" H 6825 2100 50  0001 L BNN
+F 2 "Resistor_SMD:R_0603_1608Metric" H 6825 2100 50  0001 L BNN
 F 3 "/home/dj/datasheets/SEI-RMCF_RMCP.pdf" H 6825 1925 50  0001 L BNN
 F 4 "40k2" V 6750 2050 50  0000 C CNN "Resistance"
@@
 F 0 "L3" V 6575 1875 50  0000 L BNN
 F 1 "NR6028T2R2N" H 6525 1550 50  0001 L BNN
-F 2 "" H 6525 1650 50  0001 L BNN
+F 2 "Inductor_SMD:L_Taiyo-Yuden_NR-60xx" H 6525 1650 50  0001 L BNN
 F 3 "/home/dj/datasheets/wound04_e.pdf" H 6525 1450 50  0001 L BNN
 F 4 "2.2uH" V 6375 1750 50  0000 L BNN "Inductance"
@@
 F 0 "JP1" H 7150 4075 50  0000 C CNN
 F 1 "Jumper_3_Bridged12" H 7050 4085 50  0001 C CNN
-F 2 "" H 7050 3975 50  0001 C CNN
+F 2 "Connector_PinHeader_2.54mm:PinHeader_1x03_P2.54mm_Vertical" H 7050 3975 50  0001 C CNN
 F 3 "~" H 7050 3975 50  0001 C CNN
 	1    7050 3975
@@
 F 0 "TP12" V 4950 4475 50  0000 L BNN
 F 1 "PTH_0.5_mm" V 4825 4550 50  0001 L BNN
-F 2 "" H 5050 4375 50  0001 L BNN
+F 2 "TestPoint:TestPoint_THTPad_D1.0mm_Drill0.5mm" H 5050 4375 50  0001 L BNN
 F 3 "~" H 5050 4375 50  0001 C CNN
 	1    4850 4375
@@
 F 0 "TP13" V 8875 4475 50  0000 L BNN
 F 1 "PTH_0.5_mm" V 8750 4550 50  0001 L BNN
-F 2 "" H 8975 4375 50  0001 L BNN
+F 2 "TestPoint:TestPoint_THTPad_D1.0mm_Drill0.5mm" H 8975 4375 50  0001 L BNN
 F 3 "~" H 8975 4375 50  0001 C CNN
 	1    8775 4375
@@
 F 0 "TP16" V 3750 5075 50  0000 L BNN
 F 1 "PTH_0.5_mm" V 3775 5150 50  0001 L BNN
-F 2 "" H 4000 4975 50  0001 L BNN
+F 2 "TestPoint:TestPoint_THTPad_D1.0mm_Drill0.5mm" H 4000 4975 50  0001 L BNN
 F 3 "~" H 4000 4975 50  0001 C CNN
 	1    3800 4975
@@
 F 0 "TP17" V 7675 5075 50  0000 L BNN
 F 1 "PTH_0.5_mm" V 7700 5150 50  0001 L BNN
-F 2 "" H 7925 4975 50  0001 L BNN
+F 2 "TestPoint:TestPoint_THTPad_D1.0mm_Drill0.5mm" H 7925 4975 50  0001 L BNN
 F 3 "~" H 7925 4975 50  0001 C CNN
 	1    7725 4975
@@
 F 0 "TP14" V 3025 4500 50  0000 L BNN
 F 1 "PTH_0.5_mm" V 3050 4575 50  0001 L BNN
-F 2 "" H 3275 4400 50  0001 L BNN
+F 2 "TestPoint:TestPoint_THTPad_D1.0mm_Drill0.5mm" H 3275 4400 50  0001 L BNN
 F 3 "~" H 3275 4400 50  0001 C CNN
 	1    3075 4400
@@
 F 0 "TP15" V 6950 4500 50  0000 L BNN
 F 1 "PTH_0.5_mm" V 6975 4575 50  0001 L BNN
-F 2 "" H 7200 4400 50  0001 L BNN
+F 2 "TestPoint:TestPoint_THTPad_D1.0mm_Drill0.5mm" H 7200 4400 50  0001 L BNN
 F 3 "~" H 7200 4400 50  0001 C CNN
 	1    7000 4400
@@
 F 0 "TP8" V 3200 1450 50  0000 L BNN
 F 1 "PTH_0.5_mm" V 3225 1525 50  0001 L BNN
-F 2 "" H 3450 1350 50  0001 L BNN
+F 2 "TestPoint:TestPoint_THTPad_D1.0mm_Drill0.5mm" H 3450 1350 50  0001 L BNN
 F 3 "~" H 3450 1350 50  0001 C CNN
 	1    3250 1350
@@
 F 0 "TP11" H 7125 2500 50  0000 L BNN
 F 1 "PTH_0.5_mm" V 7150 2475 50  0001 L BNN
-F 2 "" H 7375 2300 50  0001 L BNN
+F 2 "TestPoint:TestPoint_THTPad_D1.0mm_Drill0.5mm" H 7375 2300 50  0001 L BNN
 F 3 "~" H 7375 2300 50  0001 C CNN
 	1    7175 2300
@@
 F 0 "TP10" H 6000 2000 50  0000 L BNN
 F 1 "PTH_0.5_mm" V 6025 1975 50  0001 L BNN
-F 2 "" H 6250 1800 50  0001 L BNN
+F 2 "TestPoint:TestPoint_THTPad_D1.0mm_Drill0.5mm" H 6250 1800 50  0001 L BNN
 F 3 "~" H 6250 1800 50  0001 C CNN
 	1    6050 1800
@@
 F 0 "TP9" V 8125 1825 50  0000 L BNN
 F 1 "PTH_0.5_mm" V 8150 1900 50  0001 L BNN
-F 2 "" H 8375 1725 50  0001 L BNN
+F 2 "TestPoint:TestPoint_THTPad_D1.0mm_Drill0.5mm" H 8375 1725 50  0001 L BNN
 F 3 "~" H 8375 1725 50  0001 C CNN
 	1    8175 1725

Commit message: automated commit
Parts:
- removed TP15: PTH_0.5_mm, TestPoint:TestPoint_THTPad_D1.0mm_Drill0.5mm, symbol custom:PTH_0.5_mm
- TP10, TP11, TP12, TP13, TP14, TP16, TP17, TP8, TP9: footprint TestPoint:TestPoint_THTPad_D1.0mm_Drill0.5mm -> custom:TestPoint_THTPad_D1.0mm_Drill0.5mm
Changed lines of the file:
@@
 	7050 4825 7050 4750
-Wire Wire Line
-	7050 4450 7050 4400
 Wire Wire Line
 	7050 4300 7325 4300
@@
 F 0 "TP12" V 4950 4475 50  0000 L BNN
 F 1 "PTH_0.5_mm" V 4825 4550 50  0001 L BNN
-F 2 "TestPoint:TestPoint_THTPad_D1.0mm_Drill0.5mm" H 5050 4375 50  0001 L BNN
+F 2 "custom:TestPoint_THTPad_D1.0mm_Drill0.5mm" H 5050 4375 50  0001 L BNN
 F 3 "~" H 5050 4375 50  0001 C CNN
 	1    4850 4375
@@
 F 0 "TP13" V 8875 4475 50  0000 L BNN
 F 1 "PTH_0.5_mm" V 8750 4550 50  0001 L BNN
-F 2 "TestPoint:TestPoint_THTPad_D1.0mm_Drill0.5mm" H 8975 4375 50  0001 L BNN
+F 2 "custom:TestPoint_THTPad_D1.0mm_Drill0.5mm" H 8975 4375 50  0001 L BNN
 F 3 "~" H 8975 4375 50  0001 C CNN
 	1    8775 4375
@@
 F 0 "TP16" V 3750 5075 50  0000 L BNN
 F 1 "PTH_0.5_mm" V 3775 5150 50  0001 L BNN
-F 2 "TestPoint:TestPoint_THTPad_D1.0mm_Drill0.5mm" H 4000 4975 50  0001 L BNN
+F 2 "custom:TestPoint_THTPad_D1.0mm_Drill0.5mm" H 4000 4975 50  0001 L BNN
 F 3 "~" H 4000 4975 50  0001 C CNN
 	1    3800 4975
@@
 F 0 "TP17" V 7675 5075 50  0000 L BNN
 F 1 "PTH_0.5_mm" V 7700 5150 50  0001 L BNN
-F 2 "TestPoint:TestPoint_THTPad_D1.0mm_Drill0.5mm" H 7925 4975 50  0001 L BNN
+F 2 "custom:TestPoint_THTPad_D1.0mm_Drill0.5mm" H 7925 4975 50  0001 L BNN
 F 3 "~" H 7925 4975 50  0001 C CNN
 	1    7725 4975
@@
 F 0 "TP14" V 3025 4500 50  0000 L BNN
 F 1 "PTH_0.5_mm" V 3050 4575 50  0001 L BNN
-F 2 "TestPoint:TestPoint_THTPad_D1.0mm_Drill0.5mm" H 3275 4400 50  0001 L BNN
+F 2 "custom:TestPoint_THTPad_D1.0mm_Drill0.5mm" H 3275 4400 50  0001 L BNN
 F 3 "~" H 3275 4400 50  0001 C CNN
 	1    3075 4400
@@
 Wire Wire Line
 	3075 4400 3125 4400
-$Comp
-L custom:PTH_0.5_mm TP?
-U 1 1 5CC056A4
-P 7000 4400
-AR Path="/5C5AE643/5CC056A4" Ref="TP?"  Part="1"
-AR Path="/5C100B31/5CC056A4" Ref="TP15"  Part="1"
-F 0 "TP15" V 6950 4500 50  0000 L BNN
-F 1 "PTH_0.5_mm" V 6975 4575 50  0001 L BNN
-F 2 "TestPoint:TestPoint_THTPad_D1.0mm_Drill0.5mm" H 7200 4400 50  0001 L BNN
-F 3 "~" H 7200 4400 50  0001 C CNN
-	1    7000 4400
-	0    -1   1    0
-$EndComp
-Wire Wire Line
-	7000 4400 7050 4400
 Connection ~ 3125 4400
 Wire Wire Line
 	3125 4300 3125 4400
-Connection ~ 7050 4400
-Wire Wire Line
-	7050 4300 7050 4400
 $Comp
 L custom:PTH_0.5_mm TP?
@@
 F 0 "TP8" V 3200 1450 50  0000 L BNN
 F 1 "PTH_0.5_mm" V 3225 1525 50  0001 L BNN
-F 2 "TestPoint:TestPoint_THTPad_D1.0mm_Drill0.5mm" H 3450 1350 50  0001 L BNN
+F 2 "custom:TestPoint_THTPad_D1.0mm_Drill0.5mm" H 3450 1350 50  0001 L BNN
 F 3 "~" H 3450 1350 50  0001 C CNN
 	1    3250 1350
@@
 F 0 "TP11" H 7125 2500 50  0000 L BNN
 F 1 "PTH_0.5_mm" V 7150 2475 50  0001 L BNN
-F 2 "TestPoint:TestPoint_THTPad_D1.0mm_Drill0.5mm" H 7375 2300 50  0001 L BNN
+F 2 "custom:TestPoint_THTPad_D1.0mm_Drill0.5mm" H 7375 2300 50  0001 L BNN
 F 3 "~" H 7375 2300 50  0001 C CNN
 	1    7175 2300
@@
 F 0 "TP10" H 6000 2000 50  0000 L BNN
 F 1 "PTH_0.5_mm" V 6025 1975 50  0001 L BNN
-F 2 "TestPoint:TestPoint_THTPad_D1.0mm_Drill0.5mm" H 6250 1800 50  0001 L BNN
+F 2 "custom:TestPoint_THTPad_D1.0mm_Drill0.5mm" H 6250 1800 50  0001 L BNN
 F 3 "~" H 6250 1800 50  0001 C CNN
 	1    6050 1800
@@
 F 0 "TP9" V 8125 1825 50  0000 L BNN
 F 1 "PTH_0.5_mm" V 8150 1900 50  0001 L BNN
-F 2 "TestPoint:TestPoint_THTPad_D1.0mm_Drill0.5mm" H 8375 1725 50  0001 L BNN
+F 2 "custom:TestPoint_THTPad_D1.0mm_Drill0.5mm" H 8375 1725 50  0001 L BNN
 F 3 "~" H 8375 1725 50  0001 C CNN
 	1    8175 1725
@@
 Wire Wire Line
 	8125 1725 8125 1850
+Wire Wire Line
+	7050 4300 7050 4450
 $EndSCHEMATC

Commit message: automated commit
Other:
- note added: "1.8 V @ 0.3 A\n(WHEN SUPPLIED FROM +5V)"
- note removed: "1.8 V @ 0.3 A\n(SUPPLIED FROM +5V)"
- note removed: "USED RECOMMENDED VALUES\nIN DATASHEET APPNOTE"
Changed lines of the file:
@@
 	8300 5400 8300 5325
 Text Notes 7800 3825 0    50   ~ 0
-1.8 V @ 0.3 A\n(SUPPLIED FROM +5V)
+1.8 V @ 0.3 A\n(WHEN SUPPLIED FROM +5V)
 $Comp
 L power:+5V #PWR08
@@
 	1    0    0    -1
 $EndComp
-Text Notes 6800 1750 0    50   ~ 0
-USED RECOMMENDED VALUES\nIN DATASHEET APPNOTE
 $Comp
 L Jumper:Jumper_3_Bridged12 JP1
