File: nu.ai_motor_controller/battery.sch (KiCad schematic (older format))
At the start: 38 parts, among them J12 XT60_RA_MALE, J13 S4B-XH-A, J14 NP_Screw_Terminal_01x02, J15 XT60_RA_MALE, J16 S4B-XH-A, J17 S4B-XH-A, J18 XT60_RA_FEMALE, Q1 IRF9540N, Q2 SSM3K35AMFV, SW2 TACTILE_SWITCH, SW3 TACTILE_SWITCH

Commit message: automated commit
Parts:
- R20, R21, R22, R23, R24, R25, R26, R29, R30, R31: footprint 0603 -> Resistor_SMD:R_0603_1608Metric
- TP1, TP2, TP3, TP4, TP5, TP52, TP53, TP54, TP55, TP56, TP6, TP7: footprint (none) -> TestPoint:TestPoint_THTPad_D1.0mm_Drill0.5mm
Other:
- note added: "BATTERY PORT"
- note added: "CHARGING PORT"
Changed lines of the file:
@@
 F 0 "TP1" V 9300 3375 50  0000 L BNN
 F 1 "PTH_0.5_mm" V 9250 3300 50  0001 L BNN
-F 2 "" H 9475 3125 50  0001 L BNN
+F 2 "TestPoint:TestPoint_THTPad_D1.0mm_Drill0.5mm" H 9475 3125 50  0001 L BNN
 F 3 "~" H 9475 3125 50  0001 C CNN
 	1    9275 3125
@@
 F 0 "TP2" V 9300 3475 50  0000 L BNN
 F 1 "PTH_0.5_mm" V 9250 3400 50  0001 L BNN
-F 2 "" H 9475 3225 50  0001 L BNN
+F 2 "TestPoint:TestPoint_THTPad_D1.0mm_Drill0.5mm" H 9475 3225 50  0001 L BNN
 F 3 "~" H 9475 3225 50  0001 C CNN
 	1    9275 3225
@@
 F 0 "TP3" V 9300 3575 50  0000 L BNN
 F 1 "PTH_0.5_mm" V 9250 3500 50  0001 L BNN
-F 2 "" H 9475 3325 50  0001 L BNN
+F 2 "TestPoint:TestPoint_THTPad_D1.0mm_Drill0.5mm" H 9475 3325 50  0001 L BNN
 F 3 "~" H 9475 3325 50  0001 C CNN
 	1    9275 3325
@@
 F 0 "TP4" V 9300 3675 50  0000 L BNN
 F 1 "PTH_0.5_mm" V 9250 3600 50  0001 L BNN
-F 2 "" H 9475 3425 50  0001 L BNN
+F 2 "TestPoint:TestPoint_THTPad_D1.0mm_Drill0.5mm" H 9475 3425 50  0001 L BNN
 F 3 "~" H 9475 3425 50  0001 C CNN
 	1    9275 3425
@@
 F 0 "R20" H 5825 2975 50  0000 L BNN
 F 1 "RC0603JR-071KL" H 5850 2850 50  0001 L BNN
-F 2 "0603" H 5850 2925 50  0001 L BNN
+F 2 "Resistor_SMD:R_0603_1608Metric" H 5850 2925 50  0001 L BNN
 F 3 "~/datasheets/PYu-RC_Group_51_RoHS_L_10.pdf" H 5715 2935 50  0001 C CNN
 F 4 "1k0" V 5775 2925 50  0000 C CNN "Resistance"
@@
 	1    0    0    -1
 $EndComp
-Text Notes 725  2950 0    50   ~ 0
+Text Notes 1375 1850 0    50   ~ 0
 INDICATE POS AND NEG\nON SILKSCREEN
 $Comp
@@
 F 0 "R21" H 4725 2625 50  0000 L BNN
 F 1 "CR0603-JW-103ELF" V 4775 2250 50  0001 L BNN
-F 2 "0603" V 4850 2475 50  0001 L BNN
+F 2 "Resistor_SMD:R_0603_1608Metric" V 4850 2475 50  0001 L BNN
 F 3 "~/datasheets/chpreztr.pdf" V 4950 2125 50  0001 L BNN
 F 4 "10k0" V 4650 2575 50  0000 C CNN "Resistance"
@@
 F 0 "R25" V 7475 3825 50  0000 L BNN
 F 1 "CR0603-JW-103ELF" V 7625 3375 50  0001 L BNN
-F 2 "0603" V 7700 3600 50  0001 L BNN
+F 2 "Resistor_SMD:R_0603_1608Metric" V 7700 3600 50  0001 L BNN
 F 3 "~/datasheets/chpreztr.pdf" V 7800 3250 50  0001 L BNN
 F 4 "10k0" V 7500 3700 50  0000 C CNN "Resistance"
@@
 F 0 "R26" V 7575 3825 50  0000 L BNN
 F 1 "CR0603-JW-103ELF" V 7725 3375 50  0001 L BNN
-F 2 "0603" V 7800 3600 50  0001 L BNN
+F 2 "Resistor_SMD:R_0603_1608Metric" V 7800 3600 50  0001 L BNN
 F 3 "~/datasheets/chpreztr.pdf" V 7900 3250 50  0001 L BNN
 F 4 "10k0" V 7600 3700 50  0000 C CNN "Resistance"
@@
 F 0 "R24" V 7375 3825 50  0000 L BNN
 F 1 "CR0603-JW-103ELF" V 7525 3375 50  0001 L BNN
-F 2 "0603" V 7600 3600 50  0001 L BNN
+F 2 "Resistor_SMD:R_0603_1608Metric" V 7600 3600 50  0001 L BNN
 F 3 "~/datasheets/chpreztr.pdf" V 7700 3250 50  0001 L BNN
 F 4 "10k0" V 7400 3700 50  0000 C CNN "Resistance"
@@
 F 0 "R29" V 7375 4600 50  0000 L BNN
 F 1 "RC0603JR-071KL" H 7475 4400 50  0001 L BNN
-F 2 "0603" H 7475 4475 50  0001 L BNN
+F 2 "Resistor_SMD:R_0603_1608Metric" H 7475 4475 50  0001 L BNN
 F 3 "~/datasheets/PYu-RC_Group_51_RoHS_L_10.pdf" H 7340 4485 50  0001 C CNN
 F 4 "1k0" V 7400 4475 50  0000 C CNN "Resistance"
@@
 F 0 "R30" V 7475 4600 50  0000 L BNN
 F 1 "RC0603JR-071KL" H 7575 4400 50  0001 L BNN
-F 2 "0603" H 7575 4475 50  0001 L BNN
+F 2 "Resistor_SMD:R_0603_1608Metric" H 7575 4475 50  0001 L BNN
 F 3 "~/datasheets/PYu-RC_Group_51_RoHS_L_10.pdf" H 7440 4485 50  0001 C CNN
 F 4 "1k0" V 7500 4475 50  0000 C CNN "Resistance"
@@
 F 0 "R31" V 7575 4600 50  0000 L BNN
 F 1 "RC0603JR-071KL" H 7675 4400 50  0001 L BNN
-F 2 "0603" H 7675 4475 50  0001 L BNN
+F 2 "Resistor_SMD:R_0603_1608Metric" H 7675 4475 50  0001 L BNN
 F 3 "~/datasheets/PYu-RC_Group_51_RoHS_L_10.pdf" H 7540 4485 50  0001 C CNN
 F 4 "1k0" V 7600 4475 50  0000 C CNN "Resistance"
@@
 F 0 "TP5" V 6875 4250 50  0000 L BNN
 F 1 "PTH_0.5_mm" V 6875 4475 50  0001 L BNN
-F 2 "" H 7100 4300 50  0001 L BNN
+F 2 "TestPoint:TestPoint_THTPad_D1.0mm_Drill0.5mm" H 7100 4300 50  0001 L BNN
 F 3 "~" H 7100 4300 50  0001 C CNN
 	1    6900 4300
@@
 F 0 "TP6" V 6975 4250 50  0000 L BNN
 F 1 "PTH_0.5_mm" V 6975 4475 50  0001 L BNN
-F 2 "" H 7200 4300 50  0001 L BNN
+F 2 "TestPoint:TestPoint_THTPad_D1.0mm_Drill0.5mm" H 7200 4300 50  0001 L BNN
 F 3 "~" H 7200 4300 50  0001 C CNN
 	1    7000 4300
@@
 F 0 "TP7" V 7075 4250 50  0000 L BNN
 F 1 "PTH_0.5_mm" V 7075 4475 50  0001 L BNN
-F 2 "" H 7300 4300 50  0001 L BNN
+F 2 "TestPoint:TestPoint_THTPad_D1.0mm_Drill0.5mm" H 7300 4300 50  0001 L BNN
 F 3 "~" H 7300 4300 50  0001 C CNN
 	1    7100 4300
@@
 F 0 "R22" H 3075 3275 50  0000 L BNN
 F 1 "CR0603-JW-103ELF" V 3125 2900 50  0001 L BNN
-F 2 "0603" V 3200 3125 50  0001 L BNN
+F 2 "Resistor_SMD:R_0603_1608Metric" V 3200 3125 50  0001 L BNN
 F 3 "~/datasheets/chpreztr.pdf" V 3300 2775 50  0001 L BNN
 F 4 "10k0" V 3000 3225 50  0000 C CNN "Resistance"
@@
 F 0 "R23" H 5075 3275 50  0000 L BNN
 F 1 "CR0603-JW-103ELF" V 5125 2900 50  0001 L BNN
-F 2 "0603" V 5200 3125 50  0001 L BNN
+F 2 "Resistor_SMD:R_0603_1608Metric" V 5200 3125 50  0001 L BNN
 F 3 "~/datasheets/chpreztr.pdf" V 5300 2775 50  0001 L BNN
 F 4 "10k0" V 5000 3225 50  0000 C CNN "Resistance"
@@
 F 0 "TP53" H 2225 2425 50  0000 L BNN
 F 1 "PTH_0.5_mm" V 2275 2425 50  0001 L BNN
-F 2 "" H 2500 2250 50  0001 L BNN
+F 2 "TestPoint:TestPoint_THTPad_D1.0mm_Drill0.5mm" H 2500 2250 50  0001 L BNN
 F 3 "~" H 2500 2250 50  0001 C CNN
 	1    2300 2250
@@
 F 0 "TP54" H 3025 2425 50  0000 L BNN
 F 1 "PTH_0.5_mm" V 3075 2425 50  0001 L BNN
-F 2 "" H 3300 2250 50  0001 L BNN
+F 2 "TestPoint:TestPoint_THTPad_D1.0mm_Drill0.5mm" H 3300 2250 50  0001 L BNN
 F 3 "~" H 3300 2250 50  0001 C CNN
 	1    3100 2250
@@
 F 0 "TP52" V 6800 2325 50  0000 L BNN
 F 1 "PTH_0.5_mm" V 6825 2400 50  0001 L BNN
-F 2 "" H 7050 2225 50  0001 L BNN
+F 2 "TestPoint:TestPoint_THTPad_D1.0mm_Drill0.5mm" H 7050 2225 50  0001 L BNN
 F 3 "~" H 7050 2225 50  0001 C CNN
 	1    6850 2225
@@
 F 0 "TP56" H 4425 4225 50  0000 L BNN
 F 1 "PTH_0.5_mm" V 4475 4225 50  0001 L BNN
-F 2 "" H 4700 4050 50  0001 L BNN
+F 2 "TestPoint:TestPoint_THTPad_D1.0mm_Drill0.5mm" H 4700 4050 50  0001 L BNN
 F 3 "~" H 4700 4050 50  0001 C CNN
 	1    4500 4050
@@
 F 0 "TP55" V 4975 2800 50  0000 L BNN
 F 1 "PTH_0.5_mm" V 5025 2875 50  0001 L BNN
-F 2 "" H 5250 2700 50  0001 L BNN
+F 2 "TestPoint:TestPoint_THTPad_D1.0mm_Drill0.5mm" H 5250 2700 50  0001 L BNN
 F 3 "~" H 5250 2700 50  0001 C CNN
 	1    5050 2700
@@
 Wire Wire Line
 	5000 2800 5000 3075
+Text Notes 1125 2450 0    50   ~ 0
+BATTERY PORT
+Text Notes 1125 2975 0    50   ~ 0
+BATTERY PORT
+Text Notes 1050 3475 0    50   ~ 0
+CHARGING PORT
 $EndSCHEMATC

Commit message: automated commit
Parts:
- J13, J16, J17: footprint Connector_PinHeader_2.54mm:PinHeader_1x04_P2.54mm_Horizontal -> custom:X4B-XH-A
- J14: footprint (none) -> custom:TERMINAL_BLOCK_1x2
- Q1: footprint Package_TO_SOT_THT:TO-220-3_Vertical -> Package_TO_SOT_THT:TO-220-3_Horizontal_TabDown
- SW2, SW3: footprint (none) -> custom:TACTILE_SWITCH
Connections:
- net GND: now also J17.1 (Pin_1); no longer J17.4 (Pin_4)
- net TAP_0: now also J17.2 (Pin_2); no longer J17.3 (Pin_3)
- net TAP_1: now also J17.3 (Pin_3); no longer J17.2 (Pin_2)
- net TAP_2: now also J13.1 (Pin_1), J16.1 (Pin_1), J17.4 (Pin_4), TP1.1
- net VDD_BAT: no longer D8.4 (CH4)
- removed net TAP_3: J13.1 (Pin_1), J16.1 (Pin_1), J17.1 (Pin_1), TP1.1
- no-connect marks 1 -> 2
Other:
- note added: "BATTERY\nTAP"
- note added: "CHARGING\nTAP"
- note removed: "BATTERY\nTAPS"
- moved on the sheet: TP52
Changed lines of the file:
@@
 F 0 "J16" H 10225 4125 50  0000 L BNN
 F 1 "S4B-XH-A" H 10025 3625 50  0000 L BNN
-F 2 "Connector_PinHeader_2.54mm:PinHeader_1x04_P2.54mm_Horizontal" H 10125 3525 50  0001 L BNN
+F 2 "custom:X4B-XH-A" H 10125 3525 50  0001 L BNN
 F 3 "eXH.pdf" H 10125 3425 50  0001 L BNN
 	1    10125 3925
@@
 $EndComp
 Text Notes 10200 4025 0    50   ~ 0
-BATTERY\nTAPS
+BATTERY\nTAP
 $Comp
 L custom:S4B-XH-A J?
@@
 F 0 "J17" H 10225 4825 50  0000 L BNN
 F 1 "S4B-XH-A" H 10025 4325 50  0000 L BNN
-F 2 "Connector_PinHeader_2.54mm:PinHeader_1x04_P2.54mm_Horizontal" H 10125 4225 50  0001 L BNN
+F 2 "custom:X4B-XH-A" H 10125 4225 50  0001 L BNN
 F 3 "eXH.pdf" H 10125 4125 50  0001 L BNN
 	1    10125 4625
@@
 F 0 "J13" H 10225 3425 50  0000 L BNN
 F 1 "S4B-XH-A" H 10025 2925 50  0000 L BNN
-F 2 "Connector_PinHeader_2.54mm:PinHeader_1x04_P2.54mm_Horizontal" H 10125 2825 50  0001 L BNN
+F 2 "custom:X4B-XH-A" H 10125 2825 50  0001 L BNN
 F 3 "eXH.pdf" H 10125 2725 50  0001 L BNN
 	1    10125 3225
@@
 $EndComp
 Wire Wire Line
-	9925 4525 9350 4525
-Wire Wire Line
-	9350 4525 9350 3825
-Wire Wire Line
 	9350 3125 9925 3125
 Wire Wire Line
@@
 Wire Wire Line
 	9350 3825 9350 3125
-Wire Wire Line
-	9925 4625 9450 4625
-Wire Wire Line
-	9450 4625 9450 3925
-Wire Wire Line
-	9925 4725 9550 4725
-Wire Wire Line
-	9550 4725 9550 4025
-Wire Wire Line
-	9925 4825 9650 4825
-Wire Wire Line
-	9650 4825 9650 4125
 Wire Wire Line
 	9925 3925 9450 3925
@@
 	1    0    0    -1
 $EndComp
-Connection ~ 9650 4825
 Connection ~ 9650 4125
-Connection ~ 9550 4025
 Connection ~ 9450 3925
 Connection ~ 9350 3825
@@
 F 0 "J14" H 7675 2325 50  0000 C CNN
 F 1 "NP_Screw_Terminal_01x02" H 8250 2175 50  0000 C CNN
-F 2 "" H 7675 2225 50  0001 C CNN
+F 2 "custom:TERMINAL_BLOCK_1x2" H 7675 2225 50  0001 C CNN
 F 3 "~" H 7675 2225 50  0001 C CNN
 	1    7675 2225
@@
 Connection ~ 9450 3225
 Connection ~ 9550 3325
-Wire Wire Line
-	9650 4825 9650 4900
 Connection ~ 9650 3425
 Wire Wire Line
@@
 L custom:VDD_BAT #PWR056
 U 1 1 5C5B04A6
-P 6975 2125
-F 0 "#PWR056" H 7175 2175 50  0001 C CNN
-F 1 "VDD_BAT" H 6825 2275 50  0000 L BNN
-F 2 "" H 6975 2125 50  0001 C CNN
-F 3 "" H 6975 2125 50  0001 C CNN
-	1    6975 2125
-	1    0    0    -1
-$EndComp
-Wire Wire Line
-	6975 2225 6975 2125
+P 7425 2125
+F 0 "#PWR056" H 7625 2175 50  0001 C CNN
+F 1 "VDD_BAT" H 7275 2275 50  0000 L BNN
+F 2 "" H 7425 2125 50  0001 C CNN
+F 3 "" H 7425 2125 50  0001 C CNN
+	1    7425 2125
+	1    0    0    -1
+$EndComp
+Wire Wire Line
+	7425 2225 7425 2125
 Wire Wire Line
 	2025 2875 2400 2875
@@
 $EndComp
 Text Label 9625 3125 0    50   ~ 0
-TAP_3
+TAP_2
 Text Label 9625 3325 0    50   ~ 0
 TAP_0
@@
 F 0 "SW3" H 3075 4200 60  0000 L BNN
 F 1 "TACTILE_SWITCH" H 2900 3900 60  0001 L BNN
-F 2 "" H 3250 4200 60  0001 C CNN
+F 2 "custom:TACTILE_SWITCH" H 3250 4200 60  0001 C CNN
 F 3 "" H 3250 4200 60  0001 C CNN
 	1    3250 4050
@@
 F 0 "SW2" H 3925 2950 60  0000 L BNN
 F 1 "TACTILE_SWITCH" H 3750 2650 60  0001 L BNN
-F 2 "" H 4100 2950 60  0001 C CNN
+F 2 "custom:TACTILE_SWITCH" H 4100 2950 60  0001 C CNN
 F 3 "" H 4100 2950 60  0001 C CNN
 	1    4100 2800
@@
 F 0 "Q1" V 5225 2250 50  0000 L CNN
 F 1 "IRF9540N" V 5150 1975 50  0000 L CNN
-F 2 "Package_TO_SOT_THT:TO-220-3_Vertical" H 5200 2375 50  0001 L CIN
+F 2 "Package_TO_SOT_THT:TO-220-3_Horizontal_TabDown" H 5200 2375 50  0001 L CIN
 F 3 "/home/dj/datasheets/irf9540n.pdf" H 5200 2250 50  0001 L BNN
 	1    5000 2450
@@
 Connection ~ 4350 2800
 Wire Wire Line
-	4450 3250 4825 3250
-Text Label 4825 3250 2    50   ~ 0
-TERM_POS
-Text Label 7050 2225 0    50   ~ 0
-TERM_POS
-Wire Wire Line
-	6975 2225 7475 2225
+	7425 2225 7475 2225
 NoConn ~ 3750 3250
 Connection ~ 3500 4000
@@
 L custom:PTH_0.5_mm TP52
 U 1 1 5CB97973
-P 6850 2225
-F 0 "TP52" V 6800 2325 50  0000 L BNN
-F 1 "PTH_0.5_mm" V 6825 2400 50  0001 L BNN
-F 2 "TestPoint:TestPoint_THTPad_D1.0mm_Drill0.5mm" H 7050 2225 50  0001 L BNN
-F 3 "~" H 7050 2225 50  0001 C CNN
-	1    6850 2225
+P 7300 2225
+F 0 "TP52" V 7250 2325 50  0000 L BNN
+F 1 "PTH_0.5_mm" V 7275 2400 50  0001 L BNN
+F 2 "TestPoint:TestPoint_THTPad_D1.0mm_Drill0.5mm" H 7500 2225 50  0001 L BNN
+F 3 "~" H 7500 2225 50  0001 C CNN
+	1    7300 2225
 	0    -1   1    0
 $EndComp
 Wire Wire Line
-	6850 2225 6975 2225
-Connection ~ 6975 2225
+	7300 2225 7425 2225
+Connection ~ 7425 2225
 $Comp
 L custom:PTH_0.5_mm TP56
@@
 Text Notes 1050 3475 0    50   ~ 0
 CHARGING PORT
+Text Notes 10200 3350 0    50   ~ 0
+BATTERY\nTAP
+Text Notes 10200 4750 0    50   ~ 0
+CHARGING\nTAP
+Wire Wire Line
+	9650 4125 9650 4525
+Wire Wire Line
+	9350 4825 9925 4825
+Wire Wire Line
+	9350 3825 9350 4825
+Wire Wire Line
+	9925 4525 9650 4525
+Connection ~ 9650 4525
+Wire Wire Line
+	9650 4525 9650 4900
+Wire Wire Line
+	9550 4025 9550 4625
+Wire Wire Line
+	9550 4625 9925 4625
+Connection ~ 9550 4025
+Wire Wire Line
+	9925 4725 9450 4725
+Wire Wire Line
+	9450 3925 9450 4725
+NoConn ~ 4450 3250
 $EndSCHEMATC

Commit message: automated commit
Connections:
- net at F2.2, Q1.3 (S), R21.1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: now also D8.6 (CH3); no longer D8.1 (CH1)
- net at Q1.1 (G), R21.2, R23.1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: now also D8.1 (CH1); no longer D8.6 (CH3)
Changed lines of the file:
@@
 L power:GND #PWR064
 U 1 1 5C90FE16
-P 4525 3400
-F 0 "#PWR064" H 4525 3150 50  0001 C CNN
-F 1 "GND" H 4525 3250 50  0000 C CNN
-F 2 "" H 4525 3400 50  0001 C CNN
-F 3 "" H 4525 3400 50  0001 C CNN
-	1    4525 3400
-	1    0    0    -1
+P 3675 3400
+F 0 "#PWR064" H 3675 3150 50  0001 C CNN
+F 1 "GND" H 3675 3250 50  0000 C CNN
+F 2 "" H 3675 3400 50  0001 C CNN
+F 3 "" H 3675 3400 50  0001 C CNN
+	1    3675 3400
+	-1   0    0    -1
 $EndComp
 Connection ~ 2400 2350
 Connection ~ 5775 2350
 Wire Wire Line
-	4525 3400 4525 3350
+	3675 3400 3675 3350
 Text Notes 3775 3700 0    50   ~ 0
 PLACE TVS NEAR\nBUTTON PINS
@@
 F 3 "/home/dj/datasheets/SMS05T1-D.PDF" H 4600 3150 50  0001 C CNN
 	1    4100 3350
-	1    0    0    -1
+	-1   0    0    -1
 $EndComp
 Wire Wire Line
-	4525 3350 4450 3350
+	3675 3350 3750 3350
 Wire Wire Line
 	3700 3150 3750 3150

Commit message: automated commit
Connections:
- net GND: now also J17.4 (Pin_4); no longer J17.1 (Pin_1)
- net TAP_0: now also J17.3 (Pin_3); no longer J17.2 (Pin_2)
- net TAP_1: now also J17.2 (Pin_2); no longer J17.3 (Pin_3)
- net TAP_2: now also J17.1 (Pin_1); no longer J17.4 (Pin_4)
Changed lines of the file:
@@
 CHARGING\nTAP
 Wire Wire Line
-	9650 4125 9650 4525
-Wire Wire Line
-	9350 4825 9925 4825
-Wire Wire Line
-	9350 3825 9350 4825
-Wire Wire Line
-	9925 4525 9650 4525
-Connection ~ 9650 4525
-Wire Wire Line
-	9650 4525 9650 4900
-Wire Wire Line
-	9550 4025 9550 4625
-Wire Wire Line
-	9550 4625 9925 4625
+	9350 3825 9350 4525
 Connection ~ 9550 4025
 Wire Wire Line
-	9925 4725 9450 4725
+	9450 3925 9450 4625
+NoConn ~ 4450 3250
 Wire Wire Line
-	9450 3925 9450 4725
-NoConn ~ 4450 3250
+	9925 4525 9350 4525
+Wire Wire Line
+	9925 4625 9550 4625
+Wire Wire Line
+	9550 4625 9450 4625
+Wire Wire Line
+	9925 4725 9550 4725
+Wire Wire Line
+	9925 4825 9650 4825
+Wire Wire Line
+	9650 4125 9650 4825
+Connection ~ 9650 4825
+Wire Wire Line
+	9650 4825 9650 4900
+Wire Wire Line
+	9550 4025 9550 4725
 $EndSCHEMATC

Commit message: automated commit
Parts:
- Q1: footprint Package_TO_SOT_THT:TO-220-3_Horizontal_TabDown -> custom:TO-220-3_Horizontal_TabDown
Connections:
- net TAP_2: now also F2.1, J12.2 (Pin_2), J15.2 (Pin_2), J18.1 (Pin_1), TP53.1
Other:
- moved on the sheet: J12, J15, J18
Changed lines of the file:
@@
 	7475 2325 7425 2325
 Wire Wire Line
-	2025 3400 2400 3400
+	1700 3400 2400 3400
 $Comp
 L custom:PTH_0.5_mm TP1
@@
 	2225 3625 2225 3500
 Wire Wire Line
-	2025 3500 2225 3500
+	1700 3500 2225 3500
 $Comp
 L power:GND #PWR057
@@
 	7425 2225 7425 2125
 Wire Wire Line
-	2025 2875 2400 2875
-Wire Wire Line
-	2025 2975 2225 2975
+	1700 2875 2400 2875
+Wire Wire Line
+	1700 2975 2225 2975
 Wire Wire Line
 	2225 2975 2225 3500
@@
 L custom:XT60_RA_MALE J15
 U 1 1 5C51EE4F
-P 1925 2925
-F 0 "J15" H 1800 2725 50  0000 L BNN
-F 1 "XT60_RA_MALE" H 1725 2575 50  0001 L BNN
-F 2 "custom:XT60PW" H 1725 2675 50  0001 L BNN
-F 3 "/home/dj/datasheets/XT60PW.pdf" H 1725 2475 50  0001 L BNN
-F 4 "XT60_M" H 1775 3025 50  0000 L BNN "Text"
-	1    1925 2925
+P 1600 2925
+F 0 "J15" H 1475 2725 50  0000 L BNN
+F 1 "XT60_RA_MALE" H 1400 2575 50  0001 L BNN
+F 2 "custom:XT60PW" H 1400 2675 50  0001 L BNN
+F 3 "/home/dj/datasheets/XT60PW.pdf" H 1400 2475 50  0001 L BNN
+F 4 "XT60_M" H 1450 3025 50  0000 L BNN "Text"
+	1    1600 2925
 	1    0    0    1
 $EndComp
@@
 L custom:XT60_RA_MALE J12
 U 1 1 5C52243D
-P 1900 2400
-F 0 "J12" H 1775 2200 50  0000 L BNN
-F 1 "XT60_RA_MALE" H 1700 2050 50  0001 L BNN
-F 2 "custom:XT60PW" H 1700 2150 50  0001 L BNN
-F 3 "/home/dj/datasheets/XT60PW.pdf" H 1700 1950 50  0001 L BNN
-F 4 "XT60_M" H 1750 2500 50  0000 L BNN "Text"
-	1    1900 2400
+P 1575 2400
+F 0 "J12" H 1450 2200 50  0000 L BNN
+F 1 "XT60_RA_MALE" H 1375 2050 50  0001 L BNN
+F 2 "custom:XT60PW" H 1375 2150 50  0001 L BNN
+F 3 "/home/dj/datasheets/XT60PW.pdf" H 1375 1950 50  0001 L BNN
+F 4 "XT60_M" H 1425 2500 50  0000 L BNN "Text"
+	1    1575 2400
 	1    0    0    1
 $EndComp
@@
 L custom:XT60_RA_FEMALE J18
 U 1 1 5C523072
-P 1950 3450
-F 0 "J18" H 2000 3600 50  0000 L BNN
-F 1 "XT60_RA_FEMALE" H 1750 3100 50  0001 L BNN
-F 2 "custom:XT60PW" H 1750 3200 50  0001 L BNN
-F 3 "/home/dj/datasheets/XT60PW.pdf" H 1750 3000 50  0001 L BNN
-F 4 "XT60_F" H 1850 3300 50  0000 L BNN "Text"
-	1    1950 3450
+P 1625 3450
+F 0 "J18" H 1675 3600 50  0000 L BNN
+F 1 "XT60_RA_FEMALE" H 1425 3100 50  0001 L BNN
+F 2 "custom:XT60PW" H 1425 3200 50  0001 L BNN
+F 3 "/home/dj/datasheets/XT60PW.pdf" H 1425 3000 50  0001 L BNN
+F 4 "XT60_F" H 1525 3300 50  0000 L BNN "Text"
+	1    1625 3450
 	-1   0    0    -1
 $EndComp
@@
 	2225 2975 2225 2450
 Wire Wire Line
-	2225 2450 2000 2450
+	2225 2450 1675 2450
 Connection ~ 2225 2975
 Wire Wire Line
@@
 	1    0    0    1
 $EndComp
-Text Label 9625 3125 0    50   ~ 0
-TAP_2
 Text Label 9625 3325 0    50   ~ 0
 TAP_0
@@
 F 0 "Q1" V 5225 2250 50  0000 L CNN
 F 1 "IRF9540N" V 5150 1975 50  0000 L CNN
-F 2 "Package_TO_SOT_THT:TO-220-3_Horizontal_TabDown" H 5200 2375 50  0001 L CIN
+F 2 "custom:TO-220-3_Horizontal_TabDown" H 5200 2375 50  0001 L CIN
 F 3 "/home/dj/datasheets/irf9540n.pdf" H 5200 2250 50  0001 L BNN
 	1    5000 2450
@@
 Connection ~ 2300 2350
 Wire Wire Line
-	2300 2350 2000 2350
+	2300 2350 1675 2350
 $Comp
 L custom:PTH_0.5_mm TP52
@@
 Wire Wire Line
 	5000 2800 5000 3075
-Text Notes 1125 2450 0    50   ~ 0
+Text Notes 825  2450 0    50   ~ 0
 BATTERY PORT
-Text Notes 1125 2975 0    50   ~ 0
+Text Notes 825  2975 0    50   ~ 0
 BATTERY PORT
-Text Notes 1050 3475 0    50   ~ 0
+Text Notes 750  3475 0    50   ~ 0
 CHARGING PORT
 Text Notes 10200 3350 0    50   ~ 0
@@
 Wire Wire Line
 	9550 4025 9550 4725
+Text Label 9625 3125 0    50   ~ 0
+TAP_2
+Text Label 1850 2350 0    50   ~ 0
+TAP_2
 $EndSCHEMATC

Commit message: automated commit
Parts:
- added Q4: SSM3K35AMFV, Package_TO_SOT_SMD:SOT-723, symbol custom:SSM3K35AMFV
- added R41: CR0603-JW-103ELF, Resistor_SMD:R_0603_1608Metric, symbol custom:CR0603-JW-103ELF
Connections:
- net GND: now also Q4.2 (S), R41.2; no longer R29.2, R30.2, R31.2
- new net: Q4.3 (D), R29.2, R30.2, R31.2
- new net +3V3: Q4.1 (G), R41.1
Changed lines of the file:
@@
 L power:GND #PWR066
 U 1 1 5C5E3535
-P 7600 4725
-F 0 "#PWR066" H 7600 4475 50  0001 C CNN
-F 1 "GND" H 7600 4575 50  0000 C CNN
-F 2 "" H 7600 4725 50  0001 C CNN
-F 3 "" H 7600 4725 50  0001 C CNN
-	1    7600 4725
+P 7600 5500
+F 0 "#PWR066" H 7600 5250 50  0001 C CNN
+F 1 "GND" H 7600 5350 50  0000 C CNN
+F 2 "" H 7600 5500 50  0001 C CNN
+F 3 "" H 7600 5500 50  0001 C CNN
+	1    7600 5500
 	1    0    0    -1
 $EndComp
@@
 Connection ~ 7500 4675
 Wire Wire Line
-	7600 4675 7600 4725
+	7600 5450 7600 5500
 Wire Wire Line
 	7600 4325 7600 4150
@@
 Wire Wire Line
 	6675 3950 6900 3950
-Connection ~ 7600 4675
 $Comp
 L custom:PTH_0.5_mm TP5
@@
 Text Label 7600 3150 3    50   ~ 0
 TAP_0
-Text Notes 6450 4700 0    50   ~ 0
+Text Notes 6450 4675 0    50   ~ 0
 INDICATE VOLTAGES\nON SILKSCREEN
 $Comp
@@
 Text Label 1850 2350 0    50   ~ 0
 TAP_2
+$Comp
+L custom:SSM3K35AMFV Q4
+U 1 1 5C937F61
+P 7500 5250
+F 0 "Q4" H 7700 5250 50  0000 L BNN
+F 1 "SSM3K35AMFV" H 7700 5175 50  0000 L BNN
+F 2 "Package_TO_SOT_SMD:SOT-723" H 7700 5175 50  0001 L BIN
+F 3 "/home/dj/datasheets/SSM3K35AMFV.pdf" H 7700 5100 50  0001 L BNN
+	1    7500 5250
+	1    0    0    -1
+$EndComp
+Wire Wire Line
+	7600 5050 7600 4675
+Connection ~ 7600 4675
+$Comp
+L power:+3V3 #PWR?
+U 1 1 5C94DADD
+P 7200 5025
+AR Path="/5C100B31/5C94DADD" Ref="#PWR?"  Part="1"
+AR Path="/5C5AE643/5C94DADD" Ref="#PWR0104"  Part="1"
+F 0 "#PWR0104" H 7200 4875 50  0001 C CNN
+F 1 "+3V3" H 7200 5165 50  0000 C CNN
+F 2 "" H 7200 5025 50  0001 C CNN
+F 3 "" H 7200 5025 50  0001 C CNN
+	1    7200 5025
+	1    0    0    -1
+$EndComp
+Wire Wire Line
+	7200 5025 7200 5250
+Wire Wire Line
+	7200 5250 7300 5250
+$Comp
+L custom:CR0603-JW-103ELF R41
+U 1 1 5C95D060
+P 7200 5575
+F 0 "R41" V 7175 5700 50  0000 L BNN
+F 1 "CR0603-JW-103ELF" V 7325 5250 50  0001 L BNN
+F 2 "Resistor_SMD:R_0603_1608Metric" V 7400 5475 50  0001 L BNN
+F 3 "~/datasheets/chpreztr.pdf" V 7500 5125 50  0001 L BNN
+F 4 "10k0" V 7200 5575 50  0000 C CNN "Resistance"
+	1    7200 5575
+	1    0    0    -1
+$EndComp
+Wire Wire Line
+	7200 5250 7200 5425
+Connection ~ 7200 5250
+$Comp
+L power:GND #PWR0105
+U 1 1 5C961E83
+P 7200 5775
+F 0 "#PWR0105" H 7200 5525 50  0001 C CNN
+F 1 "GND" H 7200 5625 50  0000 C CNN
+F 2 "" H 7200 5775 50  0001 C CNN
+F 3 "" H 7200 5775 50  0001 C CNN
+	1    7200 5775
+	1    0    0    -1
+$EndComp
+Wire Wire Line
+	7200 5725 7200 5775
 $EndSCHEMATC
