File: nu.ai_motor_controller/battery.sch (KiCad schematic (older format))
At the start: 40 parts, among them J12 XT60_RA_MALE, J13 S4B-XH-A, J14 NP_Screw_Terminal_01x02, J15 XT60_RA_MALE, J16 S4B-XH-A, J17 S4B-XH-A, J18 XT60_RA_FEMALE, Q1 IRF9540N, Q2 SSM3K35AMFV, Q4 SSM3K35AMFV, SW2 TACTILE_SWITCH, SW3 TACTILE_SWITCH

Commit message: automated commit
Parts:
- added F1, F3: NP_FUSE_0603, Fuse:Fuse_0603_1608Metric, symbol custom:NP_FUSE_0603
- TP1, TP2, TP3, TP4, TP5, TP52, TP53, TP54, TP55, TP56, TP6, TP7: footprint TestPoint:TestPoint_THTPad_D1.0mm_Drill0.5mm -> custom:TestPoint_THTPad_D1.0mm_Drill0.5mm
Connections:
- net TAP_2: now also F1.1, F3.1
- net at D8.6 (CH3), F2.2, Q1.3 (S)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: now also F1.2, F3.2
Changed lines of the file:
@@
 F 0 "TP1" V 9300 3375 50  0000 L BNN
 F 1 "PTH_0.5_mm" V 9250 3300 50  0001 L BNN
-F 2 "TestPoint:TestPoint_THTPad_D1.0mm_Drill0.5mm" H 9475 3125 50  0001 L BNN
+F 2 "custom:TestPoint_THTPad_D1.0mm_Drill0.5mm" H 9475 3125 50  0001 L BNN
 F 3 "~" H 9475 3125 50  0001 C CNN
 	1    9275 3125
@@
 F 0 "TP2" V 9300 3475 50  0000 L BNN
 F 1 "PTH_0.5_mm" V 9250 3400 50  0001 L BNN
-F 2 "TestPoint:TestPoint_THTPad_D1.0mm_Drill0.5mm" H 9475 3225 50  0001 L BNN
+F 2 "custom:TestPoint_THTPad_D1.0mm_Drill0.5mm" H 9475 3225 50  0001 L BNN
 F 3 "~" H 9475 3225 50  0001 C CNN
 	1    9275 3225
@@
 F 0 "TP3" V 9300 3575 50  0000 L BNN
 F 1 "PTH_0.5_mm" V 9250 3500 50  0001 L BNN
-F 2 "TestPoint:TestPoint_THTPad_D1.0mm_Drill0.5mm" H 9475 3325 50  0001 L BNN
+F 2 "custom:TestPoint_THTPad_D1.0mm_Drill0.5mm" H 9475 3325 50  0001 L BNN
 F 3 "~" H 9475 3325 50  0001 C CNN
 	1    9275 3325
@@
 F 0 "TP4" V 9300 3675 50  0000 L BNN
 F 1 "PTH_0.5_mm" V 9250 3600 50  0001 L BNN
-F 2 "TestPoint:TestPoint_THTPad_D1.0mm_Drill0.5mm" H 9475 3425 50  0001 L BNN
+F 2 "custom:TestPoint_THTPad_D1.0mm_Drill0.5mm" H 9475 3425 50  0001 L BNN
 F 3 "~" H 9475 3425 50  0001 C CNN
 	1    9275 3425
@@
 Connection ~ 2225 2975
 Wire Wire Line
-	2400 2875 2400 2350
+	2400 2875 2400 2750
 Wire Wire Line
 	2400 2350 2300 2350
@@
 F 0 "TP5" V 6875 4250 50  0000 L BNN
 F 1 "PTH_0.5_mm" V 6875 4475 50  0001 L BNN
-F 2 "TestPoint:TestPoint_THTPad_D1.0mm_Drill0.5mm" H 7100 4300 50  0001 L BNN
+F 2 "custom:TestPoint_THTPad_D1.0mm_Drill0.5mm" H 7100 4300 50  0001 L BNN
 F 3 "~" H 7100 4300 50  0001 C CNN
 	1    6900 4300
@@
 F 0 "TP6" V 6975 4250 50  0000 L BNN
 F 1 "PTH_0.5_mm" V 6975 4475 50  0001 L BNN
-F 2 "TestPoint:TestPoint_THTPad_D1.0mm_Drill0.5mm" H 7200 4300 50  0001 L BNN
+F 2 "custom:TestPoint_THTPad_D1.0mm_Drill0.5mm" H 7200 4300 50  0001 L BNN
 F 3 "~" H 7200 4300 50  0001 C CNN
 	1    7000 4300
@@
 F 0 "TP7" V 7075 4250 50  0000 L BNN
 F 1 "PTH_0.5_mm" V 7075 4475 50  0001 L BNN
-F 2 "TestPoint:TestPoint_THTPad_D1.0mm_Drill0.5mm" H 7300 4300 50  0001 L BNN
+F 2 "custom:TestPoint_THTPad_D1.0mm_Drill0.5mm" H 7300 4300 50  0001 L BNN
 F 3 "~" H 7300 4300 50  0001 C CNN
 	1    7100 4300
@@
 	2900 2350 3000 2350
 Wire Wire Line
-	3000 2350 3000 3075
+	3000 2350 3000 2550
 Connection ~ 3000 2350
 Wire Wire Line
@@
 F 0 "TP53" H 2225 2425 50  0000 L BNN
 F 1 "PTH_0.5_mm" V 2275 2425 50  0001 L BNN
-F 2 "TestPoint:TestPoint_THTPad_D1.0mm_Drill0.5mm" H 2500 2250 50  0001 L BNN
+F 2 "custom:TestPoint_THTPad_D1.0mm_Drill0.5mm" H 2500 2250 50  0001 L BNN
 F 3 "~" H 2500 2250 50  0001 C CNN
 	1    2300 2250
@@
 F 0 "TP54" H 3025 2425 50  0000 L BNN
 F 1 "PTH_0.5_mm" V 3075 2425 50  0001 L BNN
-F 2 "TestPoint:TestPoint_THTPad_D1.0mm_Drill0.5mm" H 3300 2250 50  0001 L BNN
+F 2 "custom:TestPoint_THTPad_D1.0mm_Drill0.5mm" H 3300 2250 50  0001 L BNN
 F 3 "~" H 3300 2250 50  0001 C CNN
 	1    3100 2250
@@
 F 0 "TP52" V 7250 2325 50  0000 L BNN
 F 1 "PTH_0.5_mm" V 7275 2400 50  0001 L BNN
-F 2 "TestPoint:TestPoint_THTPad_D1.0mm_Drill0.5mm" H 7500 2225 50  0001 L BNN
+F 2 "custom:TestPoint_THTPad_D1.0mm_Drill0.5mm" H 7500 2225 50  0001 L BNN
 F 3 "~" H 7500 2225 50  0001 C CNN
 	1    7300 2225
@@
 F 0 "TP56" H 4425 4225 50  0000 L BNN
 F 1 "PTH_0.5_mm" V 4475 4225 50  0001 L BNN
-F 2 "TestPoint:TestPoint_THTPad_D1.0mm_Drill0.5mm" H 4700 4050 50  0001 L BNN
+F 2 "custom:TestPoint_THTPad_D1.0mm_Drill0.5mm" H 4700 4050 50  0001 L BNN
 F 3 "~" H 4700 4050 50  0001 C CNN
 	1    4500 4050
@@
 F 0 "TP55" V 4975 2800 50  0000 L BNN
 F 1 "PTH_0.5_mm" V 5025 2875 50  0001 L BNN
-F 2 "TestPoint:TestPoint_THTPad_D1.0mm_Drill0.5mm" H 5250 2700 50  0001 L BNN
+F 2 "custom:TestPoint_THTPad_D1.0mm_Drill0.5mm" H 5250 2700 50  0001 L BNN
 F 3 "~" H 5250 2700 50  0001 C CNN
 	1    5050 2700
@@
 Wire Wire Line
 	7200 5725 7200 5775
+$Comp
+L custom:NP_FUSE_0603 F3
+U 1 1 5C6FB132
+P 2700 2750
+F 0 "F3" H 2500 2800 50  0000 L BNN
+F 1 "NP_FUSE_0603" H 2450 2650 50  0001 L BNN
+F 2 "Fuse:Fuse_0603_1608Metric" H 2350 2550 50  0001 L BNN
+F 3 "" H 2300 2550 50  0001 L BNN
+F 4 "NP" H 2800 2800 50  0000 L BNN "NP"
+	1    2700 2750
+	1    0    0    -1
+$EndComp
+$Comp
+L custom:NP_FUSE_0603 F1
+U 1 1 5C6FB1D3
+P 2700 2550
+F 0 "F1" H 2500 2600 50  0000 L BNN
+F 1 "NP_FUSE_0603" H 2450 2450 50  0001 L BNN
+F 2 "Fuse:Fuse_0603_1608Metric" H 2350 2350 50  0001 L BNN
+F 3 "" H 2300 2350 50  0001 L BNN
+F 4 "NP" H 2800 2600 50  0000 L BNN "NP"
+	1    2700 2550
+	1    0    0    -1
+$EndComp
+Wire Wire Line
+	2500 2550 2400 2550
+Connection ~ 2400 2550
+Wire Wire Line
+	2400 2550 2400 2350
+Wire Wire Line
+	2500 2750 2400 2750
+Connection ~ 2400 2750
+Wire Wire Line
+	2400 2750 2400 2550
+Wire Wire Line
+	2900 2750 3000 2750
+Connection ~ 3000 2750
+Wire Wire Line
+	3000 2750 3000 3075
+Wire Wire Line
+	2900 2550 3000 2550
+Connection ~ 3000 2550
+Wire Wire Line
+	3000 2550 3000 2750
 $EndSCHEMATC

Commit message: automated commit
Parts:
- added Q5, Q6: SSM3K35AMFV, Package_TO_SOT_SMD:SOT-723, symbol custom:SSM3K35AMFV
Connections:
- net +3V3: now also Q5.1 (G), Q6.1 (G)
- net GND: now also Q5.2 (S), Q6.2 (S)
- net at Q4.3 (D), R31.2: no longer R29.2, R30.2
- new net: Q5.3 (D), R29.2
- new net: Q6.3 (D), R30.2
Other:
- note removed: "SILK: BAT"
- moved on the sheet: D7, D8, F1, F2, F3, J12, J13, J14, J15, J16, J17, J18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
