File: nu.ai_motor_controller/driver.sch (KiCad schematic (older format))
At the start: 8 parts

Commit message: cleaned up and renamed project files. Changed custom library management scheme. It now resides in my homedir as a seperate git project, and is pointed to in kicad's symbol library manager
Parts:
- U? (x4): symbol nu-rescue:MP6513-custom -> custom:MP6513
Changed lines of the file:
@@
 EESchema Schematic File Version 4
-LIBS:nu-cache
+LIBS:nu.ai_motor_controller-cache
 EELAYER 26 0
 EELAYER END
@@
 $EndDescr
 $Comp
-L nu-rescue:MP6513-custom U?
+L custom:MP6513 U?
 U 1 1 5C101246
 P 4950 2650
@@
 $EndComp
 $Comp
-L nu-rescue:MP6513-custom U?
+L custom:MP6513 U?
 U 1 1 5C10124D
 P 4950 3700
@@
 $EndComp
 $Comp
-L nu-rescue:MP6513-custom U?
+L custom:MP6513 U?
 U 1 1 5C101254
 P 4950 4750
@@
 $EndComp
 $Comp
-L nu-rescue:MP6513-custom U?
+L custom:MP6513 U?
 U 1 1 5C10125B
 P 4950 5800

Commit message: automated commit
Connections:
- net labels added: IN_1_L, IN_1_R, IN_2_L, IN_2_R
- net labels removed: IN_1_A, IN_1_B, IN_1_C, IN_1_D, IN_2_A, IN_2_B, IN_2_C, IN_2_D
- wire segments 48 -> 56
Changed lines of the file:
@@
 F 1 "MP6513" H 4950 2400 50  0000 C CNN
 F 2 "" H 4950 2650 50  0001 C CNN
-F 3 "MP6513.pdf" H 4950 2650 50  0001 C CNN
+F 3 "/home/dj/datasheet/MP6513.pdf" H 4950 2650 50  0001 C CNN
 	1    4950 2650
 	1    0    0    -1
@@
 	1    0    0    -1
 $EndComp
-Text HLabel 4400 2550 0    50   Input ~ 0
-IN_1_A
-Text HLabel 4400 2750 0    50   Input ~ 0
-IN_2_A
-Wire Wire Line
-	4600 2550 4400 2550
-Wire Wire Line
-	4400 2750 4600 2750
-Text HLabel 4400 3600 0    50   Input ~ 0
-IN_1_B
-Text HLabel 4400 3800 0    50   Input ~ 0
-IN_2_B
-Wire Wire Line
-	4600 3600 4400 3600
-Wire Wire Line
-	4400 3800 4600 3800
-Text HLabel 4400 4650 0    50   Input ~ 0
-IN_1_C
-Text HLabel 4400 4850 0    50   Input ~ 0
-IN_2_C
-Wire Wire Line
-	4600 4650 4400 4650
-Wire Wire Line
-	4400 4850 4600 4850
-Text HLabel 4400 5700 0    50   Input ~ 0
-IN_1_D
-Text HLabel 4400 5900 0    50   Input ~ 0
-IN_2_D
-Wire Wire Line
-	4600 5700 4400 5700
-Wire Wire Line
-	4400 5900 4600 5900
+Text HLabel 3850 2550 0    50   Input ~ 0
+IN_1_L
+Text HLabel 3850 2750 0    50   Input ~ 0
+IN_2_L
+Wire Wire Line
+	4600 2550 4350 2550
+Wire Wire Line
+	3850 2750 4150 2750
+Wire Wire Line
+	4600 3600 4350 3600
+Text HLabel 3850 4650 0    50   Input ~ 0
+IN_1_R
+Text HLabel 3850 4850 0    50   Input ~ 0
+IN_2_R
+Wire Wire Line
+	4600 4650 4350 4650
+Wire Wire Line
+	3850 4850 4150 4850
 Text HLabel 5500 2350 2    50   Output ~ 0
 OUT_1_A
@@
 	5700 1450 5700 1400
 Connection ~ 5700 1400
+Wire Wire Line
+	4350 3600 4350 2550
+Connection ~ 4350 2550
+Wire Wire Line
+	4350 2550 3850 2550
+Wire Wire Line
+	4150 3800 4150 2750
+Wire Wire Line
+	4150 3800 4600 3800
+Connection ~ 4150 2750
+Wire Wire Line
+	4150 2750 4600 2750
+Wire Wire Line
+	4350 5700 4350 4650
+Wire Wire Line
+	4150 5900 4150 4850
+Wire Wire Line
+	4350 5700 4600 5700
+Wire Wire Line
+	4150 5900 4600 5900
+Connection ~ 4350 4650
+Wire Wire Line
+	4350 4650 3850 4650
+Connection ~ 4150 4850
+Wire Wire Line
+	4150 4850 4600 4850
 $EndSCHEMATC

Commit message: automated commit
Connections:
- net labels added: VDD_BAT
- net labels removed: +12V
Changed lines of the file:
@@
 Wire Wire Line
 	4550 2350 4550 2250
-$Comp
-L power:+12V #PWR?
-U 1 1 5C102145
-P 4550 2250
-F 0 "#PWR?" H 4550 2100 50  0001 C CNN
-F 1 "+12V" H 4550 2390 50  0000 C CNN
-F 2 "" H 4550 2250 50  0001 C CNN
-F 3 "" H 4550 2250 50  0001 C CNN
-	1    4550 2250
-	1    0    0    -1
-$EndComp
 Wire Wire Line
 	5300 2750 5350 2750
@@
 Wire Wire Line
 	4200 1050 4200 1000
-$Comp
-L power:+12V #PWR?
-U 1 1 5C133D67
-P 4200 950
-F 0 "#PWR?" H 4200 800 50  0001 C CNN
-F 1 "+12V" H 4200 1090 50  0000 C CNN
-F 2 "" H 4200 950 50  0001 C CNN
-F 3 "" H 4200 950 50  0001 C CNN
-	1    4200 950
-	1    0    0    -1
-$EndComp
 $Comp
 L custom:CL10B105KA8NNNC C?
@@
 Wire Wire Line
 	4150 4850 4600 4850
+$Comp
+L custom:VDD_BAT #PWR?
+U 1 1 5C53B7B2
+P 4550 2250
+F 0 "#PWR?" H 4750 2300 50  0001 C CNN
+F 1 "VDD_BAT" H 4400 2400 50  0000 L BNN
+F 2 "" H 4550 2250 50  0001 C CNN
+F 3 "" H 4550 2250 50  0001 C CNN
+	1    4550 2250
+	1    0    0    -1
+$EndComp
+$Comp
+L custom:VDD_BAT #PWR?
+U 1 1 5C53B7F4
+P 4200 950
+F 0 "#PWR?" H 4400 1000 50  0001 C CNN
+F 1 "VDD_BAT" H 4050 1100 50  0000 L BNN
+F 2 "" H 4200 950 50  0001 C CNN
+F 3 "" H 4200 950 50  0001 C CNN
+	1    4200 950
+	1    0    0    -1
+$EndComp
 $EndSCHEMATC

Commit message: automated commit
Parts:
- gave numbers to parts that had none: 8
Changed lines of the file:
@@
 P 4950 2650
 AR Path="/5C101246" Ref="U?"  Part="1"
-AR Path="/5C10107F/5C101246" Ref="U?"  Part="1"
-F 0 "U?" H 4900 3100 50  0000 C CNN
+AR Path="/5C10107F/5C101246" Ref="U5"  Part="1"
+F 0 "U5" H 4900 3100 50  0000 C CNN
 F 1 "MP6513" H 4950 2400 50  0000 C CNN
 F 2 "" H 4950 2650 50  0001 C CNN
@@
 P 4950 3700
 AR Path="/5C10124D" Ref="U?"  Part="1"
-AR Path="/5C10107F/5C10124D" Ref="U?"  Part="1"
-F 0 "U?" H 4900 4150 50  0000 C CNN
+AR Path="/5C10107F/5C10124D" Ref="U6"  Part="1"
+F 0 "U6" H 4900 4150 50  0000 C CNN
 F 1 "MP6513" H 4950 3450 50  0000 C CNN
 F 2 "" H 4950 3700 50  0001 C CNN
@@
 P 4950 4750
 AR Path="/5C101254" Ref="U?"  Part="1"
-AR Path="/5C10107F/5C101254" Ref="U?"  Part="1"
-F 0 "U?" H 4900 5200 50  0000 C CNN
+AR Path="/5C10107F/5C101254" Ref="U7"  Part="1"
+F 0 "U7" H 4900 5200 50  0000 C CNN
 F 1 "MP6513" H 4950 4500 50  0000 C CNN
 F 2 "" H 4950 4750 50  0001 C CNN
@@
 P 4950 5800
 AR Path="/5C10125B" Ref="U?"  Part="1"
-AR Path="/5C10107F/5C10125B" Ref="U?"  Part="1"
-F 0 "U?" H 4900 6250 50  0000 C CNN
+AR Path="/5C10107F/5C10125B" Ref="U8"  Part="1"
+F 0 "U8" H 4900 6250 50  0000 C CNN
 F 1 "MP6513" H 4950 5550 50  0000 C CNN
 F 2 "" H 4950 5800 50  0001 C CNN
@@
 	5350 3800 5350 4850
 $Comp
-L power:GND #PWR?
+L power:GND #PWR018
 U 1 1 5C10256A
 P 5350 6000
-F 0 "#PWR?" H 5350 5750 50  0001 C CNN
+F 0 "#PWR018" H 5350 5750 50  0001 C CNN
 F 1 "GND" H 5350 5850 50  0000 C CNN
 F 2 "" H 5350 6000 50  0001 C CNN
@@
 	4200 1050 4200 1000
 $Comp
-L custom:CL10B105KA8NNNC C?
+L custom:CL10B105KA8NNNC C7
 U 1 1 5C135FCC
 P 5200 1200
-F 0 "C?" H 5350 1300 50  0000 L BNN
+F 0 "C7" H 5350 1300 50  0000 L BNN
 F 1 "CL10B105KA8NNNC" H 4250 750 50  0001 L BNN
 F 2 "Capacitor_SMD:C_0603_1608Metric" H 4250 650 50  0001 L BNN
@@
 $EndComp
 $Comp
-L custom:CL10B105KA8NNNC C?
+L custom:CL10B105KA8NNNC C8
 U 1 1 5C137068
 P 5700 1200
-F 0 "C?" H 5850 1300 50  0000 L BNN
+F 0 "C8" H 5850 1300 50  0000 L BNN
 F 1 "CL10B105KA8NNNC" H 4750 750 50  0001 L BNN
 F 2 "Capacitor_SMD:C_0603_1608Metric" H 4750 650 50  0001 L BNN
@@
 $EndComp
 $Comp
-L custom:CL10B105KA8NNNC C?
+L custom:CL10B105KA8NNNC C5
 U 1 1 5C138334
 P 4200 1200
-F 0 "C?" H 4350 1300 50  0000 L BNN
+F 0 "C5" H 4350 1300 50  0000 L BNN
 F 1 "CL10B105KA8NNNC" H 3250 750 50  0001 L BNN
 F 2 "Capacitor_SMD:C_0603_1608Metric" H 3250 650 50  0001 L BNN
@@
 $EndComp
 $Comp
-L custom:CL10B105KA8NNNC C?
+L custom:CL10B105KA8NNNC C6
 U 1 1 5C13833D
 P 4700 1200
-F 0 "C?" H 4850 1300 50  0000 L BNN
+F 0 "C6" H 4850 1300 50  0000 L BNN
 F 1 "CL10B105KA8NNNC" H 3750 750 50  0001 L BNN
 F 2 "Capacitor_SMD:C_0603_1608Metric" H 3750 650 50  0001 L BNN
@@
 	4700 1400 5200 1400
 $Comp
-L power:GND #PWR?
+L power:GND #PWR016
 U 1 1 5C140ED3
 P 5700 1450
-F 0 "#PWR?" H 5700 1200 50  0001 C CNN
+F 0 "#PWR016" H 5700 1200 50  0001 C CNN
 F 1 "GND" H 5700 1300 50  0000 C CNN
 F 2 "" H 5700 1450 50  0001 C CNN
@@
 	4150 4850 4600 4850
 $Comp
-L custom:VDD_BAT #PWR?
+L custom:VDD_BAT #PWR017
 U 1 1 5C53B7B2
 P 4550 2250
-F 0 "#PWR?" H 4750 2300 50  0001 C CNN
+F 0 "#PWR017" H 4750 2300 50  0001 C CNN
 F 1 "VDD_BAT" H 4400 2400 50  0000 L BNN
 F 2 "" H 4550 2250 50  0001 C CNN
@@
 $EndComp
 $Comp
-L custom:VDD_BAT #PWR?
+L custom:VDD_BAT #PWR015
 U 1 1 5C53B7F4
 P 4200 950
-F 0 "#PWR?" H 4400 1000 50  0001 C CNN
+F 0 "#PWR015" H 4400 1000 50  0001 C CNN
 F 1 "VDD_BAT" H 4050 1100 50  0000 L BNN
 F 2 "" H 4200 950 50  0001 C CNN

Commit message: automated commit
Parts:
- removed U5, U6, U7, U8: MP6513, symbol custom:MP6513
- added U? (x4): MP6513, symbol custom:MP6513
Connections:
- net GND: now also U?.2 (GND), U?.2 (GND), U?.2 (GND), U?.2 (GND)
- net IN_1_L: now also U?.1 (IN1), U?.1 (IN1)
- net IN_1_R: now also U?.1 (IN1), U?.1 (IN1)
- net IN_2_L: now also U?.3 (IN2), U?.3 (IN2)
- net IN_2_R: now also U?.3 (IN2), U?.3 (IN2)
- net OUT_1_A: now also U?.6 (OUT1)
- net OUT_1_B: now also U?.6 (OUT1)
- net OUT_1_C: now also U?.6 (OUT1)
- net OUT_1_D: now also U?.6 (OUT1)
- net OUT_2_A: now also U?.4 (OUT2)
- net OUT_2_B: now also U?.4 (OUT2)
- net OUT_2_C: now also U?.4 (OUT2)
- net OUT_2_D: now also U?.4 (OUT2)
- net VDD_BAT: now also U?.5 (VDD), U?.5 (VDD), U?.5 (VDD), U?.5 (VDD)
Changed lines of the file:
@@
 Comment4 ""
 $EndDescr
-$Comp
-L custom:MP6513 U?
-U 1 1 5C101246
-P 4950 2650
-AR Path="/5C101246" Ref="U?"  Part="1"
-AR Path="/5C10107F/5C101246" Ref="U5"  Part="1"
-F 0 "U5" H 4900 3100 50  0000 C CNN
-F 1 "MP6513" H 4950 2400 50  0000 C CNN
-F 2 "" H 4950 2650 50  0001 C CNN
-F 3 "/home/dj/datasheet/MP6513.pdf" H 4950 2650 50  0001 C CNN
-	1    4950 2650
-	1    0    0    -1
-$EndComp
-$Comp
-L custom:MP6513 U?
-U 1 1 5C10124D
-P 4950 3700
-AR Path="/5C10124D" Ref="U?"  Part="1"
-AR Path="/5C10107F/5C10124D" Ref="U6"  Part="1"
-F 0 "U6" H 4900 4150 50  0000 C CNN
-F 1 "MP6513" H 4950 3450 50  0000 C CNN
-F 2 "" H 4950 3700 50  0001 C CNN
-F 3 "MP6513.pdf" H 4950 3700 50  0001 C CNN
-	1    4950 3700
-	1    0    0    -1
-$EndComp
-$Comp
-L custom:MP6513 U?
-U 1 1 5C101254
-P 4950 4750
-AR Path="/5C101254" Ref="U?"  Part="1"
-AR Path="/5C10107F/5C101254" Ref="U7"  Part="1"
-F 0 "U7" H 4900 5200 50  0000 C CNN
-F 1 "MP6513" H 4950 4500 50  0000 C CNN
-F 2 "" H 4950 4750 50  0001 C CNN
-F 3 "MP6513.pdf" H 4950 4750 50  0001 C CNN
-	1    4950 4750
-	1    0    0    -1
-$EndComp
-$Comp
-L custom:MP6513 U?
-U 1 1 5C10125B
-P 4950 5800
-AR Path="/5C10125B" Ref="U?"  Part="1"
-AR Path="/5C10107F/5C10125B" Ref="U8"  Part="1"
-F 0 "U8" H 4900 6250 50  0000 C CNN
-F 1 "MP6513" H 4950 5550 50  0000 C CNN
-F 2 "" H 4950 5800 50  0001 C CNN
-F 3 "MP6513.pdf" H 4950 5800 50  0001 C CNN
-	1    4950 5800
-	1    0    0    -1
-$EndComp
 Wire Wire Line
 	4600 5500 4550 5500
@@
 	1    0    0    -1
 $EndComp
+$Comp
+L custom:MP6513 U?
+U 1 1 5C565750
+P 4950 2650
+F 0 "U?" H 4900 3100 50  0000 C CNN
+F 1 "MP6513" H 4950 2400 50  0000 C CNN
+F 2 "" H 4950 2650 50  0001 C CNN
+F 3 "/home/dj/datasheets/MP6513.pdf" H 4950 2650 50  0001 C CNN
+	1    4950 2650
+	1    0    0    -1
+$EndComp
+$Comp
+L custom:MP6513 U?
+U 1 1 5C5657C3
+P 4950 3700
+F 0 "U?" H 4900 4150 50  0000 C CNN
+F 1 "MP6513" H 4950 3450 50  0000 C CNN
+F 2 "" H 4950 3700 50  0001 C CNN
+F 3 "/home/dj/datasheets/MP6513.pdf" H 4950 3700 50  0001 C CNN
+	1    4950 3700
+	1    0    0    -1
+$EndComp
+$Comp
+L custom:MP6513 U?
+U 1 1 5C565DC5
+P 4950 4750
+F 0 "U?" H 4900 5200 50  0000 C CNN
+F 1 "MP6513" H 4950 4500 50  0000 C CNN
+F 2 "" H 4950 4750 50  0001 C CNN
+F 3 "/home/dj/datasheets/MP6513.pdf" H 4950 4750 50  0001 C CNN
+	1    4950 4750
+	1    0    0    -1
+$EndComp
+$Comp
+L custom:MP6513 U?
+U 1 1 5C565E47
+P 4950 5800
+F 0 "U?" H 4900 6250 50  0000 C CNN
+F 1 "MP6513" H 4950 5550 50  0000 C CNN
+F 2 "" H 4950 5800 50  0001 C CNN
+F 3 "/home/dj/datasheets/MP6513.pdf" H 4950 5800 50  0001 C CNN
+	1    4950 5800
+	1    0    0    -1
+$EndComp

Commit message: automated commit
Parts:
- gave numbers to parts that had none: 4
Changed lines of the file:
@@
 $EndComp
 $Comp
-L custom:MP6513 U?
+L custom:MP6513 U6
 U 1 1 5C565750
 P 4950 2650
-F 0 "U?" H 4900 3100 50  0000 C CNN
+F 0 "U6" H 4900 3100 50  0000 C CNN
 F 1 "MP6513" H 4950 2400 50  0000 C CNN
 F 2 "" H 4950 2650 50  0001 C CNN
@@
 $EndComp
 $Comp
-L custom:MP6513 U?
+L custom:MP6513 U7
 U 1 1 5C5657C3
 P 4950 3700
-F 0 "U?" H 4900 4150 50  0000 C CNN
+F 0 "U7" H 4900 4150 50  0000 C CNN
 F 1 "MP6513" H 4950 3450 50  0000 C CNN
 F 2 "" H 4950 3700 50  0001 C CNN
@@
 $EndComp
 $Comp
-L custom:MP6513 U?
+L custom:MP6513 U8
 U 1 1 5C565DC5
 P 4950 4750
-F 0 "U?" H 4900 5200 50  0000 C CNN
+F 0 "U8" H 4900 5200 50  0000 C CNN
 F 1 "MP6513" H 4950 4500 50  0000 C CNN
 F 2 "" H 4950 4750 50  0001 C CNN
@@
 $EndComp
 $Comp
-L custom:MP6513 U?
+L custom:MP6513 U10
 U 1 1 5C565E47
 P 4950 5800
-F 0 "U?" H 4900 6250 50  0000 C CNN
+F 0 "U10" H 4900 6250 50  0000 C CNN
 F 1 "MP6513" H 4950 5550 50  0000 C CNN
 F 2 "" H 4950 5800 50  0001 C CNN

Commit message: automated commit
Parts:
- added R? (x8): RC0603JR-071KL, 0603, symbol custom:RC0603JR-071KL
- added U? (x2): SGM3157YC6, Package_TO_SOT_SMD:SOT-23-6, symbol custom:SGM3157YC6
Connections:
- net labels added: VDD_uC
- wire segments 56 -> 106
Other:
- moved on the sheet: C5, C6, C7, C8, U10, U6, U7, U8
