File: nu.ai_motor_controller/driver.sch (KiCad schematic (older format))
At the start: 18 parts, among them U10 MP6513, U6 MP6513, U7 MP6513, U8 MP6513

Commit message: automated commit
Parts:
- removed R? (x6): RC0603JR-071KL, 0603, symbol custom:RC0603JR-071KL
- removed U?: SGM3157YC6, Package_TO_SOT_SMD:SOT-23-6, symbol custom:SGM3157YC6
- added J1, J2, J3, J4, J5, J6, J7, J8: PTH_1_mm, symbol custom:PTH_1_mm
- added R10, R11, R12, R32, R33, R9: RC0603JR-071KL, 0603, symbol custom:RC0603JR-071KL
- added TP18, TP19, TP20, TP21, TP22, TP23, TP24, TP25, TP26, TP27, TP28, TP29, TP30, TP31, TP32, TP33: PTH_0.5_mm, symbol custom:PTH_0.5_mm
- added U4: SGM3157YC6, Package_TO_SOT_SMD:SOT-23-6, symbol custom:SGM3157YC6
- gave numbers to parts that had none: 3
Connections:
- net labels added: L_DIR, L_MOTOR, R_DIR, R_MOTOR
- net labels removed: IN_1_L, IN_1_R, IN_2_L, IN_2_R, OUT_1_A, OUT_1_B, OUT_1_C, OUT_1_D, OUT_2_A, OUT_2_B, OUT_2_C, OUT_2_D
- wire segments 106 -> 136
Other:
- note added: "ADD 2 mm STRAIN RELIEF HOLES\nFOR EVERY PTH"
- note added: "OUT_A1"
- note added: "OUT_A2"
- note added: "OUT_B1"
- note added: "OUT_B2"
- note added: "OUT_C1"
- note added: "OUT_C2"
- note added: "OUT_D1"
- note added: "OUT_D2"
- moved on the sheet: C5, C6, C7, C8, R7, R8, U10, U3, U6, U7, U8

Commit message: automated commit
Parts:
- added C29, C30: CL10B105KA8NNNC, Capacitor_SMD:C_0603_1608Metric, symbol custom:CL10B105KA8NNNC
- added NPTH1, NPTH2, NPTH3, NPTH4, NPTH5, NPTH6, NPTH7, NPTH8: NPTH_2mm, custom:NPTH_2mm, symbol custom:NPTH_2mm
- J1, J2, J3, J4, J5, J6, J7, J8: footprint (none) -> TestPoint:TestPoint_THTPad_D2.0mm_Drill1.0mm
- R10, R11, R12, R32, R33, R7, R8, R9: footprint 0603 -> Resistor_SMD:R_0603_1608Metric
- TP18, TP19, TP20, TP21, TP22, TP23, TP24, TP25, TP26, TP27, TP28, TP29, TP30, TP31, TP32, TP33: footprint (none) -> TestPoint:TestPoint_THTPad_D1.0mm_Drill0.5mm
- U10, U6, U7, U8: footprint (none) -> custom:TSOT23-6
Connections:
- net GND: now also C29.2, C30.2
- net VDD_uC: now also C29.1, C30.1
Other:
- note added: "MOTOR CONNECTIONS"
- note removed: "ADD 2 mm STRAIN RELIEF HOLES\nFOR EVERY PTH"

Commit message: automated commit
Other:
- note added: "FRONT LEFT"
- note added: "FRONT RIGHT"
- note added: "REAR LEFT"
- note added: "REAR RIGHT"
Changed lines of the file:
@@
 Text Notes 7825 4400 0    50   ~ 0
 MOTOR CONNECTIONS
+Text Notes 7650 2850 0    50   ~ 0
+FRONT RIGHT
+Text Notes 7600 3850 0    50   ~ 0
+REAR RIGHT
+Text Notes 7600 4950 0    50   ~ 0
+FRONT LEFT
+Text Notes 7600 5950 0    50   ~ 0
+REAR LEFT
 $EndSCHEMATC

Commit message: automated commit
Parts:
- removed TP18, TP19, TP24, TP25, TP26, TP27, TP32, TP33: PTH_0.5_mm, TestPoint:TestPoint_THTPad_D1.0mm_Drill0.5mm, symbol custom:PTH_0.5_mm
Other:
- moved on the sheet: J1, J2, J3, J4, J5, J6, J7, J8, NPTH1, NPTH2, NPTH3, NPTH4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

Commit message: automated commit
Parts:
- removed TP20, TP21, TP22, TP23, TP28, TP29, TP30, TP31: PTH_0.5_mm, TestPoint:TestPoint_THTPad_D1.0mm_Drill0.5mm, symbol custom:PTH_0.5_mm
Changed lines of the file:
@@
 	2700 3025 2425 3025
-Wire Wire Line
-	1750 3125 2175 3125
 Wire Wire Line
 	2625 3225 2625 3125
@@
 Connection ~ 4225 3125
 Connection ~ 4425 2925
-Text GLabel 1750 3025 0    50   Input ~ 0
+Text GLabel 2150 3025 0    50   Input ~ 0
 R_MOTOR
-Text GLabel 1750 3125 0    50   Input ~ 0
+Text GLabel 2150 3125 0    50   Input ~ 0
 R_DIR
 $Comp
@@
 	2700 5125 2425 5125
 Wire Wire Line
-	1750 5225 2175 5225
-Wire Wire Line
 	2625 5325 2625 5225
 Wire Wire Line
@@
 	2625 5225 2700 5225
 Connection ~ 2425 5125
-Wire Wire Line
-	2425 5125 1900 5125
 $Comp
 L custom:RC0603JR-071KL R?
@@
 F 4 "1k0" V 3975 5450 50  0000 C CNN "Resistance"
 	1    3975 5450
-	1    0    0    -1
-$EndComp
-$Comp
-L custom:SGM3157YC6 U?
-U 1 1 5CB049D7
-P 3050 5175
-AR Path="/5CB049D7" Ref="U?"  Part="1"
-AR Path="/5C10107F/5CB049D7" Ref="U4"  Part="1"
-F 0 "U4" H 2800 5400 50  0000 L BNN
-F 1 "SGM3157YC6" H 2800 5000 50  0000 L BNN
-F 2 "Package_TO_SOT_SMD:SOT-23-6" H 2800 4875 50  0001 L BNN
-F 3 "/home/dj/datasheets/SGM3157YC6.pdf" H 2800 4775 50  0001 L BNN
-	1    3050 5175
 	1    0    0    -1
 $EndComp
@@
 $EndComp
 Connection ~ 3775 5025
-Text GLabel 1750 5125 0    50   Input ~ 0
+Text GLabel 2150 5125 0    50   Input ~ 0
 L_MOTOR
-Text GLabel 1750 5225 0    50   Input ~ 0
+Text GLabel 2150 5225 0    50   Input ~ 0
 L_DIR
 $Comp
@@
 Connection ~ 4225 5225
 Connection ~ 4425 5025
-Wire Wire Line
-	1900 2975 1900 3025
-$Comp
-L custom:PTH_0.5_mm TP?
-U 1 1 5CF3A85A
-P 1900 2975
-AR Path="/5C5AE643/5CF3A85A" Ref="TP?"  Part="1"
-AR Path="/5C3EC885/5CF3A85A" Ref="TP?"  Part="1"
-AR Path="/5C10107F/5CF3A85A" Ref="TP22"  Part="1"
-F 0 "TP22" H 1850 3175 50  0000 L BNN
-F 1 "PTH_0.5_mm" V 1875 3150 50  0001 L BNN
-F 2 "TestPoint:TestPoint_THTPad_D1.0mm_Drill0.5mm" H 2100 2975 50  0001 L BNN
-F 3 "~" H 2100 2975 50  0001 C CNN
-	1    1900 2975
-	1    0    0    -1
-$EndComp
-$Comp
-L custom:PTH_0.5_mm TP?
-U 1 1 5CF46407
-P 2175 2975
-AR Path="/5C5AE643/5CF46407" Ref="TP?"  Part="1"
-AR Path="/5C3EC885/5CF46407" Ref="TP?"  Part="1"
-AR Path="/5C10107F/5CF46407" Ref="TP23"  Part="1"
-F 0 "TP23" H 2125 3175 50  0000 L BNN
-F 1 "PTH_0.5_mm" V 2150 3150 50  0001 L BNN
-F 2 "TestPoint:TestPoint_THTPad_D1.0mm_Drill0.5mm" H 2375 2975 50  0001 L BNN
-F 3 "~" H 2375 2975 50  0001 C CNN
-	1    2175 2975
-	1    0    0    -1
-$EndComp
-Wire Wire Line
-	2175 2975 2175 3125
-Connection ~ 2175 3125
-Wire Wire Line
-	2175 3125 2625 3125
-Connection ~ 1900 3025
-Wire Wire Line
-	1900 3025 2425 3025
-Wire Wire Line
-	1750 3025 1900 3025
-Wire Wire Line
-	1900 5075 1900 5125
-$Comp
-L custom:PTH_0.5_mm TP?
-U 1 1 5CF67601
-P 1900 5075
-AR Path="/5C5AE643/5CF67601" Ref="TP?"  Part="1"
-AR Path="/5C3EC885/5CF67601" Ref="TP?"  Part="1"
-AR Path="/5C10107F/5CF67601" Ref="TP30"  Part="1"
-F 0 "TP30" H 1850 5275 50  0000 L BNN
-F 1 "PTH_0.5_mm" V 1875 5250 50  0001 L BNN
-F 2 "TestPoint:TestPoint_THTPad_D1.0mm_Drill0.5mm" H 2100 5075 50  0001 L BNN
-F 3 "~" H 2100 5075 50  0001 C CNN
-	1    1900 5075
-	1    0    0    -1
-$EndComp
-$Comp
-L custom:PTH_0.5_mm TP?
-U 1 1 5CF67608
-P 2175 5075
-AR Path="/5C5AE643/5CF67608" Ref="TP?"  Part="1"
-AR Path="/5C3EC885/5CF67608" Ref="TP?"  Part="1"
-AR Path="/5C10107F/5CF67608" Ref="TP31"  Part="1"
-F 0 "TP31" H 2125 5275 50  0000 L BNN
-F 1 "PTH_0.5_mm" V 2150 5250 50  0001 L BNN
-F 2 "TestPoint:TestPoint_THTPad_D1.0mm_Drill0.5mm" H 2375 5075 50  0001 L BNN
-F 3 "~" H 2375 5075 50  0001 C CNN
-	1    2175 5075
-	1    0    0    -1
-$EndComp
-Wire Wire Line
-	2175 5075 2175 5225
-Connection ~ 2175 5225
-Wire Wire Line
-	2175 5225 2625 5225
-Connection ~ 1900 5125
-Wire Wire Line
-	1900 5125 1750 5125
-Wire Wire Line
-	3625 2875 3625 2925
-$Comp
-L custom:PTH_0.5_mm TP?
-U 1 1 5CF6C119
-P 3625 2875
-AR Path="/5C5AE643/5CF6C119" Ref="TP?"  Part="1"
-AR Path="/5C3EC885/5CF6C119" Ref="TP?"  Part="1"
-AR Path="/5C10107F/5CF6C119" Ref="TP20"  Part="1"
-F 0 "TP20" H 3575 3075 50  0000 L BNN
-F 1 "PTH_0.5_mm" V 3600 3050 50  0001 L BNN
-F 2 "TestPoint:TestPoint_THTPad_D1.0mm_Drill0.5mm" H 3825 2875 50  0001 L BNN
-F 3 "~" H 3825 2875 50  0001 C CNN
-	1    3625 2875
-	1    0    0    -1
-$EndComp
-$Comp
-L custom:PTH_0.5_mm TP?
-U 1 1 5CF6C120
-P 3975 2875
-AR Path="/5C5AE643/5CF6C120" Ref="TP?"  Part="1"
-AR Path="/5C3EC885/5CF6C120" Ref="TP?"  Part="1"
-AR Path="/5C10107F/5CF6C120" Ref="TP21"  Part="1"
-F 0 "TP21" H 3925 3075 50  0000 L BNN
-F 1 "PTH_0.5_mm" V 3950 3050 50  0001 L BNN
-F 2 "TestPoint:TestPoint_THTPad_D1.0mm_Drill0.5mm" H 4175 2875 50  0001 L BNN
-F 3 "~" H 4175 2875 50  0001 C CNN
-	1    3975 2875
-	1    0    0    -1
-$EndComp
-Wire Wire Line
-	3975 2875 3975 3025
-Wire Wire Line
-	3625 4975 3625 5025
-$Comp
-L custom:PTH_0.5_mm TP?
-U 1 1 5CF7075B
-P 3625 4975
-AR Path="/5C5AE643/5CF7075B" Ref="TP?"  Part="1"
-AR Path="/5C3EC885/5CF7075B" Ref="TP?"  Part="1"
-AR Path="/5C10107F/5CF7075B" Ref="TP28"  Part="1"
-F 0 "TP28" H 3575 5175 50  0000 L BNN
-F 1 "PTH_0.5_mm" V 3600 5150 50  0001 L BNN
-F 2 "TestPoint:TestPoint_THTPad_D1.0mm_Drill0.5mm" H 3825 4975 50  0001 L BNN
-F 3 "~" H 3825 4975 50  0001 C CNN
-	1    3625 4975
-	1    0    0    -1
-$EndComp
-$Comp
-L custom:PTH_0.5_mm TP?
-U 1 1 5CF70762
-P 3975 4975
-AR Path="/5C5AE643/5CF70762" Ref="TP?"  Part="1"
-AR Path="/5C3EC885/5CF70762" Ref="TP?"  Part="1"
-AR Path="/5C10107F/5CF70762" Ref="TP29"  Part="1"
-F 0 "TP29" H 3925 5175 50  0000 L BNN
-F 1 "PTH_0.5_mm" V 3950 5150 50  0001 L BNN
-F 2 "TestPoint:TestPoint_THTPad_D1.0mm_Drill0.5mm" H 4175 4975 50  0001 L BNN
-F 3 "~" H 4175 4975 50  0001 C CNN
-	1    3975 4975
-	1    0    0    -1
-$EndComp
-Wire Wire Line
-	3975 4975 3975 5125
-Connection ~ 3625 5025
-Wire Wire Line
-	3625 5025 3400 5025
-Wire Wire Line
-	3625 5025 3775 5025
-Connection ~ 3625 2925
-Wire Wire Line
-	3625 2925 3775 2925
-Wire Wire Line
-	3400 2925 3625 2925
-Connection ~ 3975 3025
-Connection ~ 3975 5125
 $Comp
 L custom:NPTH_2mm NPTH1
@@
 Wire Wire Line
 	5375 6075 5900 6075
+Wire Wire Line
+	3400 2925 3775 2925
+$Comp
+L custom:SGM3157YC6 U?
+U 1 1 5CB049D7
+P 3050 5175
+AR Path="/5CB049D7" Ref="U?"  Part="1"
+AR Path="/5C10107F/5CB049D7" Ref="U4"  Part="1"
+F 0 "U4" H 2800 5400 50  0000 L BNN
+F 1 "SGM3157YC6" H 2800 5000 50  0000 L BNN
+F 2 "Package_TO_SOT_SMD:SOT-23-6" H 2800 4875 50  0001 L BNN
+F 3 "/home/dj/datasheets/SGM3157YC6.pdf" H 2800 4775 50  0001 L BNN
+	1    3050 5175
+	1    0    0    -1
+$EndComp
+Wire Wire Line
+	3400 5025 3775 5025
+Wire Wire Line
+	2150 3025 2425 3025
+Wire Wire Line
+	2150 3125 2625 3125
+Wire Wire Line
+	2150 5125 2425 5125
+Wire Wire Line
+	2150 5225 2625 5225
 $EndSCHEMATC

Commit message: automated commit
Parts:
- J1, J2, J3, J4, J5, J6, J7, J8: footprint TestPoint:TestPoint_THTPad_D2.0mm_Drill1.0mm -> custom:TestPoint_THTPad_D2.0mm_Drill1.0mm
Changed lines of the file:
@@
 F 0 "J1" H 6150 2725 50  0000 C CNN
 F 1 "PTH_1_mm" H 6050 2625 50  0000 C CNN
-F 2 "TestPoint:TestPoint_THTPad_D2.0mm_Drill1.0mm" H 6050 2725 50  0001 C CNN
+F 2 "custom:TestPoint_THTPad_D2.0mm_Drill1.0mm" H 6050 2725 50  0001 C CNN
 F 3 "" H 6050 2725 50  0001 C CNN
 	1    6050 2725
@@
 F 0 "J2" H 6150 2925 50  0000 C CNN
 F 1 "PTH_1_mm" H 6050 2825 50  0000 C CNN
-F 2 "TestPoint:TestPoint_THTPad_D2.0mm_Drill1.0mm" H 6050 2925 50  0001 C CNN
+F 2 "custom:TestPoint_THTPad_D2.0mm_Drill1.0mm" H 6050 2925 50  0001 C CNN
 F 3 "" H 6050 2925 50  0001 C CNN
 	1    6050 2925
@@
 F 0 "J3" H 6150 3775 50  0000 C CNN
 F 1 "PTH_1_mm" H 6050 3675 50  0000 C CNN
-F 2 "TestPoint:TestPoint_THTPad_D2.0mm_Drill1.0mm" H 6050 3775 50  0001 C CNN
+F 2 "custom:TestPoint_THTPad_D2.0mm_Drill1.0mm" H 6050 3775 50  0001 C CNN
 F 3 "" H 6050 3775 50  0001 C CNN
 	1    6050 3775
@@
 F 0 "J4" H 6150 3975 50  0000 C CNN
 F 1 "PTH_1_mm" H 6050 3875 50  0000 C CNN
-F 2 "TestPoint:TestPoint_THTPad_D2.0mm_Drill1.0mm" H 6050 3975 50  0001 C CNN
+F 2 "custom:TestPoint_THTPad_D2.0mm_Drill1.0mm" H 6050 3975 50  0001 C CNN
 F 3 "" H 6050 3975 50  0001 C CNN
 	1    6050 3975
@@
 F 0 "J5" H 6150 4825 50  0000 C CNN
 F 1 "PTH_1_mm" H 6050 4725 50  0000 C CNN
-F 2 "TestPoint:TestPoint_THTPad_D2.0mm_Drill1.0mm" H 6050 4825 50  0001 C CNN
+F 2 "custom:TestPoint_THTPad_D2.0mm_Drill1.0mm" H 6050 4825 50  0001 C CNN
 F 3 "" H 6050 4825 50  0001 C CNN
 	1    6050 4825
@@
 F 0 "J6" H 6150 5025 50  0000 C CNN
 F 1 "PTH_1_mm" H 6050 4925 50  0000 C CNN
-F 2 "TestPoint:TestPoint_THTPad_D2.0mm_Drill1.0mm" H 6050 5025 50  0001 C CNN
+F 2 "custom:TestPoint_THTPad_D2.0mm_Drill1.0mm" H 6050 5025 50  0001 C CNN
 F 3 "" H 6050 5025 50  0001 C CNN
 	1    6050 5025
@@
 F 0 "J7" H 6150 5875 50  0000 C CNN
 F 1 "PTH_1_mm" H 6050 5775 50  0000 C CNN
-F 2 "TestPoint:TestPoint_THTPad_D2.0mm_Drill1.0mm" H 6050 5875 50  0001 C CNN
+F 2 "custom:TestPoint_THTPad_D2.0mm_Drill1.0mm" H 6050 5875 50  0001 C CNN
 F 3 "" H 6050 5875 50  0001 C CNN
 	1    6050 5875
@@
 F 0 "J8" H 6150 6075 50  0000 C CNN
 F 1 "PTH_1_mm" H 6050 5975 50  0000 C CNN
-F 2 "TestPoint:TestPoint_THTPad_D2.0mm_Drill1.0mm" H 6050 6075 50  0001 C CNN
+F 2 "custom:TestPoint_THTPad_D2.0mm_Drill1.0mm" H 6050 6075 50  0001 C CNN
 F 3 "" H 6050 6075 50  0001 C CNN
 	1    6050 6075

Commit message: automated commit
Parts:
- U3, U4: footprint Package_TO_SOT_SMD:SOT-23-6 -> Package_TO_SOT_SMD:SOT-363_SC-70-6
Changed lines of the file:
@@
 F 0 "U3" H 2800 3300 50  0000 L BNN
 F 1 "SGM3157YC6" H 2800 2900 50  0000 L BNN
-F 2 "Package_TO_SOT_SMD:SOT-23-6" H 2800 2775 50  0001 L BNN
-F 3 "/home/dj/datasheets/SGM3157YC6.pdf" H 2800 2675 50  0001 L BNN
+F 2 "Package_TO_SOT_SMD:SOT-363_SC-70-6" H 2800 2775 50  0001 L BNN
+F 3 "/home/dj/datasheets/SGM00371010.pdf" H 2800 2675 50  0001 L BNN
 	1    3050 3075
 	1    0    0    -1
@@
 F 0 "U4" H 2800 5400 50  0000 L BNN
 F 1 "SGM3157YC6" H 2800 5000 50  0000 L BNN
-F 2 "Package_TO_SOT_SMD:SOT-23-6" H 2800 4875 50  0001 L BNN
-F 3 "/home/dj/datasheets/SGM3157YC6.pdf" H 2800 4775 50  0001 L BNN
+F 2 "Package_TO_SOT_SMD:SOT-363_SC-70-6" H 2800 4875 50  0001 L BNN
+F 3 "/home/dj/datasheets/SGM00371010.pdf" H 2800 4775 50  0001 L BNN
 	1    3050 5175
 	1    0    0    -1
