File: nu.ai_motor_controller/nu.ai_motor_controller.kicad_pcb (KiCad board)
At the start: 4 copper layers, 108 x 92 mm, 190 parts, among them J1 PTH_1_mm, J10 Conn_02x05_Odd_Even, J11 DX4R105JJCR1800, J12 XT60_RA_MALE, J13 S4B-XH-A, J14 NP_Screw_Terminal_01x02, J15 XT60_RA_MALE, J16 S4B-XH-A, J17 S4B-XH-A, J18 XT60_RA_FEMALE, J2 PTH_1_mm, J3 PTH_1_mm, J4 PTH_1_mm, J5 PTH_1_mm, J6 PTH_1_mm, J7 PTH_1_mm, J8 PTH_1_mm, J9 Conn_02x12_Odd_Even, Q1 IRF9540N, Q2 SSM3K35AMFV, Q3 SSM3K35AMFV, SW1 TACTILE_SWITCH, SW2 TACTILE_SWITCH, SW3 TACTILE_SWITCH, U1 AZ2117, U10 MP6513, U2 AZ2117, U3 SGM3157YC6, U4 SGM3157YC6, U5 LMR23625CFDDAR, U6 MP6513, U7 MP6513, U8 MP6513, U9 ATmega32U4-AU, Y1 7M-16.000MAAE-T

Commit message: automated commit
Parts:
- moved TP27 11.0 mm to (109.3, 120.2)
- moved TP26 10.6 mm to (109.3, 117.2)
- moved J3 0.36 mm to (164.1, 59.3)
- moved J4 0.36 mm to (164.1, 64.4)
Routing:
- net Net-(J5-Pad1): track 12.9 -> 6.75 mm
- net Net-(J2-Pad1): track 8.52 -> 5.95 mm
- net Net-(J1-Pad1): track 7.15 -> 4.83 mm
- net I2C_SDA: track 10.6 -> 9.14 mm, vias 1 -> 0
- net GND: track 46.3 -> 44.9 mm, vias 39 -> 40
- net Net-(J6-Pad1): track 13.3 -> 14.4 mm
- net USART_RX: track 10.9 -> 9.90 mm, vias 1 -> 0
- net VDD_BAT: track 26.0 -> 25.2 mm
- added copper zone on F.Cu, net Net-(J3-Pad1)
- added copper zone on F.Cu, net Net-(J4-Pad1)
- added copper zone on F.Cu, net Net-(J7-Pad1)
- added copper zone on F.Cu, net Net-(J8-Pad1)

Commit message: automated commit
Parts:
- Q1: footprint Package_TO_SOT_THT:TO-220-3_Horizontal_TabDown -> custom:TO-220-3_Horizontal_TabDown
- moved TP33 24.8 mm to (161.6, 120.2)
- moved TP32 19.1 mm to (155.2, 120.2)
- moved TP14 16.3 mm to (117.5, 80.0)
- moved JP1 13.3 mm to (146.5, 112.5), turned to 0 degrees
- moved TP11 11.8 mm to (105.5, 96.9)
- moved TP22 8.89 mm to (129.1, 66.3)
- moved NPTH6 7.30 mm to (99.4, 126.7)
- moved TP21 5.59 mm to (123.5, 66.3)
- moved TP15 3.43 mm to (141.7, 121.3)
- moved TP54 3.25 mm to (94.5, 75.5)
- moved TP53 2.67 mm to (89.3, 88.6)
- moved C4 2.03 mm to (108.5, 101.5)
- moved NPTH5 1.45 mm to (97.0, 120.6)
- moved R1 1.27 mm to (108.5, 99.9)
- moved TP17 1.02 mm to (137.5, 121.3)
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Connections:
- F2 pad 1: Net-(F2-Pad1) -> /battery/TAP_2
- J12 pad 2: Net-(F2-Pad1) -> /battery/TAP_2
- J15 pad 2: Net-(F2-Pad1) -> /battery/TAP_2
- J18 pad 1: Net-(F2-Pad1) -> /battery/TAP_2
- TP53 pad 1: Net-(F2-Pad1) -> /battery/TAP_2
Routing:
- net /battery/TAP_1: track 0.00 -> 140.5 mm
- net /battery/TAP_0: track 0.00 -> 138.5 mm
- net Net-(J8-Pad1): track 0.00 -> 13.3 mm
- net GND: track 44.9 -> 54.2 mm, vias 40 -> 55
- net Net-(D8-Pad1): track 10.6 -> 19.4 mm
- net Net-(C27-Pad1): track 0.00 -> 5.81 mm
- net Net-(J7-Pad1): track 0.00 -> 5.58 mm
- net Net-(C4-Pad2): track 0.00 -> 5.43 mm
- net +5V: track 0.00 -> 5.36 mm, vias 0 -> 6
- net Net-(R3-Pad2): track 8.10 -> 3.99 mm
- net Net-(D8-Pad6): track 15.2 -> 19.1 mm
- net Net-(R8-Pad1): track 1.72 -> 4.90 mm
- net Net-(R12-Pad1): track 1.70 -> 4.75 mm
- net Net-(R11-Pad1): track 1.70 -> 4.75 mm
- net Net-(C3-Pad2): track 2.37 -> 5.41 mm
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- added copper zone on F.Cu, net +3V3
- added copper zone on F.Cu, net +5V
- added copper zone on In2.Cu, net +5V
- added copper zone on F.Cu, net /battery/TAP_2
- added copper zone on In2.Cu, net /battery/TAP_2
- added copper zone on F.Cu, net Net-(C27-Pad1)
- added copper zone on F.Cu, net Net-(C3-Pad2)
- added copper zone on F.Cu, net Net-(C4-Pad2)
- added copper zone on F.Cu, net Net-(R3-Pad2)
- added copper zone on In2.Cu, net VDD_BAT

Commit message: automated commit
Parts:
- moved TP53 2.16 mm to (89.5, 86.5)
Changed lines of the file:
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@@
   )
   (module TestPoint:TestPoint_THTPad_D1.0mm_Drill0.5mm (layer F.Cu)
-    (at 89.335 88.625)
+    (at 89.462 86.466)
     (descr "THT pad as test Point, diameter 1.0mm, hole diameter 0.5mm")
     (tags "test point THT pad")
     (attr virtual)
-    (fp_text reference TP53 (at -3.175 0) (layer F.SilkS)
+    (fp_text reference TP53 (at -0.508 2.159) (layer F.SilkS)
       (effects (font (size 1 1) (thickness 0.15)))
     )
@@
   (module custom:X4B-XH-A (layer F.Cu)
     (at 83.62 80.37)
-    (fp_text reference J16 (at 5.715 5.969) (layer F.SilkS)
+    (fp_text reference J16 (at 5.334 4.191) (layer F.SilkS)
       (effects (font (size 1 1) (thickness 0.15)))
     )
@@
   (segment (start 100.638 109.326) (end 100.638 107.578) (width 0.25) (layer F.Cu) (net 1))
   (via (at 99.368 110.088) (size 0.8) (drill 0.4) (layers F.Cu B.Cu) (net 1))
-  (via (at 160.836 63.098) (size 0.8) (drill 0.4) (layers F.Cu B.Cu) (net 3))
   (segment (start 160.074 61.828) (end 158.326 61.828) (width 0.25) (layer F.Cu) (net 1))
   (segment (start 124.768 80.878) (end 121.974 83.672) (width 0.25) (layer F.Cu) (net 1))
   (segment (start 124.768 75.798) (end 124.768 80.878) (width 0.25) (layer F.Cu) (net 1))
-  (via (at 159.82 63.098) (size 0.8) (drill 0.4) (layers F.Cu B.Cu) (net 3))
   (segment (start 126.292 75.747) (end 126.343 75.798) (width 0.25) (layer F.Cu) (net 2))
   (segment (start 126.292 74.341) (end 126.292 75.747) (width 0.25) (layer F.Cu) (net 2))
   (segment (start 126.343 80.421) (end 129.594 83.672) (width 0.25) (layer F.Cu) (net 2))
   (segment (start 126.343 75.798) (end 126.343 80.421) (width 0.25) (layer F.Cu) (net 2))
+  (via (at 160.836 63.098) (size 0.8) (drill 0.4) (layers F.Cu B.Cu) (net 3))
+  (via (at 159.82 63.098) (size 0.8) (drill 0.4) (layers F.Cu B.Cu) (net 3))
   (segment (start 163.301 44.846) (end 169.801 44.846) (width 0.25) (layer F.Cu) (net 3))
   (via (at 141.278 73.766) (size 0.8) (drill 0.4) (layers F.Cu B.Cu) (net 3))
@@
   (segment (start 118.748 116.692) (end 118.748 115.473) (width 0.25) (layer F.Cu) (net 3))
   (segment (start 118.748 115.473) (end 118.799 115.422) (width 0.25) (layer F.Cu) (net 3))
+  (via (at 109.401 78.592) (size 0.8) (drill 0.4) (layers F.Cu B.Cu) (net 3))
+  (via (at 110.671 78.592) (size 0.8) (drill 0.4) (layers F.Cu B.Cu) (net 3))
+  (segment (start 104.0605 78.7) (end 104.448 78.3125) (width 0.25) (layer F.Cu) (net 3))
+  (segment (start 103.058 78.7) (end 104.0605 78.7) (width 0.25) (layer F.Cu) (net 3))
   (segment (start 116.322 98.658) (end 116.132 98.468) (width 0.25) (layer F.Cu) (net 4))
   (segment (start 121.466 98.658) (end 116.322 98.658) (width 0.25) (layer F.Cu) (net 4))
@@
   (segment (start 116.196 93.832) (end 116.132 93.768) (width 0.25) (layer F.Cu) (net 6))
   (segment (start 121.466 93.832) (end 116.196 93.832) (width 0.25) (layer F.Cu) (net 6))
-  (via (at 109.401 78.592) (size 0.8) (drill 0.4) (layers F.Cu B.Cu) (net 3))
-  (via (at 110.671 78.592) (size 0.8) (drill 0.4) (layers F.Cu B.Cu) (net 3))
-  (segment (start 104.0605 78.7) (end 104.448 78.3125) (width 0.25) (layer F.Cu) (net 3))
-  (segment (start 103.058 78.7) (end 104.0605 78.7) (width 0.25) (layer F.Cu) (net 3))
   (segment (start 106.8265 96.88) (end 106.171106 96.88) (width 0.25) (layer F.Cu) (net 7))
   (segment (start 106.171106 96.88) (end 105.464 96.88) (width 0.25) (layer F.Cu) (net 7))
@@
   (segment (start 94.491 75.595) (end 94.542 75.544) (width 0.25) (layer F.Cu) (net 47))
   (segment (start 94.491 79.1) (end 94.491 75.595) (width 0.25) (layer F.Cu) (net 47))
-  (via (at 89.208 79.989) (size 0.8) (drill 0.4) (layers F.Cu B.Cu) (net 60))
-  (via (at 87.811 79.989) (size 0.8) (drill 0.4) (layers F.Cu B.Cu) (net 60))
-  (via (at 87.811 82.783) (size 0.8) (drill 0.4) (layers F.Cu B.Cu) (net 60))
-  (via (at 89.208 82.783) (size 0.8) (drill 0.4) (layers F.Cu B.Cu) (net 60))
-  (via (at 87.811 81.386) (size 0.8) (drill 0.4) (layers F.Cu B.Cu) (net 60))
   (segment (start 117.148 58.272) (end 112.322 58.272) (width 0.25) (layer F.Cu) (net 49))
   (segment (start 109.528 63.098) (end 109.274 62.844) (width 0.25) (layer F.Cu) (net 50))
@@
   (segment (start 144.011654 80.947225) (end 144.011654 80.137223) (width 0.25) (layer F.Cu) (net 59))
   (segment (start 144.70234 85.444271) (end 144.70234 81.637911) (width 0.25) (layer F.Cu) (net 59))
+  (via (at 89.208 79.989) (size 0.8) (drill 0.4) (layers F.Cu B.Cu) (net 60))
+  (via (at 87.811 79.989) (size 0.8) (drill 0.4) (layers F.Cu B.Cu) (net 60))
+  (via (at 87.811 82.783) (size 0.8) (drill 0.4) (layers F.Cu B.Cu) (net 60))
+  (via (at 89.208 82.783) (size 0.8) (drill 0.4) (layers F.Cu B.Cu) (net 60))
+  (via (at 87.811 81.386) (size 0.8) (drill 0.4) (layers F.Cu B.Cu) (net 60))
   (segment (start 83.62 79.1) (end 85.652 81.132) (width 0.5) (layer B.Cu) (net 61))
   (segment (start 85.652 93.578) (end 83.62 95.61) (width 0.5) (layer B.Cu) (net 61))
@@
     (polygon
       (pts
-        (xy 95.431 56.113) (xy 95.431 73.258) (xy 89.716 78.973) (xy 89.716 88.498) (xy 87.811 90.403)
-        (xy 87.811 103.484) (xy 89.462 105.135) (xy 91.494 105.135) (xy 105.972 119.613) (xy 160.201 119.613)
-        (xy 169.218 110.596) (xy 169.218 85.831) (xy 171.631 83.418) (xy 181.283 83.418) (xy 182.934 85.069)
-        (xy 182.934 110.596) (xy 183.061 134.98) (xy 74.984 134.98) (xy 74.984 55.986) (xy 77.143 53.827)
-        (xy 87.176 53.827) (xy 93.018 53.7)
-      )
-    )
+        (xy 95.431 56.113) (xy 95.431 73.258) (xy 89.716 78.973) (xy 89.716 84.434) (xy 90.732 85.45)
+        (xy 90.732 87.482) (xy 87.811 90.403) (xy 87.811 103.484) (xy 89.462 105.135) (xy 91.494 105.135)
+        (xy 105.972 119.613) (xy 160.201 119.613) (xy 169.218 110.596) (xy 169.218 85.831) (xy 171.631 83.418)
+        (xy 181.283 83.418) (xy 182.934 85.069) (xy 182.934 110.596) (xy 183.061 134.98) (xy 74.984 134.98)
+        (xy 74.984 55.986) (xy 77.143 53.827) (xy 87.176 53.827) (xy 93.018 53.7)
+      )
+    )

Commit message: automated commit
Parts:
- removed REF**: Symbol_HighVoltage_SilkTop_Small, custom:Symbol_HighVoltage_SilkTop_Small
- removed TP18, TP19, TP24, TP25, TP26, TP27, TP32, TP33: PTH_0.5_mm, TestPoint:TestPoint_THTPad_D1.0mm_Drill0.5mm
- moved R35 94.4 mm to (35.5, 45.7), turned to 270 degrees
- moved Q3 92.9 mm to (37.8, 45.7), turned to 0 degrees
- moved R34 90.6 mm to (39.8, 46.4), turned to 90 degrees
- moved BZ1 86.6 mm to (47.7, 46.2), turned to 90 degrees
- moved L2 82.2 mm to (220.3, 53.8), turned to 0 degrees
- moved C11 80.4 mm to (216.9, 58.1), turned to 0 degrees
- moved R16 79.3 mm to (216.9, 56.5), turned to 0 degrees
- moved C15 78.5 mm to (213.6, 61.3), turned to 0 degrees
- moved R15 78.5 mm to (216.9, 55.0), turned to 0 degrees
- moved C19 77.4 mm to (217.0, 52.8), turned to 0 degrees
- moved C18 76.0 mm to (210.9, 62.2), turned to 270 degrees
- moved C20 71.1 mm to (211.4, 54.5), turned to 270 degrees
- moved R13 69.4 mm to (213.4, 46.0), turned to 180 degrees
- moved C10 68.2 mm to (210.1, 50.7)
- moved C12 67.9 mm to (203.9, 62.1), turned to 270 degrees
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Routing:
- net Net-(J6-Pad1): track 14.4 -> 0.30 mm
- net Net-(J8-Pad1): track 13.3 -> 0.00 mm
- net Net-(J5-Pad1): track 6.75 -> 0.00 mm
- net Net-(J2-Pad1): track 5.95 -> 0.00 mm
- net +5V: track 5.36 -> 11.1 mm
- net Net-(J7-Pad1): track 5.58 -> 0.00 mm
- net +3V3: track 0.00 -> 5.34 mm
- net Net-(J1-Pad1): track 4.83 -> 0.00 mm
- net GND: track 54.2 -> 57.7 mm, vias 55 -> 58
- net RST_TVS: track 8.05 -> 10.8 mm
- added copper zone on F.Cu, net +1V8

Commit message: automated commit
Parts:
- moved R6 107.0 mm to (251.2, 115.3), turned to 0 degrees
- moved TP17 105.4 mm to (248.6, 111.8), turned to 0 degrees
- moved R4 101.2 mm to (248.0, 115.3), turned to 0 degrees
- moved TP15 98.0 mm to (244.4, 111.8), turned to 90 degrees
- moved TP13 96.9 mm to (249.3, 126.4), turned to 180 degrees
- moved U2 95.4 mm to (247.0, 120.7), turned to 270 degrees
- moved C28 88.1 mm to (244.7, 126.0), turned to 180 degrees
- moved C27 88.1 mm to (242.4, 118.9), turned to 270 degrees
- moved JP1 81.9 mm to (239.7, 120.5), turned to 180 degrees
- moved D2 81.7 mm to (237.9, 139.6)
- moved D4 81.7 mm to (228.0, 138.3)
- moved D5 81.7 mm to (239.7, 129.4)
- moved J9 81.7 mm to (231.8, 115.4)
- moved TP36 81.7 mm to (242.0, 134.5)
- moved TP38 81.7 mm to (242.0, 138.0)
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Routing:
- net Net-(C17-Pad1): track 13.8 -> 10.0 mm
- net PWM_4A: track 4.27 -> 6.65 mm
- net RESETn: track 0.00 -> 2.26 mm
- net Net-(C16-Pad1): track 11.8 -> 10.2 mm
- net JTAG_TDI: track 10.1 -> 11.1 mm
- net JTAG_TMS: track 9.68 -> 10.5 mm
- net JTAG_TDO: track 9.46 -> 8.74 mm

Commit message: automated commit
Parts:
- moved D1 18.2 mm to (160.6, 36.7)
- moved R27 17.8 mm to (156.3, 35.8)
- moved TP50 17.8 mm to (153.2, 35.8)
Changed lines of the file:
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@@
   )
   (module custom:SOT-457 (layer F.Cu)
-    (at 158.042 54.716 270)
+    (at 160.582 36.682 270)
     (fp_text reference D1 (at 0.254 -2.54 270) (layer F.SilkS)
       (effects (font (size 1 1) (thickness 0.15)))
@@
   )
   (module Resistor_SMD:R_0603_1608Metric (layer F.Cu)
-    (at 153.724 53.446 180)
+    (at 156.264 35.793 180)
     (descr "Resistor SMD 0603 (1608 Metric), square (rectangular) end terminal, IPC_7351 nominal, (Body size source: http://www.tortai-tech.com/upload/download/2011102023233369053.pdf), generated with kicad-footprint-generator")
     (tags resistor)
@@
   )
   (module TestPoint:TestPoint_THTPad_D1.0mm_Drill0.5mm (layer F.Cu)
-    (at 150.676 53.446 270)
+    (at 153.216 35.793 270)
     (descr "THT pad as test Point, diameter 1.0mm, hole diameter 0.5mm")
     (tags "test point THT pad")
@@
   (segment (start 45.2915 86.480501) (end 45.2915 88.193) (width 0.25) (layer F.Cu) (net 82))
   (segment (start 47.044 86.480501) (end 47.044 88.2185) (width 0.25) (layer F.Cu) (net 83))
-  (segment (start 152.9365 53.446) (end 150.676 53.446) (width 0.25) (layer F.Cu) (net 84))
+  (segment (start 155.4765 35.793) (end 153.216 35.793) (width 0.25) (layer F.Cu) (net 84))
   (segment (start 128.601 161.65) (end 129.467 161.65) (width 0.25) (layer F.Cu) (net 85))
   (segment (start 127.773 160.822) (end 128.601 161.65) (width 0.25) (layer F.Cu) (net 85))

Commit message: automated commit
Parts:
- moved D4 88.1 mm to (143.8, 112.5)
- moved D2 88.1 mm to (153.7, 113.7)
- moved J9 88.1 mm to (147.6, 89.6)
- moved R6 88.1 mm to (167.0, 89.5)
- moved TP13 88.1 mm to (165.1, 100.6)
- moved TP36 88.1 mm to (157.8, 108.7)
- moved TP44 88.1 mm to (143.0, 102.3)
- moved TP47 88.1 mm to (143.8, 118.6)
- moved U2 88.1 mm to (162.8, 94.9)
- moved C27 88.1 mm to (158.2, 93.1)
- moved C28 88.1 mm to (160.5, 100.2)
- moved D5 88.1 mm to (155.5, 103.6)
- moved JP1 88.1 mm to (155.5, 94.7)
- moved R4 88.1 mm to (163.8, 89.5)
- moved TP17 88.1 mm to (164.4, 86.0)
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
Commit message: automated commit
Parts:
- removed TP20, TP21, TP22, TP23, TP28, TP29, TP30, TP31: PTH_0.5_mm, TestPoint:TestPoint_THTPad_D1.0mm_Drill0.5mm
- added C32: ESH336M035AC3AA, Capacitor_THT:CP_Radial_D5.0mm_P2.00mm, F.Cu at (134.7, 76.6)
- added D9: CM1293A-04SO, custom:SOT-457, B.Cu at (174.3, 68.6)
- added Q4: SSM3K35AMFV, Package_TO_SOT_SMD:SOT-723, F.Cu at (53.0, 92.0)
- added R41: CR0603-JW-103ELF, Resistor_SMD:R_0603_1608Metric, F.Cu at (50.6, 91.8)
- D6, R18, R19, R36, TP35: moved to B.Cu
- moved C26 86.3 mm to (138.4, 101.7)
- moved R3 86.3 mm to (127.7, 98.4)
- moved R5 86.3 mm to (127.7, 95.1)
- moved TP12 86.3 mm to (136.2, 94.1)
- moved U1 86.3 mm to (133.0, 99.4)
- moved TP16 85.5 mm to (125.9, 96.8)
- moved C25 82.3 mm to (127.0, 101.8), turned to 180 degrees
- moved TP14 80.2 mm to (105.7, 103.2)
- moved TP35 56.9 mm to (162.2, 62.7), turned to 180 degrees
- moved C30 53.7 mm to (126.2, 106.3)
- moved R12 53.7 mm to (119.1, 107.3)
- moved R32 53.7 mm to (126.2, 108.1)
- moved U4 53.7 mm to (122.6, 106.3)
- moved R11 53.7 mm to (119.1, 105.3)
- moved R33 53.7 mm to (126.2, 104.5)
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Connections:
- D6 pad 1: /microcontroller/M_USB_D+ -> Net-(D6-Pad1)
- D6 pad 3: /microcontroller/M_USB_D- -> Net-(D6-Pad3)
- J11 pad 1: Net-(J11-Pad1) -> /microcontroller/VBUS
- R29 pad 2: GND -> Net-(Q4-Pad3)
- R30 pad 2: GND -> Net-(Q4-Pad3)
- R31 pad 2: GND -> Net-(Q4-Pad3)
Routing:
- net /microcontroller/M_USB_D-: track 0.00 -> 17.4 mm, vias 0 -> 1
- net /microcontroller/M_USB_D+: track 0.00 -> 16.3 mm, vias 0 -> 1
- net GND: track 57.7 -> 70.5 mm, vias 58 -> 65
- net +5V: track 11.1 -> 3.53 mm, vias 6 -> 7
- net +3V3: track 5.34 -> 0.00 mm
- net /microcontroller/UGND: track 5.59 -> 9.92 mm, vias 0 -> 3
- net Net-(R8-Pad1): track 4.90 -> 1.72 mm
- net R_DIR: track 5.29 -> 2.14 mm
- net Net-(R12-Pad1): track 4.75 -> 1.70 mm
- net Net-(R11-Pad1): track 4.75 -> 1.70 mm
- net Net-(R7-Pad1): track 4.77 -> 1.72 mm
- net R_MOTOR: track 4.45 -> 2.04 mm
- net L_DIR: track 4.31 -> 2.01 mm
- net L_MOTOR: track 4.32 -> 2.04 mm
- net VDD_BAT: track 25.2 -> 23.2 mm, vias 12 -> 17
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- added copper zone on In1.Cu, net /microcontroller/UGND
- added copper zone on F.Cu, net Net-(C21-Pad1)
