File: nu.ai_motor_controller/nu.ai_motor_controller.kicad_pcb (KiCad board)
At the start: 4 copper layers, 108 x 92 mm, 177 parts, among them J1 PTH_1_mm, J10 Conn_02x05_Odd_Even, J11 DX4R105JJCR1800, J12 XT60_RA_MALE, J13 S4B-XH-A, J14 NP_Screw_Terminal_01x02, J15 XT60_RA_MALE, J16 S4B-XH-A, J17 S4B-XH-A, J18 XT60_RA_FEMALE, J2 PTH_1_mm, J3 PTH_1_mm, J4 PTH_1_mm, J5 PTH_1_mm, J6 PTH_1_mm, J7 PTH_1_mm, J8 PTH_1_mm, J9 Conn_02x12_Odd_Even, Q1 IRF9540N, Q2 SSM3K35AMFV, Q3 SSM3K35AMFV, Q4 SSM3K35AMFV, SW1 TACTILE_SWITCH, SW2 TACTILE_SWITCH, SW3 TACTILE_SWITCH, U1 AZ2117, U10 MP6513, U2 AZ2117, U3 SGM3157YC6, U4 SGM3157YC6, U5 LMR23625CFDDAR, U6 MP6513, U7 MP6513, U8 MP6513, U9 ATmega32U4-AU, Y1 7M-16.000MAAE-T

Commit message: automated commit
Parts:
- removed TP36, TP37, TP38, TP39, TP40, TP41, TP42, TP43, TP44, TP45, TP46, TP47, TP48, TP49, TP50, TP51: PTH_0.5_mm, TestPoint:TestPoint_THTPad_D1.0mm_Drill0.5mm
- C6, J3, J4, U7: moved to B.Cu
- moved TP5 105.4 mm to (141.3, 114.2)
- moved TP7 103.3 mm to (138.0, 114.3)
- moved R24 103.2 mm to (140.7, 120.3), turned to 90 degrees
- moved R29 101.1 mm to (140.7, 117.0), turned to 90 degrees
- moved R25 99.7 mm to (138.8, 120.3), turned to 90 degrees
- moved TP6 98.9 mm to (139.6, 112.8)
- moved R30 97.6 mm to (138.8, 117.0), turned to 90 degrees
- moved R26 96.3 mm to (136.9, 120.3), turned to 90 degrees
- moved R31 94.1 mm to (136.9, 117.0), turned to 90 degrees
- moved R41 87.3 mm to (135.1, 113.6), turned to 180 degrees
- moved Q4 85.3 mm to (135.0, 115.4), turned to 270 degrees
- moved J7 30.0 mm to (161.7, 123.5)
- moved J8 25.1 mm to (155.9, 129.4)
- moved R35 16.8 mm to (115.4, 71.7), turned to 180 degrees
- moved Q3 13.6 mm to (115.4, 74.0), turned to 270 degrees
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Connections:
- D1 pad 4: Net-(D1-Pad4) -> (no net)
- D1 pad 6: Net-(D1-Pad6) -> (no net)
- D3 pad 1: JTAG_TMS -> JTAG_TCK
- D3 pad 3: JTAG_TCK -> JTAG_TMS
- D5 pad 6: Net-(D5-Pad6) -> (no net)
- D6 pad 1: Net-(D6-Pad1) -> (no net)
- D6 pad 3: Net-(D6-Pad3) -> (no net)
- D8 pad 3: Net-(D8-Pad3) -> (no net)
- D8 pad 4: Net-(D8-Pad4) -> (no net)
- D9 pad 5: Net-(D9-Pad5) -> (no net)
- J10 pad 7: Net-(J10-Pad7) -> (no net)
- J11 pad 4: Net-(J11-Pad4) -> (no net)
- J9 pad 2: +3V3 -> GND
- J9 pad 4: +3V3 -> GND
- J9 pad 5: GND -> +3V3
- J9 pad 6: GND -> +3V3
- U9 pad 1: Net-(U9-Pad1) -> (no net)
Routing:
- net Net-(R11-Pad1): track 1.70 -> 36.2 mm, vias 0 -> 2
- net Net-(R12-Pad1): track 1.70 -> 33.8 mm, vias 0 -> 2
- net SPI_SCK: track 9.22 -> 2.63 mm
- net USART_RX: track 9.90 -> 3.85 mm
- net BAT_1: track 1.75 -> 7.53 mm
- net SPI_MOSI: track 8.27 -> 2.63 mm, vias 1 -> 0
- net SPI_SSn: track 11.5 -> 6.03 mm
- net I2C_SDA: track 9.14 -> 3.85 mm
- net JTAG_TCK: track 8.70 -> 13.9 mm
- net PWM_4D: track 9.42 -> 4.27 mm, vias 1 -> 0
- net PWM_3A: track 17.5 -> 12.9 mm
- net BAT_2: track 1.73 -> 6.22 mm
- net BAT_0: track 1.74 -> 5.66 mm
- net GND: track 70.5 -> 74.1 mm, vias 65 -> 69
- net JTAG_TDO: track 8.74 -> 12.3 mm, vias 1 -> 0
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- added copper zone on B.Cu, net GND
- added copper zone on B.Cu, net Net-(J3-Pad1)
- added copper zone on B.Cu, net Net-(J4-Pad1)
- added copper zone on F.Cu, net Net-(Q4-Pad3)
- added copper zone on B.Cu, net VDD_BAT
- added copper zone on In2.Cu, net VDD_uC
- removed copper zone on F.Cu, net Net-(J3-Pad1)
- removed copper zone on F.Cu, net Net-(J4-Pad1)

Commit message: automated commit
Parts:
- C14, C15, L1: moved to B.Cu
- moved D1 17.6 mm to (163.0, 54.1)
- moved TP35 17.1 mm to (176.1, 72.8)
- moved TP54 8.08 mm to (102.5, 74.4)
- moved L1 6.83 mm to (151.2, 67.8), turned to 90 degrees
- moved TP55 6.70 mm to (105.5, 74.4)
- moved C14 6.21 mm to (151.2, 63.6), turned to 90 degrees
- moved TP34 4.81 mm to (130.2, 80.0)
- moved C15 4.80 mm to (155.2, 70.2), turned to 180 degrees
- moved R14 1.59 mm to (145.8, 71.4)
- moved C13 0.32 mm to (155.5, 57.9)
- moved C10 0.28 mm to (154.9, 63.4)
Routing:
- net RST_TVS: track 10.8 -> 88.0 mm, vias 0 -> 1
- net Net-(D8-Pad6): track 19.1 -> 71.1 mm
- net Net-(D8-Pad1): track 19.4 -> 70.6 mm, vias 0 -> 2
- net /microcontroller/VBUS: track 2.05 -> 42.4 mm, vias 0 -> 2
- net R_MOTOR: track 2.04 -> 29.0 mm
- net Net-(R8-Pad1): track 1.72 -> 26.4 mm, vias 0 -> 1
- net Net-(R7-Pad1): track 1.72 -> 23.2 mm, vias 0 -> 1
- net /microcontroller/uC_RSTn: track 8.96 -> 22.3 mm
- net GND: track 74.1 -> 84.0 mm, vias 69 -> 77
- net VDD_uC: track 21.9 -> 30.3 mm, vias 6 -> 11
- net /microcontroller/uC_AVCC: track 5.01 -> 0.00 mm, vias 1 -> 2
- net Net-(R14-Pad2): track 4.10 -> 2.08 mm
- added copper zone on B.Cu, net /microcontroller/uC_AVCC
- added copper zone on F.Cu, net /microcontroller/uC_AVCC

Commit message: automated commit
Parts:
- R27: moved to B.Cu
- moved R27 18.3 mm to (160.7, 53.6), turned to 270 degrees
- moved TP17 9.32 mm to (167.6, 94.7)
- moved TP15 8.40 mm to (160.3, 94.3)
Routing:
- net SPI_MISO: track 6.90 -> 75.7 mm, vias 0 -> 1
- net I2C_SCL: track 6.81 -> 73.6 mm, vias 0 -> 2
- net I2C_SDA: track 3.85 -> 69.7 mm, vias 0 -> 2
- net SPI_MOSI: track 2.63 -> 66.0 mm, vias 0 -> 1
- net SPI_SCK: track 2.63 -> 63.5 mm, vias 0 -> 1
- net USART_RX: track 3.85 -> 64.5 mm, vias 0 -> 1
- net L_DIR: track 2.01 -> 58.9 mm, vias 0 -> 2
- net BAT_0: track 5.66 -> 62.3 mm, vias 0 -> 1
- net USART_TX: track 7.50 -> 63.8 mm, vias 0 -> 1
- net L_MOTOR: track 2.04 -> 58.4 mm, vias 0 -> 2
- net SPI_SSn: track 6.03 -> 60.2 mm, vias 0 -> 1
- net BAT_2: track 6.22 -> 59.4 mm, vias 0 -> 1
- net BAT_1: track 7.53 -> 60.5 mm, vias 0 -> 1
- net Net-(Q3-Pad1): track 1.87 -> 53.3 mm, vias 0 -> 2
- net +5V: track 3.53 -> 44.7 mm
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- added copper zone on B.Cu, net VDD_uC

Commit message: automated commit
Parts:
- added MH5: M4_MOUNTING_HOLE, MountingHole:MountingHole_4.3mm_M4_Pad, F.Cu at (178.1, 78.3)
- added R42: NP_R_0603, custom:NP_0603, F.Cu at (172.8, 81.6)
- moved TP6 6.48 mm to (143.3, 118.1)
- moved TP7 5.21 mm to (134.4, 118.1)
- moved TP13 0.78 mm to (165.8, 100.3)
- moved C5 0.36 mm to (114.2, 60.6)
Connections:
- D5 pad 3: PWM_4D -> PWM_3A
- D5 pad 4: PWM_3A -> PWM_4D
- J9 pad 11: PWM_3A -> PWM_4D
- J9 pad 14: PWM_4D -> PWM_3A
Routing:
- net PWM_4D: track 4.27 -> 54.7 mm, vias 0 -> 1
- net PWM_4A: track 4.27 -> 49.2 mm, vias 0 -> 1
- net PWM_3A: track 12.9 -> 46.0 mm, vias 0 -> 1
- net /microcontroller/uC_RSTn: track 22.3 -> 46.1 mm, vias 0 -> 1
- net BAT_1: track 60.5 -> 66.6 mm, vias 1 -> 2
- net Net-(MH5-Pad1): track 0.00 -> 5.91 mm
- net +1V8: track 0.00 -> 4.07 mm
- net BAT_0: track 62.3 -> 65.9 mm
- net GND: track 85.8 -> 89.0 mm, vias 78 -> 80
- net USART_TX: track 63.8 -> 65.4 mm
- net USART_RX: track 64.5 -> 65.9 mm
- net I2C_SDA: track 69.7 -> 70.8 mm
- net I2C_SCL: track 73.6 -> 74.3 mm
- added copper zone on F.Cu, net Net-(R4-Pad2)

Commit message: automated commit
Parts:
- removed TP15: PTH_0.5_mm, TestPoint:TestPoint_THTPad_D1.0mm_Drill0.5mm
- added F1: NP_FUSE_0603, Fuse:Fuse_0603_1608Metric, F.Cu at (90.0, 78.6)
- added F3: NP_FUSE_0603, Fuse:Fuse_0603_1608Metric, F.Cu at (90.0, 84.2)
- TP1, TP10, TP11, TP12, TP13, TP14, TP16, TP17, TP2, TP3, TP34, TP35, TP4, TP5, TP52, TP53, TP54, TP55, TP56, TP6, TP7, TP8, TP9: footprint TestPoint:TestPoint_THTPad_D1.0mm_Drill0.5mm -> custom:TestPoint_THTPad_D1.0mm_Drill0.5mm
- moved TP35 9.35 mm to (167.3, 69.5)
- moved C25 4.02 mm to (129.8, 104.6), turned to 270 degrees
- moved TP53 1.46 mm to (88.6, 87.7)
- moved D1 0.13 mm to (163.1, 54.1)
Routing:
- net +5V: track 44.7 -> 34.2 mm
- net Net-(D8-Pad1): track 70.6 -> 64.7 mm, vias 2 -> 1
- net GND: track 89.0 -> 91.7 mm
- net Net-(C27-Pad1): track 2.68 -> 0.00 mm
- net /microcontroller/UGND: track 9.92 -> 12.0 mm
- net Net-(R11-Pad1): track 35.9 -> 37.4 mm
- net SPI_SSn: track 60.2 -> 61.6 mm
- net /microcontroller/VBUS: track 29.6 -> 28.4 mm
- net SPI_MOSI: track 66.0 -> 65.3 mm
- net /battery/TAP_2: vias 6 -> 12

Commit message: automated commit
Parts:
- J1, J2, J3, J4, J5, J6, J7, J8: footprint TestPoint:TestPoint_THTPad_D2.0mm_Drill1.0mm -> custom:TestPoint_THTPad_D2.0mm_Drill1.0mm
- MH1, MH2, MH3, MH4, MH5: footprint MountingHole:MountingHole_4.3mm_M4_Pad -> custom:MountingHole_4.3mm_M4_Pad
Connections:
- D1 pad 4: (no net) -> Net-(D1-Pad4)
- D1 pad 6: (no net) -> Net-(D1-Pad6)
- D5 pad 6: (no net) -> Net-(D5-Pad6)
- D6 pad 1: (no net) -> Net-(D6-Pad1)
- D6 pad 3: (no net) -> Net-(D6-Pad3)
- D8 pad 3: (no net) -> Net-(D8-Pad3)
- D8 pad 4: (no net) -> Net-(D8-Pad4)
- D9 pad 5: (no net) -> Net-(D9-Pad5)
- J10 pad 7: (no net) -> Net-(J10-Pad7)
- J11 pad 4: (no net) -> Net-(J11-Pad4)
- U9 pad 1: (no net) -> Net-(U9-Pad1)

Commit message: automated commit
Parts:
- moved TP35 1.77 mm to (166.3, 70.9)
Routing:
- net /microcontroller/VBUS: track 28.4 -> 31.3 mm
- net /microcontroller/M_USB_D+: track 16.3 -> 17.2 mm
- net SPI_MISO: track 75.7 -> 75.2 mm
