File: nu.ai_motor_controller/nu.ai_motor_controller.kicad_pcb (KiCad board)
At the start: 4 copper layers, 108 x 92 mm, 183 parts, among them J1 PTH_1_mm, J10 Conn_02x05_Odd_Even, J11 DX4R105JJCR1800, J12 XT60_RA_MALE, J13 S4B-XH-A, J14 NP_Screw_Terminal_01x02, J15 XT60_RA_MALE, J16 S4B-XH-A, J17 S4B-XH-A, J18 XT60_RA_FEMALE, J2 PTH_1_mm, J3 PTH_1_mm, J4 PTH_1_mm, J5 PTH_1_mm, J6 PTH_1_mm, J7 PTH_1_mm, J8 PTH_1_mm, J9 Conn_02x12_Odd_Even, Q1 IRF9540N, Q2 SSM3K35AMFV, Q3 SSM3K35AMFV, Q4 AO3407A, Q5 AO3407A, Q6 AO3407A, Q7 SSM3K35AMFV, Q8 SSM3K35AMFV, Q9 SSM3K35AMFV, SW1 TACTILE_SWITCH, SW2 TACTILE_SWITCH, SW3 TACTILE_SWITCH, U1 AZ2117, U10 MP6513, U2 AZ2117, U3 SGM3157YC6, U4 SGM3157YC6, U5 LMR23625CFDDAR, U6 MP6513, U7 MP6513, U8 MP6513, U9 ATmega32U4-AU, Y1 7M-16.000MAAE-T

Commit message: automated commit
Parts:
- moved NPTH6 6.77 mm to (103.6, 121.5)
- moved REF** 2.23 mm to (143.5, 56.4) (x2)
Changed lines of the file:
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@@
   )
   (module custom:Symbol_HighVoltage_SilkTop_Small (layer F.Cu)
-    (at 145.542 57.3024 180)
+    (at 143.51 56.388 180)
     (descr "Symbol, High Voltage, Type 2, Copper Top, Very Small,")
     (tags "Symbol, High Voltage, Type 2, Copper Top, Very Small,")
@@
   (module custom:NPTH_2mm (layer F.Cu)
     (at 96.955 120.629)
-    (fp_text reference NPTH5 (at 3.81 1.27) (layer F.SilkS)
+    (fp_text reference NPTH5 (at 0.7842 2.4086) (layer F.SilkS)
       (effects (font (size 1 1) (thickness 0.15)))
     )
@@
       (effects (font (size 1 1) (thickness 0.15)))
     )
-    (fp_text user %R (at 3.883 1.291) (layer B.SilkS)
+    (fp_text user %R (at 0.7842 2.4086) (layer B.SilkS)
       (effects (font (size 1 1) (thickness 0.15)) (justify mirror))
     )
@@
   )
   (module custom:NPTH_2mm (layer F.Cu)
-    (at 99.368 126.725)
+    (at 103.632 121.4628)
     (fp_text reference NPTH6 (at 4.191 0) (layer F.SilkS)
       (effects (font (size 1 1) (thickness 0.15)))
@@
   )
   (module custom:Symbol_HighVoltage_SilkTop_Small (layer B.Cu)
-    (at 145.542 57.3024)
+    (at 143.51 56.388)
     (descr "Symbol, High Voltage, Type 2, Copper Top, Very Small,")
     (tags "Symbol, High Voltage, Type 2, Copper Top, Very Small,")

Commit message: automated commit
Other:
- board text added: "NU.AI_MOTOR_CONTROLER REV 1.1"
- board text removed: "NU.AI_MOTOR_CONTROLER REV 1.0"
Changed lines of the file:
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@@
     (effects (font (size 1 1) (thickness 0.15)))
   )
-  (gr_text "NU.AI_MOTOR_CONTROLER\nREV 1.0" (at 107.188 88.5444) (layer B.SilkS)
+  (gr_text "NU.AI_MOTOR_CONTROLER\nREV 1.1" (at 107.188 88.5444) (layer B.SilkS)
     (effects (font (size 1.5 1.5) (thickness 0.3)) (justify mirror))
   )
@@
   (gr_line (start 97.028 59.3852) (end 97.028 58.3692) (layer F.SilkS) (width 0.2))
   (gr_line (start 96.52 58.8772) (end 97.536 58.8772) (layer F.SilkS) (width 0.2))
-  (gr_text "NU.AI_MOTOR_CONTROLER\nREV 1.0" (at 107.188 88.5444) (layer B.Cu)
+  (gr_text "NU.AI_MOTOR_CONTROLER\nREV 1.1" (at 107.188 88.5444) (layer B.Cu)
     (effects (font (size 1.5 1.5) (thickness 0.3)) (justify mirror))
   )

Commit message: automated commit
Other:
- board text added: "BACK"
- board text added: "FRONT"
- board text added: "LEFT"
- board text added: "RIGHT"
Changed lines of the file:
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@@
-(kicad_pcb (version 20171130) (host pcbnew 5.0.1)
+(kicad_pcb (version 20171130) (host pcbnew 5.1.0)
   (general
     (thickness 1.6)
-    (drawings 60)
+    (drawings 64)
     (tracks 1091)
     (zones 0)
@@
     (zone_45_only yes)
     (trace_min 0.2)
-    (segment_width 0.2)
-    (edge_width 0.15)
     (via_size 0.8)
     (via_drill 0.4)
@@
     (uvia_min_size 0.2)
     (uvia_min_drill 0.1)
+    (edge_width 0.15)
+    (segment_width 0.2)
     (pcb_text_width 0.3)
     (pcb_text_size 1.5 1.5)
@@
     (fp_line (start -0.49784 -2.19964) (end 0.70104 0.89916) (layer B.SilkS) (width 0.381))
   )
+  (gr_text LEFT (at 128.7272 147.828) (layer Dwgs.User)
+    (effects (font (size 5 5) (thickness 0.75)))
+  )
+  (gr_text BACK (at 206.8576 90.3224) (layer Dwgs.User)
+    (effects (font (size 5 5) (thickness 0.75)))
+  )
+  (gr_text RIGHT (at 129.9972 25.8064) (layer Dwgs.User)
+    (effects (font (size 5 5) (thickness 0.75)))
+  )
+  (gr_text FRONT (at 47.1932 89.9668) (layer Dwgs.User)
+    (effects (font (size 5 5) (thickness 0.75)))
+  )
   (dimension 92.049614 (width 0.3) (layer F.SilkS)

Commit message: automated commit
Parts:
- J14: moved to B.Cu
- moved TP55 3.56 mm to (106.7, 71.1)
- moved TP54 3.33 mm to (102.5, 71.1)
- turned J14 to 90 degrees
Connections:
- D1 pad 4: (no net) -> Net-(D1-Pad4)
- D1 pad 6: (no net) -> Net-(D1-Pad6)
- D5 pad 3: (no net) -> Net-(D5-Pad3)
- D5 pad 6: (no net) -> Net-(D5-Pad6)
- D6 pad 1: (no net) -> Net-(D6-Pad1)
- D6 pad 3: (no net) -> Net-(D6-Pad3)
- D8 pad 3: (no net) -> Net-(D8-Pad3)
- D8 pad 4: (no net) -> Net-(D8-Pad4)
- D9 pad 5: (no net) -> Net-(D9-Pad5)
- J10 pad 7: (no net) -> Net-(J10-Pad7)
- J11 pad 4: (no net) -> Net-(J11-Pad4)
- J14 pad 1: VDD_BAT -> GND
- J14 pad 2: GND -> VDD_BAT
- U9 pad 1: (no net) -> Net-(U9-Pad1)
Routing:
- net VDD_uC: track 30.8 -> 25.4 mm, vias 14 -> 12
- net /microcontroller/uC_AVCC: track 10.6 -> 6.04 mm
- net Net-(D8-Pad6): track 71.1 -> 69.1 mm
- net Net-(D8-Pad1): track 64.7 -> 63.6 mm
- net PWM_4A: track 49.2 -> 48.4 mm

Commit message: automated commit
Parts:
- U3, U4: footprint Package_TO_SOT_SMD:SOT-23-6 -> Package_TO_SOT_SMD:SOT-363_SC-70-6
Routing:
- net Net-(R12-Pad1): track 33.8 -> 34.8 mm
